File: PCB/Main Board/Protection.kicad_sch (KiCad schematic)
At the start: 0 parts

Commit message: InAmp Progress
Other:
- company: (none) -> Harry and Yuki - EEE3 Instrumentation
Changed lines of the file:
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@@
 	(generator_version "9.0")
 	(paper "A4")
+	(title_block
+		(date "2026-01-15")
+		(rev "Draft")
+		(company "Harry and Yuki - EEE3 Instrumentation")
+		(comment 1 "Work in Progress")
+	)
 	(hierarchical_label "In"
 		(shape bidirectional)
