File: PCB/Main Board/Amplifier.kicad_sch (KiCad schematic)
At the start: 30 parts

Commit message: InAmp Progress
Parts:
- removed JP?: SolderJumper_2_Bridged, Jumper:SolderJumper-2_P1.3mm_Bridged_RoundedPad1.0x1.5mm, symbol Jumper:SolderJumper_2_Bridged
- removed R?: 10k, symbol Device:R
- added R1: 22.6k, symbol Device:R
- added R3: 11.3k, symbol Device:R
- added U1: DG411xY, Package_SO:SOIC-16_3.9x9.9mm_P1.27mm, symbol Analog_Switch:DG411xY
- R?: value 10k -> 18k
Connections:
- net Out: now also R3.1; no longer U?.6
- net at R?.2, U?.7: now also R?.2, U?.2 (-), U1.6
- net InvAmpx10: now reaches U?.8
- net at R?.1, R?.2, R?.2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: now also R1.1
- net ACC27k: now reaches U?.8
- net ACC270: now reaches U?.8
- net InAmpx10: now reaches U?.8
- net ACCen: now reaches U?.8
- net ACC2.7k: now reaches U?.8
- net InAmpx3: now reaches U?.1
- new net: R1.2, U1.7
- new net: R3.2, U?.6
- new net InvAmp/2: U1.8
Other:
- note removed: "Optional Additional gain For extended range"
- company: (none) -> Harry and Yuki - EEE3 Instrumentation
- title: (none) -> Instrumentation Amplifier
- moved on the sheet: C?, JP?, R?, U?, U?A, U?B

Commit message: ABB, InAmp
Parts:
- R1: value 22.6k -> 11k
- R3: value 11.3k -> 5.5k
- R?: value 10k -> 49k
- R?: value 18k -> 9.1k
Other:
- note added: "11.11k"
- note added: "49.9k"
- note added: "5.544k"
- note added: "9.09k"
- note added: "Only for voltage amplification"
Changed lines of the file:
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@@
 		)
 	)
+	(text "11.11k"
+		(exclude_from_sim no)
+		(at 265.43 63.5 0)
+		(effects
+			(font
+				(size 1.27 1.27)
+			)
+			(justify right top)
+		)
+	)
 	(text "Cut if \npopulating"
 		(exclude_from_sim no)
@@
 		)
 	)
+	(text "Only for voltage\namplification"
+		(exclude_from_sim no)
+		(at 163.83 83.82 0)
+		(effects
+			(font
+				(size 1.27 1.27)
+			)
+			(justify right top)
+		)
+	)
+	(text "5.544k"
+		(exclude_from_sim no)
+		(at 266.7 63.5 0)
+		(effects
+			(font
+				(size 1.27 1.27)
+			)
+			(justify left top)
+		)
+	)
+	(text "49.9k\n"
+		(exclude_from_sim no)
+		(at 266.7 66.04 0)
+		(effects
+			(font
+				(size 1.27 1.27)
+			)
+			(justify left top)
+		)
+	)
 	(text "Cutoffs:\n27Hz\n270Hz\n2.7kHz\n27kHz"
 		(exclude_from_sim no)
@@
 		)
 	)
+	(text "9.09k\n"
+		(exclude_from_sim no)
+		(at 265.43 66.04 0)
+		(effects
+			(font
+				(size 1.27 1.27)
+			)
+			(justify right top)
+		)
+	)
 	(text "R-R 3.6V OpAmp"
 		(exclude_from_sim no)
@@
 			)
 		)
-		(property "Value" "10k"
+		(property "Value" "49k"
 			(at 234.95 66.04 90)
 			(effects
@@
 			)
 		)
-		(property "Value" "22.6k"
+		(property "Value" "11k"
 			(at 190.5 53.34 90)
 			(effects
@@
 			)
 		)
-		(property "Value" "18k"
+		(property "Value" "9.1k"
 			(at 196.85 66.04 90)
 			(effects
@@
 			)
 		)
-		(property "Value" "11.3k"
+		(property "Value" "5.5k"
 			(at 241.3 53.34 90)
 			(effects

Commit message: Panik
Parts:
- added C?: 2.2p, symbol Device:C
- added C?: 22p, symbol Device:C
Connections:
- net Out: now also C?.2, C?.2
- net at R?.2, R?.2, U1.6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: now also C?.1
- net at R3.2, U?.6: now also C?.1
Other:
- note added: "Guard potential"
- note added: "Recheck capacitor values after opamp selection"
- moved on the sheet: R1, R3, R?, U1B, U?B

Commit message: Paniking further
Other:
- note removed: "Guard potential"
- moved on the sheet: U?A, U?B
Changed lines of the file:
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@@
 		)
 	)
-	(text "Guard potential"
-		(exclude_from_sim no)
-		(at 59.69 104.14 0)
-		(effects
-			(font
-				(size 1.27 1.27)
-			)
-		)
-	)
 	(text "9.09k\n"
 		(exclude_from_sim no)
@@
 	(wire
 		(pts
-			(xy 36.83 60.96) (xy 36.83 68.58)
+			(xy 36.83 60.96) (xy 36.83 72.39)
 		)
 		(stroke
@@
 	(wire
 		(pts
-			(xy 57.15 83.82) (xy 57.15 88.9)
+			(xy 57.15 87.63) (xy 57.15 88.9)
 		)
 		(stroke
@@
 	(wire
 		(pts
-			(xy 57.15 60.96) (xy 57.15 68.58)
+			(xy 57.15 60.96) (xy 57.15 72.39)
 		)
 		(stroke
@@
 	(wire
 		(pts
-			(xy 36.83 83.82) (xy 36.83 88.9)
+			(xy 36.83 87.63) (xy 36.83 88.9)
 		)
 		(stroke
@@
 	(hierarchical_label "InAmpx3"
 		(shape input)
-		(at 31.75 76.2 180)
+		(at 31.75 80.01 180)
 		(effects
 			(font
@@
 	(hierarchical_label "InAmpx10"
 		(shape input)
-		(at 52.07 76.2 180)
+		(at 52.07 80.01 180)
 		(effects
 			(font
@@
 	(symbol
 		(lib_id "Analog_Switch:DG411xY")
-		(at 57.15 76.2 270)
+		(at 57.15 80.01 270)
 		(unit 2)
 		(exclude_from_sim no)
@@
 		(dnp no)
 		(property "Reference" "U?"
-			(at 53.34 71.12 90)
+			(at 53.34 74.93 90)
 			(effects
 				(font
@@
 		)
 		(property "Value" "DG411xY"
-			(at 53.34 73.66 90)
+			(at 53.34 77.47 90)
 			(effects
 				(font
@@
 		)
 		(property "Footprint" "Package_SO:SOIC-16_3.9x9.9mm_P1.27mm"
-			(at 54.61 76.2 0)
+			(at 54.61 80.01 0)
 			(effects
 				(font
@@
 		)
 		(property "Datasheet" "https://datasheets.maximintegrated.com/en/ds/DG411-DG413.pdf"
-			(at 57.15 76.2 0)
+			(at 57.15 80.01 0)
 			(effects
 				(font
@@
 		)
 		(property "Description" "Quad SPST Monolithic CMOS Analog Switches, normally ON, 17Ohm Ron, SOIC-16"
-			(at 57.15 76.2 0)
+			(at 57.15 80.01 0)
 			(effects
 				(font
@@
 	(symbol
 		(lib_id "Analog_Switch:DG411xY")
-		(at 36.83 76.2 270)
+		(at 36.83 80.01 270)
 		(unit 1)
 		(exclude_from_sim no)
@@
 		(dnp no)
 		(property "Reference" "U?"
-			(at 33.02 71.12 90)
+			(at 33.02 74.93 90)
 			(effects
 				(font
@@
 		)
 		(property "Value" "DG411xY"
-			(at 33.02 73.66 90)
+			(at 33.02 77.47 90)
 			(effects
 				(font
@@
 		)
 		(property "Footprint" "Package_SO:SOIC-16_3.9x9.9mm_P1.27mm"
-			(at 34.29 76.2 0)
+			(at 34.29 80.01 0)
 			(effects
 				(font
@@
 		)
 		(property "Datasheet" "https://datasheets.maximintegrated.com/en/ds/DG411-DG413.pdf"
-			(at 36.83 76.2 0)
+			(at 36.83 80.01 0)
 			(effects
 				(font
@@
 		)
 		(property "Description" "Quad SPST Monolithic CMOS Analog Switches, normally ON, 17Ohm Ron, SOIC-16"
-			(at 36.83 76.2 0)
+			(at 36.83 80.01 0)
 			(effects
 				(font

Commit message: Signal
Connections:
- net +1V8 renamed +1.65V
Changed lines of the file:
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@@
+		)
+	)
+	(global_label "+1.65V"
+		(shape input)
+		(at 215.9 85.09 180)
+		(fields_autoplaced yes)
+		(effects
+			(font
+				(size 1.27 1.27)
+			)
+			(justify right)
+		)
+		(property "Intersheetrefs" "${INTERSHEET_REFS}"
+			(at 206.0205 85.09 0)
+			(effects
+				(font
+					(size 1.27 1.27)
+				)
+				(justify right)
+				(hide yes)
+			)
+		)
+	)
+	(global_label "+1.65V"
+		(shape input)
+		(at 165.1 158.75 0)
+		(fields_autoplaced yes)
+		(effects
+			(font
+				(size 1.27 1.27)
+			)
+			(justify left)
+		)
+		(property "Intersheetrefs" "${INTERSHEET_REFS}"
+			(at 174.9795 158.75 0)
+			(effects
+				(font
+					(size 1.27 1.27)
+				)
+				(justify left)
+				(hide yes)
+			)
 		)
 	)
@@
 	)
 	(symbol
-		(lib_id "power:+1V8")
-		(at 165.1 158.75 270)
-		(unit 1)
-		(exclude_from_sim no)
-		(in_bom yes)
-		(on_board yes)
-		(dnp no)
-		(fields_autoplaced yes)
-		(property "Reference" "#PWR0501"
-			(at 161.29 158.75 0)
-			(effects
-				(font
-					(size 1.27 1.27)
-				)
-				(hide yes)
-			)
-		)
-		(property "Value" "+1V8"
-			(at 168.91 158.7499 90)
-			(effects
-				(font
-					(size 1.27 1.27)
-				)
-				(justify left)
-			)
-		)
-		(property "Footprint" ""
-			(at 165.1 158.75 0)
-			(effects
-				(font
-					(size 1.27 1.27)
-				)
-				(hide yes)
-			)
-		)
-		(property "Datasheet" ""
-			(at 165.1 158.75 0)
-			(effects
-				(font
-					(size 1.27 1.27)
-				)
-				(hide yes)
-			)
-		)
-		(property "Description" "Power symbol creates a global label with name \"+1V8\""
-			(at 165.1 158.75 0)
-			(effects
-				(font
-					(size 1.27 1.27)
-				)
-				(hide yes)
-			)
-		)
-		(pin "1"
-		)
-		(instances
-			(project "Main Board"
-				(path "/20aae4b7-3fb8-4924-82e8-1e7a29a313f8/bd9549aa-e467-4112-8861-8ba41215560f"
-					(reference "#PWR0501")
-					(unit 1)
-				)
-				(path "/20aae4b7-3fb8-4924-82e8-1e7a29a313f8/cbba8371-ef6e-448c-bffb-b5e389595b93"
-					(reference "#PWR0601")
-					(unit 1)
-				)
-			)
-		)
-	)
-	(symbol
 		(lib_id "Device:R")
 		(at 133.35 133.35 90)
@@
 					(unit 1)
 				)
-			)
-		)
-	)
-	(symbol
-		(lib_id "power:+1V8")
-		(at 215.9 85.09 90)
-		(unit 1)
-		(exclude_from_sim no)
-		(in_bom yes)
-		(on_board yes)
-		(dnp no)
-		(fields_autoplaced yes)
-		(property "Reference" "#PWR0502"
-			(at 219.71 85.09 0)
-			(effects
-				(font
-					(size 1.27 1.27)
-				)
-				(hide yes)
-			)
-		)
-		(property "Value" "+1V8"
-			(at 212.09 85.0899 90)
-			(effects
-				(font
-					(size 1.27 1.27)
-				)
-				(justify left)
-			)
-		)
-		(property "Footprint" ""
-			(at 215.9 85.09 0)
-			(effects
-				(font
-					(size 1.27 1.27)
-				)
-				(hide yes)
-			)
-		)
-		(property "Datasheet" ""
-			(at 215.9 85.09 0)
-			(effects
-				(font
-					(size 1.27 1.27)
-				)
-				(hide yes)
-			)
-		)
-		(property "Description" "Power symbol creates a global label with name \"+1V8\""
-			(at 215.9 85.09 0)
-			(effects
-				(font
-					(size 1.27 1.27)
-				)
-				(hide yes)
-			)
-		)
-		(pin "1"
-		)
-		(instances
-			(project ""
-				(path "/20aae4b7-3fb8-4924-82e8-1e7a29a313f8/bd9549aa-e467-4112-8861-8ba41215560f"
-					(reference "#PWR0502")
-					(unit 1)
-				)
-				(path "/20aae4b7-3fb8-4924-82e8-1e7a29a313f8/cbba8371-ef6e-448c-bffb-b5e389595b93"
-					(reference "#PWR0602")
-					(unit 1)
-				)

Commit message: parts selection
Parts:
- removed C?: 22n, symbol Device:C
- removed R? (x3): 100k, symbol Device:R
- removed R?: 300, symbol Device:R
- removed R?: 3k, symbol Device:R
- removed R?: 270k, symbol Device:R
- removed R?: 22k, symbol Device:R
- removed R?: 30k, symbol Device:R
- removed U? (x3): ${SIM.PARAMS}, symbol Simulation_SPICE:OPAMP
- removed U? (x6): DG411xY, Package_SO:SOIC-16_3.9x9.9mm_P1.27mm, symbol Analog_Switch:DG411xY
- added C?: 2.2n, symbol Device:C
- added C?: 100n, symbol Device:C
- added R?: 300k, symbol Device:R
- added R?: 3k, symbol Device:R
- added R?: 10M, symbol Device:R
- added R?: 30k, symbol Device:R
- added R?: 2.7M, symbol Device:R
- added U (x3), U? (x2): TLV4172IPWR, symbol Device:Opamp_Quad
- added U? (x5): CD4066BM, Package_SO:SO-14_3.9x8.65mm_P1.27mm, symbol Analog_Switch:CD4066BM
- added U?: ${SIM.PARAMS}, symbol Simulation_SPICE:OPAMP
Connections:
- net +1.65V: now also U?.1 (+)
- net In+: now also U.3 (+)
- net In-: now also U?.5 (+)
- net at JP?.1 (A), R?.2: now also C?.1, R?.1, U?.11, U?.5
- net at R?.1: now also U?.6 (-), U?.7
- net at R1.1, R?.1, R?.2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: now also R?.2, U?.1, U?.4, U?.8
- net at R?.1: now also U.1, U.2 (-)
- new net: C?.2, R?.1, R?.1, R?.1, R?.1, R?.2, U?.10, U?.2 (-)
- new net: R?.2, U?.2
- new net: R?.2, U?.9
- new net: R?.2, U?.3
- new net 18V: C?.2, U?.14 (V_{DD})
- new net ACC_2.7k: U?.5
- new net ACC_270: U?.13
- new net ACC_27k: U?.6
- new net ACC_EN: U?.12
- new net GND: C?.1, U?.7 (V_{SS})
Other:
- note added: "i have moved the gain, sorry if i wasnt meant to delete this, i have a screenshot if we need to restore it sorry"
- note added: "these two are for the other amp but the schematics are linked"
- moved on the sheet: C?, JP?, R1, R3, R?, U1B, U?, U?B

Commit message: :anguished:
Parts:
- removed C?: 100n, symbol Device:C
- removed U (x3), U? (x2): TLV4172IPWR, symbol Device:Opamp_Quad
- removed U1, U?: DG411xY, Package_SO:SOIC-16_3.9x9.9mm_P1.27mm, symbol Analog_Switch:DG411xY
- removed U? (x5): CD4066BM, Package_SO:SO-14_3.9x8.65mm_P1.27mm, symbol Analog_Switch:CD4066BM
- removed U? (x3): ${SIM.PARAMS}, symbol Simulation_SPICE:OPAMP
- added C? (x10): 100n, symbol Device:C
- added C? (x2): 100p, symbol Device:C
- added JP?: SolderJumper_2_Bridged, Jumper:SolderJumper-2_P1.3mm_Bridged_RoundedPad1.0x1.5mm, symbol Jumper:SolderJumper_2_Bridged
- added R?: 20k, symbol Device:R
- added R?: 10k, symbol Device:R
- added R?: 2.21k, symbol Device:R
- added R?: 21.7k, symbol Device:R
- added R?: 4.72k, symbol Device:R
- added U? (x10): DG201, Package_SO:SOIC-16_3.9x9.9mm_P1.27mm, symbol More_symbols:DG201
- added U? (x6): OPA1662, Package_SO:SOIC-8_3.9x4.9mm_P1.27mm, symbol Device:Opamp_Dual
- added U? (x3): TLV2172, Package_SO:SOIC-8_3.9x4.9mm_P1.27mm, symbol Device:Opamp_Dual
Connections:
- net ACC_2.7k: now also U?.8
- net ACC_270: now also U?.9
- net ACC_27k: now also U?.1
- net ACC_EN: now also U?.16
- net GND: now also C?.1, C?.1, C?.1, C?.1, C?.1, C?.2, C?.2, C?.2, C?.2, C?.2, U?.5 (GND), U?.5 (GND)
- net In+: now also U?.3 (+)
- net In-: now also U?.5 (+)
- net InvAmpx10: now also U?.8
- net InvAmp/2: now also U?.1
- net Out: now also C?.2, R?.2, U?.7; no longer C?.2, C?.2, R3.1, R?.1
- net at R?.1: now also U?.6 (-), U?.7
- net at C?.1, R?.2, R?.2: now also U?.2, U?.2 (-), U?.7
- net at R1.2: now also U?.3
- net at C?.2, R?.1, R?.1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: now also U?.14, U?.6 (-)
- net at R?.2: now also U?.11
- net at R1.1, R?.1, R?.2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: now also U?.1, U?.10, U?.2, U?.6
- net at R?.2: now also U?.3
- net at R?.1, R?.2: now also U?.3 (+)
- net at C?.1, R?.1: now also JP?.2 (B), U?.15, U?.7; no longer JP?.1 (A), R?.2
- net at R?.2: now also U?.7
- net at C?.1, R3.2: now also U?.6
- net at R?.1: now also U?.1, U?.2 (-)
- net at R?.1, R?.2: now also U?.2 (-)
- net +1.65V renamed +1.65VA
- net +1.65VA: now also C?.2, U?.10, U?.15, U?.3 (+), U?.5 (+)
- new net: C?.2, C?.2, R3.1, R?.1, R?.1, U?.1
- new net: R?.1, R?.2, R?.2, U?.6 (-)
- new net: R?.1, U?.14
- new net: JP?.1 (A), JP?.1 (A), R?.2
- new net: R?.1, U?.11
- new net: C?.1, R?.1, R?.2
- new net: C?.1, R?.2, U?.5 (+)
- new net +18V: C?.1, C?.1, C?.1, C?.1, C?.1, U?.13 (V+), U?.13 (V+), U?.8 (V+), U?.8 (V+), U?.8 (V+)
- new net -18V: C?.2, C?.2, C?.2, C?.2, C?.2, U?.4 (V-), U?.4 (V-), U?.4 (V-), U?.4 (V-), U?.4 (V-)
Other:
- note added: "redo values"
- note removed: "Recheck capacitor values after opamp selection"
- note removed: "these two are for the other amp but the schematics are linked"
- moved on the sheet: C?, JP?, R1, R3, R?
