File: PCB/Main Board/Amplifier.kicad_sch (KiCad schematic)
At the start: 54 parts

Commit message: :cry:
Parts:
- removed R?: 10k, symbol Device:R
- removed U?: DG201, Package_SO:SOIC-16_3.9x9.9mm_P1.27mm, symbol More_symbols:DG201
- added C?: 22p, symbol Device:C
- added R?: 1.5k, symbol Device:R
- added R?: 1.1k, symbol Device:R
- added R?: 10k, symbol Device:R
- added R?: 3.9k, symbol Device:R
- added U?: DG201, Package_SO:SOIC-16_3.9x9.9mm_P1.27mm, symbol More_symbols:DG201
- C?: value 2.2n -> 5.6n
- C?: value 100p -> 47p
- C?: value 22p -> 7p
- C?: value 100p -> 56p
- R1: value 11k -> 12k
- R3: value 5.5k -> 39k
- R?: value 20k -> 9k
- R?: value 49k -> 100k
- R?: value 3k -> 2.7k
- R?: value 2.21k -> 1k
- R?: value 21.7k -> 50.4k
- R?: value 30k -> 27k
- R?: value 9.1k -> 39k
- R?: value 4.72k -> 4.85k
- U?: value OPA1662 -> TLV2172.
- U? (x2): value OPA1662 -> TLV2172
Connections:
- net +1.65VA: now also U?.15; no longer U?.10
- net at C?.1, R?.2, R?.2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: now also U?.11
- net at C?.2, C?.2, R?.1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: now also C?.2, R?.1, R?.1; no longer R3.1
- net at R1.2: now also R?.1; no longer U?.3
- net at R?.1: now also U?.14; no longer U?.11
- net ACC_2.7k renamed AC_1k
- net ACC_270 renamed AC_100
- net ACC_27k renamed AC_10k
- net ACC_EN renamed AC_EN
- net InvAmpx10 renamed x3
- net InvAmp/2 renamed /4
- new net: R?.2, U?.3
- new net: R?.1, R?.2
- new net: C?.1, R?.2, U?.10
- new net: R3.1, R?.2
- new net x1: U?.9
- new net x100: U?.16
Other:
- note added: "Cut to isolate"
- note added: "Falstad"
- note removed: "11.11k"
- note removed: "49.9k"
- note removed: "5.544k"
- note removed: "9.09k"
- note removed: "Cutoffs: 27Hz 270Hz 2.7kHz 27kHz"
- note removed: "i have moved the gain, sorry if i wasnt meant to delete this, i have a screenshot if we need to restore it sorry"
- note removed: "redo values"
- moved on the sheet: C?, JP?, R1, R3, R?, U?A, U?B, U?C, U?D

Commit message: 😫
Parts:
- added JP3, JP5: SolderJumper_2_Bridged, Jumper:SolderJumper-2_P1.3mm_Bridged_RoundedPad1.0x1.5mm, symbol Jumper:SolderJumper_2_Bridged
- added JP7, JP9: SolderJumper_2_Open, Jumper:SolderJumper-2_P1.3mm_Open_RoundedPad1.0x1.5mm, symbol Jumper:SolderJumper_2_Open
Connections:
- net +18V: now also JP9.1 (A); no longer C?.1, U?.8 (V+)
- net -18V: now also JP7.2 (B); no longer C?.2, U?.4 (V-)
- net GND: now also JP5.1 (A)
- net x100 renamed ~{x100}
- new net: C?.2, JP5.2 (B), JP7.1 (A), U?.4 (V-)
- new net: C?.1, JP3.1 (A), JP9.2 (B), U?.8 (V+)
- new net +3.3VA: JP3.2 (B)
Other:
- note removed: "R-R 3.6V OpAmp"

Commit message: Amplifier Switch
Parts:
- removed R? (x4): 10k, symbol Device:R
- removed U? (x3): OPA1662, Package_SO:SOIC-8_3.9x4.9mm_P1.27mm, symbol Device:Opamp_Dual
- removed U?: TLV2172., Package_SO:SOIC-8_3.9x4.9mm_P1.27mm, symbol Device:Opamp_Dual
- removed U? (x5): TLV2172, Package_SO:SOIC-8_3.9x4.9mm_P1.27mm, symbol Device:Opamp_Dual
- added U? (x6): OPA2197xD, Package_SO:SOIC-8_3.9x4.9mm_P1.27mm, symbol Amplifier_Operational:OPA2197xD
- added U?: INA828D, Package_SO:SOIC-8_3.9x4.9mm_P1.27mm, symbol INA828:INA828D
Connections:
- net +1.65VA: now also U?.3 (+), U?.3 (+)
- net +18V: now also U?.7 (Vs+), U?.8 (V+)
- net -18V: now also U?.4 (V-), U?.4 (Vs-)
- net GND: now also U?.5 (+)
- net In+: now also U?.3 (+)
- net In-: now also U?.2 (-)
- net Out: now also U?.7
- net at C?.2, R?.1, R?.1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: now also U?.2 (-)
- net at C?.1, JP?.2 (B), R?.1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: now also U?.1
- net at C?.1, R?.2, R?.2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: now also U?.2 (-)
- net at C?.2, C?.2, C?.2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: now also U?.1
- net at C?.2, JP5.2 (B), JP7.1 (A): now also U?.4 (V-)
- net at R?.1, R?.2: now also U?.6 (-)
- net at JP?.1 (A), JP?.1 (A): now also U?.5 (Ref)
- net at R1.1, R?.1, R?.2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: now also U?.6
- net at C?.1, R?.2: now also U?.5 (+)
- net at C?.1, JP3.1 (A), JP9.2 (B): now also U?.8 (V+)
- new net: U?.6 (-), U?.7
- no-connect marks 0 -> 2
Other:
- moved on the sheet: C?, JP3, JP5, JP7, JP9, JP?, R1, R?, U?A, U?B, U?C, U?D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

Commit message: quality of life changes plus wiring plus buffering plus value changes
Parts:
- added R? (x4): 10k, symbol Device:R
Connections:
- net +1.65VA: now also U?.7, R?.2, R?.2
- net +3.3VA: now also R?.2
- net GND: now also R?.1; no longer U?.5 (+)
- net at U?.6 (-): now also R?.1, R?.1; no longer U?.7
- new net: R?.1, R?.2, U?.5 (+)
Other:
- moved on the sheet: U?B

Commit message: footprints and minor
Parts:
- gave numbers to parts that had none: 42
- renumbered JP7 to JP11, JP5 to JP12, JP9 to JP8, JP3 to JP9, R1 to R27, R3 to R29

Commit message: minor
Parts:
- added C? (x2): 100n, symbol Device:C
- added JP?: SolderJumper_2_Open, Jumper:SolderJumper-2_P1.3mm_Open_RoundedPad1.0x1.5mm, symbol Jumper:SolderJumper_2_Open
Connections:
- net +18V: now also C?.2
- net -18V: now also C?.2
- net GND: now also C?.1, C?.1
Other:
- note added: "unity gain"
- note removed: "Only for voltage amplification"
- note removed: "Optional AC coupling For DC bias"
- moved on the sheet: C28, C29, C30, C31, C32, C33, C34, C35, C36, C37, C38, JP10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
