File: PCB/Main Board/Power.kicad_sch (KiCad schematic)
At the start: 9 parts, among them J1 Conn_01x03_Pin, U4 ${SIM.PARAMS}, U5 MIC5205-3.6YM5

Commit message: Signal
Connections:
- net +1V8 renamed +1.65V
Changed lines of the file:
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@@
-	)
-	(junction
-		(at 152.4 114.3)
-		(diameter 0)
-		(color 0 0 0 0)
 	)
 	(junction
@@
 			(width 0)
 			(type default)
+		)
+	)
+	(global_label "-1.65V"
+		(shape input)
+		(at 139.7 143.51 180)
+		(fields_autoplaced yes)
+		(effects
+			(font
+				(size 1.27 1.27)
+			)
+			(justify right)
+		)
+		(property "Intersheetrefs" "${INTERSHEET_REFS}"
+			(at 129.8205 143.51 0)
+			(effects
+				(font
+					(size 1.27 1.27)
+				)
+				(justify right)
+				(hide yes)
+			)
+		)
+	)
+	(global_label "+1.65V"
+		(shape input)
+		(at 152.4 114.3 0)
+		(fields_autoplaced yes)
+		(effects
+			(font
+				(size 1.27 1.27)
+			)
+			(justify left)
+		)
+		(property "Intersheetrefs" "${INTERSHEET_REFS}"
+			(at 162.2795 114.3 0)
+			(effects
+				(font
+					(size 1.27 1.27)
+				)
+				(justify left)
+				(hide yes)
+			)
 		)
 	)
@@
 					(unit 1)
 				)
-			)
-		)
-	)
-	(symbol
-		(lib_id "power:+1V8")
-		(at 152.4 114.3 270)
-		(unit 1)
-		(exclude_from_sim no)
-		(in_bom yes)
-		(on_board yes)
-		(dnp no)
-		(fields_autoplaced yes)
-		(property "Reference" "#PWR0101"
-			(at 148.59 114.3 0)
-			(effects
-				(font
-					(size 1.27 1.27)
-				)
-				(hide yes)
-			)
-		)
-		(property "Value" "+1V8"
-			(at 156.21 114.2999 90)
-			(effects
-				(font
-					(size 1.27 1.27)
-				)
-				(justify left)
-			)
-		)
-		(property "Footprint" ""
-			(at 152.4 114.3 0)
-			(effects
-				(font
-					(size 1.27 1.27)
-				)
-				(hide yes)
-			)
-		)
-		(property "Datasheet" ""
-			(at 152.4 114.3 0)
-			(effects
-				(font
-					(size 1.27 1.27)
-				)
-				(hide yes)
-			)
-		)
-		(property "Description" "Power symbol creates a global label with name \"+1V8\""
-			(at 152.4 114.3 0)
-			(effects
-				(font
-					(size 1.27 1.27)
-				)
-				(hide yes)
-			)
-		)
-		(pin "1"
-		)
-		(instances
-			(project "Main Board"
-				(path "/20aae4b7-3fb8-4924-82e8-1e7a29a313f8/19c51356-5fe8-4a9f-9623-d1f705fed6f9"
-					(reference "#PWR0101")
-					(unit 1)
-				)

Commit message: :anguished:
Parts:
- added R? (x2): 100k, symbol Device:R
- added U?: ${SIM.PARAMS}, symbol Simulation_SPICE:OPAMP
- U5: value MIC5205-3.6YM5 -> MIC5205-3.3YM5
Connections:
- net GND: now also U?.1 (+)
- net +1.65V renamed +1.65VA
- net +1.65VA: now also R?.1
- net +15V renamed +18V
- net +3V3 renamed +3.3V
- net -15V renamed -18V
- new net: R?.1, R?.2, U?.2 (-)
- new net -1.65VA: R?.2, U?.5

Commit message: AAAAAA
Parts:
- removed R? (x2): 100k, symbol Device:R
- removed U?: ${SIM.PARAMS}, symbol Simulation_SPICE:OPAMP

Commit message: minor: pwr, stm, filters
Parts:
- added FB?: FerriteBead, symbol Device:FerriteBead
Connections:
- net +3.3V: now also FB?.2; no longer R5.1
- new net +3.3VA: FB?.1, R5.1
Other:
- moved on the sheet: R5, R6
Changed lines of the file:
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@@
 	)
 	(junction
-		(at 114.3 114.3)
+		(at 114.3 116.84)
 		(diameter 0)
 		(color 0 0 0 0)
@@
 	(wire
 		(pts
-			(xy 114.3 101.6) (xy 114.3 104.14)
+			(xy 114.3 104.14) (xy 114.3 106.68)
 		)
 		(stroke
@@
 	(wire
 		(pts
-			(xy 114.3 114.3) (xy 120.65 114.3)
+			(xy 114.3 116.84) (xy 132.08 116.84)
 		)
 		(stroke
@@
 	(wire
 		(pts
-			(xy 120.65 116.84) (xy 132.08 116.84)
-		)
-		(stroke
-			(width 0)
-			(type default)
-		)
-	)
-	(wire
-		(pts
 			(xy 120.65 60.96) (xy 114.3 60.96)
 		)
@@
 	(wire
 		(pts
+			(xy 154.94 114.3) (xy 152.4 114.3)
+		)
+		(stroke
+			(width 0)
+			(type default)
+		)
+	)
+	(wire
+		(pts
 			(xy 120.65 55.88) (xy 120.65 60.96)
 		)
@@
 	(wire
 		(pts
-			(xy 114.3 124.46) (xy 114.3 127)
+			(xy 114.3 127) (xy 114.3 129.54)
 		)
 		(stroke
@@
 	(wire
 		(pts
-			(xy 120.65 114.3) (xy 120.65 116.84)
-		)
-		(stroke
-			(width 0)
-			(type default)
-		)
-	)
-	(wire
-		(pts
 			(xy 114.3 63.5) (xy 127 63.5)
 		)
@@
 	(wire
 		(pts
-			(xy 114.3 111.76) (xy 114.3 114.3)
+			(xy 114.3 114.3) (xy 114.3 116.84)
 		)
 		(stroke
@@
 	(wire
 		(pts
-			(xy 114.3 114.3) (xy 114.3 116.84)
+			(xy 114.3 116.84) (xy 114.3 119.38)
 		)
 		(stroke
@@
 	)
 	(symbol
+		(lib_id "Device:FerriteBead")
+		(at 181.61 88.9 90)
+		(unit 1)
+		(exclude_from_sim no)
+		(in_bom yes)
+		(on_board yes)
+		(dnp no)
+		(fields_autoplaced yes)
+		(property "Reference" "FB?"
+			(at 181.5592 81.28 90)
+			(effects
+				(font
+					(size 1.27 1.27)
+				)
+			)
+		)
+		(property "Value" "FerriteBead"
+			(at 181.5592 83.82 90)
+			(effects
+				(font
+					(size 1.27 1.27)
+				)
+			)
+		)
+		(property "Footprint" ""
+			(at 181.61 90.678 90)
+			(effects
+				(font
+					(size 1.27 1.27)
+				)
+				(hide yes)
+			)
+		)
+		(property "Datasheet" "~"
+			(at 181.61 88.9 0)
+			(effects
+				(font
+					(size 1.27 1.27)
+				)
+				(hide yes)
+			)
+		)
+		(property "Description" "Ferrite bead"
+			(at 181.61 88.9 0)
+			(effects
+				(font
+					(size 1.27 1.27)
+				)
+				(hide yes)
+			)
+		)
+		(pin "1"
+		)
+		(pin "2"
+		)
+		(instances
+			(project ""
+				(path "/20aae4b7-3fb8-4924-82e8-1e7a29a313f8/19c51356-5fe8-4a9f-9623-d1f705fed6f9"
+					(reference "FB?")
+					(unit 1)
+				)
+			)
+		)
+	)
+	(symbol
 		(lib_id "power:+3.3VA")
-		(at 114.3 101.6 0)
+		(at 114.3 104.14 0)
 		(unit 1)
 		(exclude_from_sim no)
@@
 		(fields_autoplaced yes)
 		(property "Reference" "#PWR0905"
-			(at 114.3 105.41 0)
+			(at 114.3 107.95 0)
 			(effects
 				(font
@@
 		)
 		(property "Value" "+3.3VA"
-			(at 114.3 96.52 0)
-			(effects
-				(font
-					(size 1.27 1.27)
-				)
-			)
-		)
-		(property "Footprint" ""
-			(at 114.3 101.6 0)
+			(at 114.3 99.06 0)
+			(effects
+				(font
+					(size 1.27 1.27)
+				)
+			)
+		)
+		(property "Footprint" ""
+			(at 114.3 104.14 0)
 			(effects
 				(font
@@
 		)
 		(property "Datasheet" ""
-			(at 114.3 101.6 0)
+			(at 114.3 104.14 0)
 			(effects
 				(font
@@
 		)
 		(property "Description" "Power symbol creates a global label with name \"+3.3VA\""
-			(at 114.3 101.6 0)
+			(at 114.3 104.14 0)
 			(effects
 				(font
@@
 	(symbol
 		(lib_id "More_power:+1.65VA")
-		(at 152.4 114.3 270)
+		(at 154.94 114.3 270)
 		(unit 1)
 		(exclude_from_sim no)
@@
 		(fields_autoplaced yes)
 		(property "Reference" "#PWR0909"
-			(at 148.59 114.3 0)
+			(at 151.13 114.3 0)
 			(effects
 				(font
@@
 		)
 		(property "Value" "+1.65VA"
-			(at 156.21 114.2999 90)
+			(at 158.75 114.2999 90)
 			(effects
 				(font
@@
 		)
 		(property "Footprint" ""
-			(at 152.4 114.3 0)
+			(at 154.94 114.3 0)
 			(effects
 				(font
@@
 		)
 		(property "Datasheet" ""
-			(at 152.4 114.3 0)
+			(at 154.94 114.3 0)
 			(effects
 				(font
@@
 		)
 		(property "Description" "Power symbol creates a global label with name \"+1.65VA\""
-			(at 152.4 114.3 0)
+			(at 154.94 114.3 0)
 			(effects
 				(font
@@
 	(symbol
 		(lib_id "Device:R")
-		(at 114.3 107.95 0)
+		(at 114.3 110.49 0)
 		(unit 1)
 		(exclude_from_sim no)
@@
 		(fields_autoplaced yes)
 		(property "Reference" "R5"
-			(at 116.84 106.6799 0)
+			(at 116.84 109.2199 0)
 			(effects
 				(font
@@
 		)
 		(property "Value" "100k"
-			(at 116.84 109.2199 0)
+			(at 116.84 111.7599 0)
 			(effects
 				(font
@@
 		)
 		(property "Footprint" ""
-			(at 112.522 107.95 90)
+			(at 112.522 110.49 90)
 			(effects
 				(font
@@
 		)
 		(property "Datasheet" "~"
-			(at 114.3 107.95 0)
+			(at 114.3 110.49 0)
 			(effects
 				(font
@@
 		)
 		(property "Description" "Resistor"
-			(at 114.3 107.95 0)
+			(at 114.3 110.49 0)
 			(effects
 				(font
@@
 	(symbol
 		(lib_id "power:+3.3V")
-		(at 177.8 88.9 270)
+		(at 185.42 88.9 270)
 		(unit 1)
 		(exclude_from_sim no)
@@
 		(fields_autoplaced yes)
 		(property "Reference" "#PWR0907"
-			(at 173.99 88.9 0)
+			(at 181.61 88.9 0)
 			(effects
 				(font
@@
 		)
 		(property "Value" "+3.3V"
-			(at 181.61 88.8999 90)
+			(at 189.23 88.8999 90)
 			(effects
 				(font
@@
 		)
 		(property "Footprint" ""
-			(at 177.8 88.9 0)
+			(at 185.42 88.9 0)
 			(effects
 				(font
@@
 		)
 		(property "Datasheet" ""
-			(at 177.8 88.9 0)
+			(at 185.42 88.9 0)
 			(effects
 				(font
@@
 		)
 		(property "Description" "Power symbol creates a global label with name \"+3.3V\""
-			(at 177.8 88.9 0)
+			(at 185.42 88.9 0)
 			(effects
 				(font
@@
 	(symbol
 		(lib_id "power:GND")
-		(at 114.3 127 0)
+		(at 114.3 129.54 0)
 		(unit 1)
 		(exclude_from_sim no)
@@
 		(fields_autoplaced yes)
 		(property "Reference" "#PWR02"
-			(at 114.3 133.35 0)
+			(at 114.3 135.89 0)
 			(effects
 				(font
@@
 		)
 		(property "Value" "GND"
-			(at 114.3 132.08 0)
-			(effects
-				(font
-					(size 1.27 1.27)
-				)
-			)
-		)
-		(property "Footprint" ""
-			(at 114.3 127 0)
+			(at 114.3 134.62 0)
+			(effects
+				(font
+					(size 1.27 1.27)
+				)
+			)
+		)
+		(property "Footprint" ""
+			(at 114.3 129.54 0)
 			(effects
 				(font
@@
 		)
 		(property "Datasheet" ""
-			(at 114.3 127 0)
+			(at 114.3 129.54 0)
 			(effects
 				(font
@@
 		)
 		(property "Description" "Power symbol creates a global label with name \"GND\" , ground"
-			(at 114.3 127 0)
+			(at 114.3 129.54 0)
 			(effects
 				(font
@@
 	(symbol
 		(lib_id "Device:R")
-		(at 114.3 120.65 0)
+		(at 114.3 123.19 0)
 		(unit 1)
 		(exclude_from_sim no)
@@
 		(fields_autoplaced yes)
 		(property "Reference" "R6"
-			(at 116.84 119.3799 0)
+			(at 116.84 121.9199 0)
 			(effects
 				(font
@@
 		)
 		(property "Value" "100k"
-			(at 116.84 121.9199 0)
+			(at 116.84 124.4599 0)
 			(effects
 				(font
@@
 		)
 		(property "Footprint" ""
-			(at 112.522 120.65 90)
+			(at 112.522 123.19 90)
 			(effects
 				(font
@@
 		)
 		(property "Datasheet" "~"
-			(at 114.3 120.65 0)
+			(at 114.3 123.19 0)
 			(effects
 				(font
@@
 		)
 		(property "Description" "Resistor"
-			(at 114.3 120.65 0)
-			(effects
-				(font
+			(at 114.3 123.19 0)
+			(effects
+				(font

Commit message: power supply
Parts:
- removed C3: 220p, symbol Device:C
- removed U5: MIC5205-3.3YM5, Package_TO_SOT_SMD:SOT-23-5, symbol Regulator_Linear:MIC5205-3.6YM5
- added C10, C11, C12, C5, C6, C7, C8, C9: 1u, symbol Device:C
- added C3: 220µ, symbol Device:C_Polarized
- added R10, R12, R9: 1k, symbol Device:R
- added R11, R13, R8: 10k, symbol Device:R_Variable
- added R14: 240, symbol Device:R
- added R15: 5k, symbol Device:R_Variable
- added R7: 5k, symbol Device:R
- added U2, U6, U7: LM317L_SOT-89, Package_TO_SOT_SMD:SOT-89-3, symbol Regulator_Linear:LM317L_SOT-89
- added U3: LM337_SOT223, Package_TO_SOT_SMD:SOT-223-3_TabPin2, symbol Regulator_Linear:LM337_SOT223
- C4: value 2.2µ -> 220µ
- R5, R6: value 100k -> 10k
Connections:
- net +1.65VA: now also R7.2; no longer U4.2 (-)
- net +18V: now also C6.1, R9.1, U2.2 (VO); no longer C1.1, J1.1 (Pin_1)
- net +3.3V: now also C10.1, R12.1, U6.2 (VO); no longer C4.1
- net -18V: now also C12.1, R14.1, U3.3 (VO); no longer C2.2, J1.3 (Pin_3)
- net GND: now also C4.1, C10.2, C11.2, C12.2, C3.2, C5.2, C6.2, C7.2, C8.2, C9.2, R11.2, R13.2, R15.1, R8.2; no longer C4.2
- new net: R7.1, U4.2 (-)
- new net: R10.2, R11.1, U7.1 (ADJ)
- new net: R14.2, R15.2, U3.1 (ADJ)
- new net: R12.2, R13.1, U6.1 (ADJ)
- new net: R8.1, R9.2, U2.1 (ADJ)
- new net +12V: C8.1, R10.1, U7.2 (VO)
- new net VIN+: C1.1, C3.1, C5.1, C7.1, C9.1, J1.1 (Pin_1), U2.3 (VI), U6.3 (VI), U7.3 (VI)
- new net VIN-: C11.1, C2.2, C4.2, J1.3 (Pin_3), U3.2 (VI)
Other:
- note added: "+20V to -20V"
- moved on the sheet: C1, C2, FB?, J1, R5, R6, U4
