File: PCB/Main Board/Power.kicad_sch (KiCad schematic)
At the start: 30 parts, among them J1 Conn_01x03_Pin, U2 LM317L_SOT-89, U3 LM337_SOT223, U4 ${SIM.PARAMS}, U6 LM317L_SOT-89, U7 LM317L_SOT-89

Commit message: Amplifier Switch
Parts:
- removed U4: ${SIM.PARAMS}, symbol Simulation_SPICE:OPAMP
- added C? (x2): 100n, symbol Device:C
- added U? (x3): OPA2197xD, Package_SO:SOIC-8_3.9x4.9mm_P1.27mm, symbol Amplifier_Operational:OPA2197xD
Connections:
- net +1.65VA: now also U?.1
- net GND: now also C?.1, C?.2, U?.5 (+)
- net at R7.1: now also U?.2 (-)
- net at R5.2, R6.1: now also U?.3 (+)
- new net: C?.2, U?.4 (V-)
- new net: C?.1, U?.8 (V+)
- new net: U?.6 (-), U?.7
Other:
- moved on the sheet: R7

Commit message: quality of life changes plus wiring plus buffering plus value changes
Parts:
- removed C? (x2): 100n, symbol Device:C
- removed R5, R6: 10k, symbol Device:R
- removed R7: 5k, symbol Device:R
- removed U? (x3): OPA2197xD, Package_SO:SOIC-8_3.9x4.9mm_P1.27mm, symbol Amplifier_Operational:OPA2197xD
- added TP? (x3): TestPoint, TestPoint:TestPoint_THTPad_4.0x4.0mm_Drill2.0mm, symbol Connector:TestPoint
Connections:
- net GND: now also TP?.1
- net VIN+: now also TP?.1
- net VIN-: now also TP?.1
Other:
- moved on the sheet: C1, C2, C3, C4, J1

Commit message: footprints and minor
Parts:
- added D? (x2): D_Schottky, symbol Device:D_Schottky
- gave numbers to parts that had none: 4
- renumbered C5 to C70, C6 to C71, C1 to C72, C3 to C73, C2 to C74, C4 to C75, C7 to C76, C8 to C77, C9 to C78, C10 to C79, C11 to C80, C12 to C81, J1 to J6, R15 to R100, R14 to R101, R9 to R94, R8 to R95, R10 to R96, R11 to R97, R12 to R98, R13 to R99, U2 to U23, U7 to U24, U6 to U25, U3 to U26
Connections:
- net VIN+: now also D?.1 (K); no longer J6.1 (Pin_1), TP1.1
- net VIN-: now also D?.2 (A); no longer J6.3 (Pin_3), TP3.1
- new net: D?.2 (A), J6.1 (Pin_1), TP1.1
- new net: D?.1 (K), J6.3 (Pin_3), TP3.1
Other:
- note added: "do we need an emi filter here?"
- moved on the sheet: C70, C71, C72, C73, C74, C75, C76, C77, C78, C79, C80, C81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

Commit message: minor
Parts:
- gave numbers to parts that had none: 2
Changed lines of the file:
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@@
 		(dnp no)
 		(fields_autoplaced yes)
-		(property "Reference" "D?"
+		(property "Reference" "D5"
 			(at 61.2775 39.37 0)
 			(effects
@@
 			(project ""
 				(path "/20aae4b7-3fb8-4924-82e8-1e7a29a313f8/19c51356-5fe8-4a9f-9623-d1f705fed6f9"
-					(reference "D?")
+					(reference "D5")
 					(unit 1)
 				)
@@
 		(dnp no)
 		(fields_autoplaced yes)
-		(property "Reference" "D?"
+		(property "Reference" "D6"
 			(at 60.6425 62.23 0)
 			(effects
@@
 			(project "Main Board"
 				(path "/20aae4b7-3fb8-4924-82e8-1e7a29a313f8/19c51356-5fe8-4a9f-9623-d1f705fed6f9"
-					(reference "D?")
-					(unit 1)
-				)
+					(reference "D6")
+					(unit 1)
+				)

Commit message: footprints and stm wiring
Parts:
- added C?: 220µ, symbol Device:C_Polarized
- added D?: LED, symbol Device:LED
- added JP?: SolderJumper_3_Open, symbol Jumper:SolderJumper_3_Open
- added R?: 220, symbol Device:R
Connections:
- net +12V: now also JP?.2 (C); no longer C77.1, R96.1, U24.2 (VO)
- net +3.3V: now also R?.1
- net GND: now also C?.2, D?.1 (K)
- net VIN+: now also JP?.3 (B)
- new net: D?.2 (A), R?.2
- new net: C77.1, C?.1, JP?.1 (A), R96.1, U24.2 (VO)
Other:
- moved on the sheet: C72, C73, C74, C75, D5, D6, FB1, J6, TP1, TP2, TP3

Commit message: relays and layout begin
Parts:
- removed C72, C74: 22µ, symbol Device:C_Polarized
- removed C73, C75, C?: 220µ, symbol Device:C_Polarized
- removed JP?: SolderJumper_3_Open, symbol Jumper:SolderJumper_3_Open
- removed TP1, TP2, TP3: TestPoint, TestPoint:TestPoint_THTPad_4.0x4.0mm_Drill2.0mm, symbol Connector:TestPoint
- removed U23, U24, U25: LM317L_SOT-89, Package_TO_SOT_SMD:SOT-89-3, symbol Regulator_Linear:LM317L_SOT-89
- added C76, C77, C81, C82: 22u, Capacitor_SMD:C_1210_3225Metric, symbol Device:C
- added D7: SBR3U60P1-7, Diode_SMD:D_PowerDI-123, symbol Device:D_Schottky
- added J7: Screw_Terminal_01x03, TerminalBlock_4Ucon:TerminalBlock_4Ucon_1x03_P3.50mm_Horizontal, symbol Connector:Screw_Terminal_01x03
- added U23, U24, U25: LM317_SOT-223, Package_TO_SOT_SMD:SOT-223-3_TabPin2, symbol Regulator_Linear:LM317_SOT-223
- C74: renamed from C70; footprint (none) -> Capacitor_SMD:C_0805_2012Metric
- C75: renamed from C71; footprint (none) -> Capacitor_SMD:C_0805_2012Metric
- C78: renamed from C76; footprint (none) -> Capacitor_SMD:C_0805_2012Metric
- C79: renamed from C77; value 1u -> 220u; footprint (none) -> Capacitor_SMD:C_0805_2012Metric
- C83: renamed from C78; footprint (none) -> Capacitor_SMD:C_0805_2012Metric
- C84: renamed from C79; footprint (none) -> Capacitor_SMD:C_0805_2012Metric
- C85: renamed from C80; footprint (none) -> Capacitor_SMD:C_0805_2012Metric
- C86: renamed from C81; footprint (none) -> Capacitor_SMD:C_0805_2012Metric
- D5, D6: value D_Schottky -> SBR3U60P1-7; footprint (none) -> Diode_SMD:D_PowerDI-123; Height (none) -> 1; Manufacturer_Name (none) -> Diodes Incorporated; Manufacturer_Part_Number (none) -> SBR3U60P1-7; Mouser Part Number (none) -> 621-SBR3U60P1-7; Mouser Price/Stock (none) -> https://www.mouser.co.uk/ProductDetail/Diodes-Incorporated/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
- D8: renamed from D?; footprint (none) -> LED_SMD:LED_0805_2012Metric
- FB1: footprint (none) -> Inductor_SMD:L_0805_2012Metric
- J6: footprint (none) -> Connector_PinHeader_2.00mm:PinHeader_1x03_P2.00mm_Vertical
- R100: renamed from R99; footprint (none) -> Potentiometer_SMD:Potentiometer_Bourns_3214W_Vertical
- R101: renamed from R100; footprint (none) -> Potentiometer_SMD:Potentiometer_Bourns_3214W_Vertical
- R102: renamed from R101; footprint (none) -> Resistor_SMD:R_0805_2012Metric
- R94, R96, R98: footprint (none) -> Resistor_SMD:R_0805_2012Metric
- R95, R97: footprint (none) -> Potentiometer_SMD:Potentiometer_Bourns_3214W_Vertical
- R99: renamed from R?; footprint (none) -> Resistor_SMD:R_0805_2012Metric
Connections:
- net +12V: now also C79.1, D5.2 (A), R96.1, U24.2 (VO)
- net +18V: now also U23.2 (VO)
- net +3.3V: now also U25.2 (VO)
- net GND: now also C76.1, C77.1, C81.2, C82.2, J7.2 (Pin_2)
- net VIN+: now also D6.1 (K), C76.2, C77.2, U23.3 (VI), U24.3 (VI), U25.3 (VI)
- net VIN-: now also C81.1, C82.1, D7.2 (A); no longer D6.2 (A)
- net at J6.1 (Pin_1): now also D6.2 (A), J7.1 (Pin_1); no longer D5.2 (A)
- net at R96.2, R97.1: now also U24.1 (ADJ)
- net at R100.1, R98.2: now also U25.1 (ADJ)
- net at J6.3 (Pin_3): now also D7.1 (K), J7.3 (Pin_3); no longer D6.1 (K)
- net at R94.2, R95.1: now also U23.1 (ADJ)
Other:
- note added: "if the bourns pots are too expensive then can bridge with 0805 its easily"
- moved on the sheet: C78, C79, C83, C84, C85, C86, D8, FB1, J6, R100, R101, R102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

Commit message: minor and layout
Other:
- note added: "do we need an emi filter here? (yes but i removed it its not that important)"
- note removed: "do we need an emi filter here?"
- moved on the sheet: C74, C75, C78, C79, C83, C84, C85, C86, D5, D8, FB1, R100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
