File: PCB/Main Board/Power.kicad_sch (KiCad schematic)
At the start: 32 parts, among them J6 Conn_01x03_Pin, J7 Screw_Terminal_01x03, U23 LM317_SOT-223, U24 LM317_SOT-223, U25 LM317_SOT-223, U26 LM337_SOT223

Commit message: :ghost:
Parts:
- renumbered C76 to C1301, C81 to C1302, C77 to C1303, C82 to C1304, C74 to C1305, C78 to C1306, C83 to C1307, C85 to C1308, C75 to C1309, C79 to C1310, C84 to C1311, C86 to C1312, D6 to D1301, D7 to D1302, D5 to D1303, D8 to D1304, FB1 to FB1301, J6 to J1301, J7 to J1302, R95 to R1301, R97 to R1302, R100 to R1303, R101 to R1304, R94 to R1305, R96 to R1306, R98 to R1307, R102 to R1308, R99 to R1309, U23 to U1301, U24 to U1302, U25 to U1303, U26 to U1304

Commit message: :-1:
Parts:
- renumbered C1301 to C801, C1302 to C802, C1303 to C803, C1304 to C804, C1305 to C805, C1306 to C806, C1307 to C807, C1308 to C808, C1309 to C809, C1310 to C810, C1311 to C811, C1312 to C812, D1301 to D801, D1302 to D802, D1303 to D803, D1304 to D804, FB1301 to FB801, J1301 to J801, J1302 to J802, R1301 to R801, R1302 to R802, R1303 to R803, R1304 to R804, R1305 to R805, R1306 to R806, R1307 to R807, R1308 to R808, R1309 to R809, U1301 to U801, U1302 to U802, U1303 to U803, U1304 to U804

Commit message: sorry i fell asleep b4 layout
Parts:
- renumbered C805 to C801, C809 to C802, C806 to C803, C810 to C804, C801 to C805, C803 to C806, C802 to C807, C804 to C808, C807 to C809, C811 to C810, C808 to C811, D803 to D801, D801 to D802, D802 to D803, J802 to J801, J801 to J802, R805 to R801, R801 to R802, R806 to R803, R802 to R804, R807 to R805, R809 to R806, R803 to R807, R804 to R808, R808 to R809
Other:
- note removed: "do we need an emi filter here? (yes but i removed it its not that important)"
- note removed: "if the bourns pots are too expensive then can bridge with 0805 its easily"

Commit message: HI
Parts:
- renumbered C805 to C801, C807 to C802, C806 to C803, C808 to C804, C801 to C805, C803 to C806, C809 to C807, C811 to C808, C802 to C809, C804 to C810, C810 to C811, D802 to D801, D803 to D802, D801 to D803, J802 to J801, J801 to J802, R802 to R801, R804 to R802, R807 to R803, R808 to R804, R801 to R805, R803 to R806, R805 to R807, R809 to R808, R806 to R809

Commit message: please be nice
Parts:
- removed R801, R802, R803: 10k, Potentiometer_SMD:Potentiometer_Bourns_3214W_Vertical, symbol Device:R_Variable
- removed R804: 5k, Potentiometer_SMD:Potentiometer_Bourns_3214W_Vertical, symbol Device:R_Variable
- added RV801, RV802, RV803: 10k, Potentiometer_Bourns_3214W_Vertical, symbol Device:R_Potentiometer
- added RV804: 5k, Potentiometer_Bourns_3214W_Vertical, symbol Device:R_Potentiometer
- J802: renamed from J801; footprint Connector_PinHeader_2.00mm:PinHeader_1x03_P2.00mm_Vertical -> Connector_PinHeader_2.54mm:PinHeader_1x03_P2.54mm_Vertical
- renumbered C805 to C801, C809 to C802, C806 to C803, C810 to C804, C801 to C805, C803 to C806, C802 to C807, C804 to C808, C807 to C809, C811 to C810, C808 to C811, D803 to D801, D801 to D802, D802 to D803, J802 to J801, R805 to R801, R806 to R802, R807 to R803, R809 to R804, R808 to R805
Connections:
- net GND: now also RV801.3, RV802.3, RV803.3, RV804.3
- net at R802.2, U802.1 (ADJ): now also RV802.2
- net at R805.2, U804.1 (ADJ): now also RV804.2
- net at R803.2, U803.1 (ADJ): now also RV803.2
- net at R801.2, U801.1 (ADJ): now also RV801.2
- no-connect marks 0 -> 4

Commit message: Final Schematic
Parts:
- renumbered C805 to C60, C807 to C61, C806 to C62, C808 to C63, C801 to C64, C803 to C65, C809 to C66, C811 to C67, C802 to C68, C804 to C69, C810 to C70, C812 to C71, D802 to D6, D803 to D7, D801 to D8, D804 to D9, FB801 to FB1, J802 to J8, J801 to J9, R801 to R90, R802 to R91, R803 to R92, R805 to R93, R804 to R94, RV801 to RV1, RV802 to RV2, RV803 to RV3, RV804 to RV4, U801 to U20, U802 to U21, U803 to U22, U804 to U23
Other:
- title: (none) -> Power Supply

Commit message: minor cleanup from the party
Parts:
- renumbered C64 to C801, C68 to C802, C65 to C803, C69 to C804, C60 to C805, C62 to C806, C61 to C807, C63 to C808, C66 to C809, C70 to C810, C67 to C811, C71 to C812, D8 to D801, D6 to D802, D7 to D803, D9 to D804, FB1 to FB801, J9 to J801, J8 to J802, R90 to R801, R91 to R802, R92 to R803, R94 to R804, R93 to R805, RV1 to RV801, RV2 to RV802, RV3 to RV803, RV4 to RV804, U20 to U801, U21 to U802, U22 to U803, U23 to U804

Commit message: footprints and tps
Parts:
- added TP?: -18V, TestPoint:TestPoint_Pad_2.0x2.0mm, symbol Connector:TestPoint
- added TP?: +18V, TestPoint:TestPoint_Pad_2.0x2.0mm, symbol Connector:TestPoint
- added TP?: +3.3VA, TestPoint:TestPoint_Pad_2.0x2.0mm, symbol Connector:TestPoint
- added TP?: +12V, TestPoint:TestPoint_Pad_2.0x2.0mm, symbol Connector:TestPoint
- added TP?: +3.3V, TestPoint:TestPoint_Pad_2.0x2.0mm, symbol Connector:TestPoint
- RV801, RV802, RV803, RV804: footprint Potentiometer_Bourns_3214W_Vertical -> Potentiometer_SMD:Potentiometer_Bourns_TC33X_Vertical
Connections:
- net +12V: now also TP?.1
- net +18V: now also TP?.1
- net +3.3V: now also TP?.1
- net +3.3VA: now also TP?.1
- net -18V: now also TP?.1
