File: PCB/Main Board/Resistors.kicad_sch (KiCad schematic)
At the start: 13 parts

Commit message: Panik
Parts:
- removed K?: Fujitsu_FTR-LYAA005x, Relay_THT:Relay_SPST-NO_Fujitsu_FTR-LYAA005x_FormA_Vertical, symbol Relay:Fujitsu_FTR-LYAA005x
- added K? (x4): COTO_3602_Split, Relay_THT:Relay_DPDT_Omron_G5V-2, symbol Relay:COTO_3602_Split
- added U? (x2): DG411xY, Package_SO:SOIC-16_3.9x9.9mm_P1.27mm, symbol Analog_Switch:DG411xY
Connections:
- net In: now also JP?.1 (A), R?.1, K?.14
- net Out: now also R?.2, R?.2
- net at JP?.2 (B): now also R?.1, K?.13, K?.14
- net at R?.1: now also K?.13, U?.7
- net at R?.1: now also K?.13, K?.14
Other:
- note added: "Cut if populating"
- note added: "Optional For higher ranges"
- moved on the sheet: JP?, R?

Commit message: Paniking further
Parts:
- removed JP?: SolderJumper_2_Bridged, Jumper:SolderJumper-2_P1.3mm_Bridged_RoundedPad1.0x1.5mm, symbol Jumper:SolderJumper_2_Bridged
- removed K? (x4): COTO_3602_Split, Relay_THT:Relay_DPDT_Omron_G5V-2, symbol Relay:COTO_3602_Split
- removed R?: 30k, symbol Device:R
- removed R?: 3k, symbol Device:R
- removed R?: 300, symbol Device:R
- removed R?: 30, symbol Device:R
- removed U? (x2): DG411xY, Package_SO:SOIC-16_3.9x9.9mm_P1.27mm, symbol Analog_Switch:DG411xY
- added SW1, SW2: SW_DPDT_x2, symbol Switch:SW_DPDT_x2
- added SW10, SW11, SW12, SW14, SW16, SW17, SW4, SW5, SW7: SW_DIP_x01, symbol Switch:SW_DIP_x01
Connections:
- net In: now also R?.1, R?.1, R?.1, R?.1, R?.1, R?.1
- net at R?.2: now also SW7.1
- net at R?.2: now also SW14.1, SW16.1
- net at R?.2: now also SW2.2 (B)
- net at R?.2: now also SW11.1, SW12.1
- net at R?.2: now also SW5.1
- net Out: no longer names the net of R?.2
- net Out: now also SW1.2 (B); no longer R?.2
- new net: SW10.1, SW11.2, SW16.2, SW4.1, SW5.2, SW7.2
- new net Guard_{int}: SW1.1 (A), SW2.1 (A)
- new net I_{Out}: R?.2, SW1.3 (C), SW17.1, SW2.3 (C), SW4.2
- new net V_{Out}: SW10.2, SW12.2, SW14.2, SW17.2
Other:
- note removed: "Cut if populating"
- note removed: "Optional For higher ranges"
- moved on the sheet: R?

Commit message: parts selection
Parts:
- removed SW1, SW2: SW_DPDT_x2, symbol Switch:SW_DPDT_x2
- removed SW10, SW11, SW12, SW14, SW16, SW17, SW4, SW5, SW7: SW_DIP_x01, symbol Switch:SW_DIP_x01
- added K? (x4): Relay_SPST-NO, symbol Relay:Relay_SPST-NO
- added U? (x3): DG419LDY, Package_SO:SOIC-8_3.9x4.9mm_P1.27mm, symbol Analog_Switch:DG419LDY
Connections:
- net at R?.2: now also U?.1 (x2)
- net at R?.2: now also K?.14 (x4)
- net I_{Out} renamed I_OUT
- net I_OUT: now also K?.13, K?.13, K?.13, K?.13, U?.8, U?.8
- net In renamed IN
- new net GND: K?.A2, K?.A2, K?.A2, K?.A2
- new net GUARD: U?.2, U?.2
- new net SELECT_10: K?.A1
- new net SELECT_100: K?.A1
- new net SELECT_100k: U?.6
- new net SELECT_10k: K?.A1
- new net SELECT_1k: K?.A1
- new net SELECT_432k: U?.6
Other:
- note added: "have selected suitable/cheap relay and analogue SPDT switches we dont need the other switches in this config i think (!?)"
- moved on the sheet: R?

Commit message: :cry:
Parts:
- removed U?: DG419LDY, Package_SO:SOIC-8_3.9x4.9mm_P1.27mm, symbol Analog_Switch:DG419LDY
Other:
- note removed: "have selected suitable/cheap relay and analogue SPDT switches we dont need the other switches in this config i think (!?)"
- moved on the sheet: K?, R?, U?A

Commit message: 😫
Parts:
- added R10: 30, symbol Device:R
- added R7: 30k, symbol Device:R
- added R8: 3k, symbol Device:R
- added R9: 300, symbol Device:R
Connections:
- net IN: now also R10.1, R7.1, R8.1, R9.1
Other:
- moved on the sheet: K?

Commit message: minor
Parts:
- removed R10: 30, symbol Device:R
- removed R7: 30k, symbol Device:R
- removed R8: 3k, symbol Device:R
- removed R9: 300, symbol Device:R
Other:
- moved on the sheet: K?

Commit message: power supply
Connections:
- net GND renamed +12V
