File: PCB/Main Board/Resistors.kicad_sch (KiCad schematic)
At the start: 13 parts

Commit message: footprints and minor
Parts:
- removed K? (x4): Relay_SPST-NO, symbol Relay:Relay_SPST-NO
- added K3, K4, K5, K6: G2RL-1, Relay_THT:Relay_SPDT_Omron_G2RL-1, symbol Relay:G2RL-1
- gave numbers to parts that had none: 9
Connections:
- net +12V: now also K3.A2, K4.A2, K5.A2, K6.A2
- net GUARD: now also K3.12, K4.12, K5.12, K6.12
- net I_OUT: now also K3.11, K4.11, K5.11, K6.11
- net SELECT_10: now also K3.A1
- net SELECT_100: now also K4.A1
- net SELECT_10k: now also K6.A1
- net SELECT_1k: now also K5.A1
- net at R89.2: now also K5.14
- net at R87.2: now also K3.14
- net at R88.2: now also K4.14
- net at R90.2: now also K6.14
Other:
- moved on the sheet: R87

Commit message: relays and layout begin
Parts:
- removed K3, K4, K5, K6: G2RL-1, Relay_THT:Relay_SPDT_Omron_G2RL-1, symbol Relay:G2RL-1
- added K4, K5, K6, K7: AGQ200A12, AGQ200A03X, symbol AGQ200A12:AGQ200A12
- added U10: DG201, Package_SO:SOIC-16_3.9x9.9mm_P1.27mm, symbol More_symbols:DG201
- R45: renamed from R87; footprint (none) -> Resistor_SMD:R_0805_2012Metric
- R46: renamed from R88; footprint (none) -> Resistor_SMD:R_0805_2012Metric
- R47: renamed from R89; footprint (none) -> Resistor_SMD:R_0805_2012Metric
- R48: renamed from R90; footprint (none) -> Resistor_SMD:R_0805_2012Metric
- R49: renamed from R91; footprint (none) -> Resistor_SMD:R_0805_2012Metric
- R50: renamed from R92; footprint (none) -> Resistor_SMD:R_0805_2012Metric
- R51: renamed from R93; footprint (none) -> Resistor_SMD:R_0805_2012Metric
- renumbered U21 to U11, U22 to U12
Connections:
- net +12V: now also K4.1, K5.1, K6.1, K7.1
- net I_OUT: now also K4.4, K5.4, K6.4, K7.4
- net SELECT_10: now also K4.8
- net SELECT_100: now also K5.8
- net SELECT_10k: now also K7.8
- net SELECT_1k: now also K6.8
- net at R47.2: now also K6.3
- net at R46.2: now also K5.3
- net at R45.2: now also K4.3
- net at R48.2: now also K7.3
- new net +18V: U10.13 (V+)
- new net -18V: U10.4 (V-)
- new net GND: U10.5 (GND)
- no-connect marks 0 -> 16
Other:
- note added: "i did double-check it i just need a quick one-over"
- note added: "need to check the pinout of this relay"
- note added: "there is only one supply for two switches???"
- moved on the sheet: R45, R46, R47, R48, R49, R50, R51, U11A, U12A

Commit message: minor and layout
Parts:
- removed R50: 432k, Resistor_SMD:R_0805_2012Metric, symbol Device:R
- removed U10: DG201, Package_SO:SOIC-16_3.9x9.9mm_P1.27mm, symbol More_symbols:DG201
- removed U12: DG419LDY, Package_SO:SOIC-8_3.9x4.9mm_P1.27mm, symbol Analog_Switch:DG419LDY
Connections:
- net GUARD: now also K4.2, K5.2, K6.2, K7.2
- no-connect marks 16 -> 12
Other:
- moved on the sheet: K4, K5, K6, K7, R45, R46, R47, R48, R49, R51, U11A

Commit message: amplifer floorplan and relay footprint + minor
Parts:
- K4, K5, K6, K7: footprint AGQ200A03X -> AGQ200A12_footprint
Changed lines of the file:
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@@
 			)
 		)
-		(property "Footprint" "AGQ200A03X"
+		(property "Footprint" "AGQ200A12_footprint"
 			(at 147.32 134.29 0)
 			(effects
@@
 			)
 		)
-		(property "Footprint" "AGQ200A03X"
+		(property "Footprint" "AGQ200A12_footprint"
 			(at 171.45 107.62 0)
 			(effects
@@
 			)
 		)
-		(property "Footprint" "AGQ200A03X"
+		(property "Footprint" "AGQ200A12_footprint"
 			(at 96.52 181.28 0)
 			(effects
@@
 			)
 		)
-		(property "Footprint" "AGQ200A03X"
+		(property "Footprint" "AGQ200A12_footprint"
 			(at 123.19 158.42 0)
 			(effects

Commit message: :ghost:
Parts:
- renumbered K7 to K801, K6 to K802, K5 to K803, K4 to K804, R45 to R801, R46 to R802, R47 to R803, R48 to R804, R49 to R805, R51 to R806, U11 to U801
Changed lines of the file:
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@@
 		(dnp no)
 		(fields_autoplaced yes)
-		(property "Reference" "R47"
+		(property "Reference" "R803"
 			(at 41.91 88.9 90)
 			(effects
@@
 			(project "Main Board"
 				(path "/20aae4b7-3fb8-4924-82e8-1e7a29a313f8/6b7fef71-3444-4c8f-b2e2-502774ba9b51/2542314c-0b08-493b-856b-65d680d18812"
-					(reference "R47")
+					(reference "R803")
 					(unit 1)
 				)
@@
 		(on_board yes)
 		(dnp no)
-		(property "Reference" "#PWR087"
+		(property "Reference" "#PWR0801"
 			(at 88.9 107.95 0)
 			(effects
@@
 			(project "Main Board"
 				(path "/20aae4b7-3fb8-4924-82e8-1e7a29a313f8/6b7fef71-3444-4c8f-b2e2-502774ba9b51/2542314c-0b08-493b-856b-65d680d18812"
-					(reference "#PWR087")
+					(reference "#PWR0801")
 					(unit 1)
 				)
@@
 		(on_board yes)
 		(dnp no)
-		(property "Reference" "#PWR086"
+		(property "Reference" "#PWR0802"
 			(at 115.57 85.09 0)
 			(effects
@@
 			(project "Main Board"
 				(path "/20aae4b7-3fb8-4924-82e8-1e7a29a313f8/6b7fef71-3444-4c8f-b2e2-502774ba9b51/2542314c-0b08-493b-856b-65d680d18812"
-					(reference "#PWR086")
+					(reference "#PWR0802")
 					(unit 1)
 				)
@@
 		(dnp no)
 		(fields_autoplaced yes)
-		(property "Reference" "R45"
+		(property "Reference" "R801"
 			(at 40.64 38.1 90)
 			(effects
@@
 			(project "Main Board"
 				(path "/20aae4b7-3fb8-4924-82e8-1e7a29a313f8/6b7fef71-3444-4c8f-b2e2-502774ba9b51/2542314c-0b08-493b-856b-65d680d18812"
-					(reference "R45")
+					(reference "R801")
 					(unit 1)
 				)
@@
 		(dnp no)
 		(fields_autoplaced yes)
-		(property "Reference" "K5"
+		(property "Reference" "K803"
 			(at 135.89 50.8 0)
 			(effects
@@
 			(project "Main Board"
 				(path "/20aae4b7-3fb8-4924-82e8-1e7a29a313f8/6b7fef71-3444-4c8f-b2e2-502774ba9b51/2542314c-0b08-493b-856b-65d680d18812"
-					(reference "K5")
+					(reference "K803")
 					(unit 1)
 				)
@@
 		(on_board yes)
 		(dnp no)
-		(property "Reference" "#PWR084"
+		(property "Reference" "#PWR0804"
 			(at 163.83 34.29 0)
 			(effects
@@
 			(project "Main Board"
 				(path "/20aae4b7-3fb8-4924-82e8-1e7a29a313f8/6b7fef71-3444-4c8f-b2e2-502774ba9b51/2542314c-0b08-493b-856b-65d680d18812"
-					(reference "#PWR084")
+					(reference "#PWR0804")
 					(unit 1)
 				)
@@
 		(dnp no)
 		(fields_autoplaced yes)
-		(property "Reference" "K4"
+		(property "Reference" "K804"
 			(at 160.02 24.13 0)
 			(effects
@@
 			(project ""
 				(path "/20aae4b7-3fb8-4924-82e8-1e7a29a313f8/6b7fef71-3444-4c8f-b2e2-502774ba9b51/2542314c-0b08-493b-856b-65d680d18812"
-					(reference "K4")
+					(reference "K804")
 					(unit 1)
 				)
@@
 		(dnp no)
 		(fields_autoplaced yes)
-		(property "Reference" "K7"
+		(property "Reference" "K801"
 			(at 85.09 97.79 0)
 			(effects
@@
 			(project "Main Board"
 				(path "/20aae4b7-3fb8-4924-82e8-1e7a29a313f8/6b7fef71-3444-4c8f-b2e2-502774ba9b51/2542314c-0b08-493b-856b-65d680d18812"
-					(reference "K7")
+					(reference "K801")
 					(unit 1)
 				)
@@
 		(dnp no)
 		(fields_autoplaced yes)
-		(property "Reference" "R49"
+		(property "Reference" "R805"
 			(at 41.91 128.27 90)
 			(effects
@@
 			(project "Main Board"
 				(path "/20aae4b7-3fb8-4924-82e8-1e7a29a313f8/6b7fef71-3444-4c8f-b2e2-502774ba9b51/2542314c-0b08-493b-856b-65d680d18812"
-					(reference "R49")
+					(reference "R805")
 					(unit 1)
 				)
@@
 		(dnp no)
 		(fields_autoplaced yes)
-		(property "Reference" "U11"
+		(property "Reference" "U801"
 			(at 58.42 125.73 0)
 			(effects
@@
 			(project ""
 				(path "/20aae4b7-3fb8-4924-82e8-1e7a29a313f8/6b7fef71-3444-4c8f-b2e2-502774ba9b51/2542314c-0b08-493b-856b-65d680d18812"
-					(reference "U11")
+					(reference "U801")
 					(unit 1)
 				)
@@
 		(on_board yes)
 		(dnp no)
-		(property "Reference" "#PWR085"
+		(property "Reference" "#PWR0803"
 			(at 139.7 60.96 0)
 			(effects
@@
 			(project "Main Board"
 				(path "/20aae4b7-3fb8-4924-82e8-1e7a29a313f8/6b7fef71-3444-4c8f-b2e2-502774ba9b51/2542314c-0b08-493b-856b-65d680d18812"
-					(reference "#PWR085")
+					(reference "#PWR0803")
 					(unit 1)
 				)
@@
 		(dnp no)
 		(fields_autoplaced yes)
-		(property "Reference" "R46"
+		(property "Reference" "R802"
 			(at 40.64 64.77 90)
 			(effects
@@
 			(project "Main Board"
 				(path "/20aae4b7-3fb8-4924-82e8-1e7a29a313f8/6b7fef71-3444-4c8f-b2e2-502774ba9b51/2542314c-0b08-493b-856b-65d680d18812"
-					(reference "R46")
+					(reference "R802")
 					(unit 1)
 				)
@@
 		(dnp no)
 		(fields_autoplaced yes)
-		(property "Reference" "R48"
+		(property "Reference" "R804"
 			(at 41.91 111.76 90)
 			(effects
@@
 			(project "Main Board"
 				(path "/20aae4b7-3fb8-4924-82e8-1e7a29a313f8/6b7fef71-3444-4c8f-b2e2-502774ba9b51/2542314c-0b08-493b-856b-65d680d18812"
-					(reference "R48")
+					(reference "R804")
 					(unit 1)
 				)
@@
 		(dnp no)
 		(fields_autoplaced yes)
-		(property "Reference" "K6"
+		(property "Reference" "K802"
 			(at 111.76 74.93 0)
 			(effects
@@
 			(project "Main Board"
 				(path "/20aae4b7-3fb8-4924-82e8-1e7a29a313f8/6b7fef71-3444-4c8f-b2e2-502774ba9b51/2542314c-0b08-493b-856b-65d680d18812"
-					(reference "K6")
+					(reference "K802")
 					(unit 1)
 				)
@@
 		(dnp no)
 		(fields_autoplaced yes)
-		(property "Reference" "R51"
+		(property "Reference" "R806"
 			(at 41.91 142.24 90)
 			(effects
@@
 			(project "Main Board"
 				(path "/20aae4b7-3fb8-4924-82e8-1e7a29a313f8/6b7fef71-3444-4c8f-b2e2-502774ba9b51/2542314c-0b08-493b-856b-65d680d18812"
-					(reference "R51")
-					(unit 1)
-				)
+					(reference "R806")
+					(unit 1)
+				)

Commit message: :-1:
Parts:
- removed U801: DG419LDY, Package_SO:SOIC-8_3.9x4.9mm_P1.27mm, symbol Analog_Switch:DG419LDY
- added K501: AGQ200A12, AGQ200A12_footprint, symbol AGQ200A12:AGQ200A12
- renumbered K801 to K502, K802 to K503, K803 to K504, K804 to K505, R801 to R501, R802 to R502, R806 to R503, R803 to R504, R804 to R505, R805 to R506
Connections:
- net +12V: now also K501.1
- net GUARD: now also K501.2
- net I_OUT: now also K501.4
- net SELECT_100k: now also K501.8
- net at R506.2: now also K501.3
Other:
- note removed: "there is only one supply for two switches???"
- moved on the sheet: R503, R506

Commit message: sorry i fell asleep b4 layout
Parts:
- added C501, C502, C503, C504, C505, C506: 100n, Capacitor_SMD:C_0805_2012Metric, symbol Device:C
- renumbered K505 to K501, K504 to K502, K502 to K504, K501 to K505, R504 to R503, R505 to R504, R506 to R505, R503 to R506
Connections:
- net IN: now also C501.1, C502.1, C503.1, C504.1, C505.1, C506.1
- net I_OUT: now also C506.2
- net at K503.3, R503.2: now also C503.2
- net at K501.3, R501.2: now also C501.2
- net at K502.3, R502.2: now also C502.2
- net at K505.3, R505.2: now also C505.2
- net at K504.3, R504.2: now also C504.2
Other:
- moved on the sheet: K501, K502, K503, K504, K505, R501, R502, R503, R504, R505, R506

Commit message: HI
Parts:
- K501: renamed from K505; footprint AGQ200A12_footprint -> AGQ:RELAY_AGQ_A_PAN
- K502: renamed from K504; footprint AGQ200A12_footprint -> AGQ:RELAY_AGQ_A_PAN
- K503: footprint AGQ200A12_footprint -> AGQ:RELAY_AGQ_A_PAN
- K504: renamed from K502; footprint AGQ200A12_footprint -> AGQ:RELAY_AGQ_A_PAN
- K505: renamed from K501; footprint AGQ200A12_footprint -> AGQ:RELAY_AGQ_A_PAN
- R501: footprint Resistor_SMD:R_0805_2012Metric -> Resistor_THT:R_Axial_DIN0516_L15.5mm_D5.0mm_P20.32mm_Horizontal
Other:
- note added: "RS02B10R00FE70"
- note removed: "i did double-check it i just need a quick one-over"
- note removed: "need to check the pinout of this relay"
Changed lines of the file:
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@@
 		(company "Harry and Yuki - EEE3 Instrumentation")
 	)
-	(text "i did double-check it i just need a quick one-over"
+	(text "RS02B10R00FE70"
 		(exclude_from_sim no)
-		(at 111.76 30.48 0)
-		(effects
-			(font
-				(size 1.27 1.27)
-			)
-		)
-	)
-	(text "need to check the pinout of this relay \n"
-		(exclude_from_sim no)
-		(at 113.03 27.94 0)
+		(at 46.99 27.94 0)
 		(effects
 			(font
@@
 		(on_board yes)
 		(dnp no)
-		(property "Reference" "#PWR0504"
+		(property "Reference" "#PWR0502"
 			(at 95.25 100.33 0)
 			(effects
@@
 			(project "Main Board"
 				(path "/20aae4b7-3fb8-4924-82e8-1e7a29a313f8/6b7fef71-3444-4c8f-b2e2-502774ba9b51/2542314c-0b08-493b-856b-65d680d18812"
-					(reference "#PWR0504")
+					(reference "#PWR0502")
 					(unit 1)
 				)
@@
 		(on_board yes)
 		(dnp no)
-		(property "Reference" "#PWR0505"
+		(property "Reference" "#PWR0501"
 			(at 73.66 130.81 0)
 			(effects
@@
 			(project "Main Board"
 				(path "/20aae4b7-3fb8-4924-82e8-1e7a29a313f8/6b7fef71-3444-4c8f-b2e2-502774ba9b51/2542314c-0b08-493b-856b-65d680d18812"
-					(reference "#PWR0505")
+					(reference "#PWR0501")
 					(unit 1)
 				)
@@
 			)
 		)
-		(property "Footprint" "Resistor_SMD:R_0805_2012Metric"
+		(property "Footprint" "Resistor_THT:R_Axial_DIN0516_L15.5mm_D5.0mm_P20.32mm_Horizontal"
 			(at 46.99 38.608 90)
 			(effects
@@
 		(dnp no)
 		(fields_autoplaced yes)
-		(property "Reference" "K502"
+		(property "Reference" "K504"
 			(at 142.24 43.18 0)
 			(effects
@@
 			)
 		)
-		(property "Footprint" "AGQ200A12_footprint"
+		(property "Footprint" "AGQ:RELAY_AGQ_A_PAN"
 			(at 153.67 126.67 0)
 			(effects
@@
 			(project "Main Board"
 				(path "/20aae4b7-3fb8-4924-82e8-1e7a29a313f8/6b7fef71-3444-4c8f-b2e2-502774ba9b51/2542314c-0b08-493b-856b-65d680d18812"
-					(reference "K502")
+					(reference "K504")
 					(unit 1)
 				)
@@
 		(on_board yes)
 		(dnp no)
-		(property "Reference" "#PWR0501"
+		(property "Reference" "#PWR0505"
 			(at 170.18 26.67 0)
 			(effects
@@
 			(project "Main Board"
 				(path "/20aae4b7-3fb8-4924-82e8-1e7a29a313f8/6b7fef71-3444-4c8f-b2e2-502774ba9b51/2542314c-0b08-493b-856b-65d680d18812"
-					(reference "#PWR0501")
+					(reference "#PWR0505")
 					(unit 1)
 				)
@@
 		(dnp no)
 		(fields_autoplaced yes)
-		(property "Reference" "K505"
+		(property "Reference" "K501"
 			(at 69.85 120.65 0)
 			(effects
@@
 			)
 		)
-		(property "Footprint" "AGQ200A12_footprint"
+		(property "Footprint" "AGQ:RELAY_AGQ_A_PAN"
 			(at 81.28 204.14 0)
 			(effects
@@
 			(project "Main Board"
 				(path "/20aae4b7-3fb8-4924-82e8-1e7a29a313f8/6b7fef71-3444-4c8f-b2e2-502774ba9b51/2542314c-0b08-493b-856b-65d680d18812"
-					(reference "K505")
+					(reference "K501")
 					(unit 1)
 				)
@@
 		(dnp no)
 		(fields_autoplaced yes)
-		(property "Reference" "K501"
+		(property "Reference" "K505"
 			(at 166.37 16.51 0)
 			(effects
@@
 			)
 		)
-		(property "Footprint" "AGQ200A12_footprint"
+		(property "Footprint" "AGQ:RELAY_AGQ_A_PAN"
 			(at 177.8 100 0)
 			(effects
@@
 			(project ""
 				(path "/20aae4b7-3fb8-4924-82e8-1e7a29a313f8/6b7fef71-3444-4c8f-b2e2-502774ba9b51/2542314c-0b08-493b-856b-65d680d18812"
-					(reference "K501")
+					(reference "K505")
 					(unit 1)
 				)
@@
 		(dnp no)
 		(fields_autoplaced yes)
-		(property "Reference" "K504"
+		(property "Reference" "K502"
 			(at 91.44 90.17 0)
 			(effects
@@
 			)
 		)
-		(property "Footprint" "AGQ200A12_footprint"
+		(property "Footprint" "AGQ:RELAY_AGQ_A_PAN"
 			(at 102.87 173.66 0)
 			(effects
@@
 			(project "Main Board"
 				(path "/20aae4b7-3fb8-4924-82e8-1e7a29a313f8/6b7fef71-3444-4c8f-b2e2-502774ba9b51/2542314c-0b08-493b-856b-65d680d18812"
-					(reference "K504")
+					(reference "K502")
 					(unit 1)
 				)
@@
 		(on_board yes)
 		(dnp no)
-		(property "Reference" "#PWR0502"
+		(property "Reference" "#PWR0504"
 			(at 146.05 53.34 0)
 			(effects
@@
 			(project "Main Board"
 				(path "/20aae4b7-3fb8-4924-82e8-1e7a29a313f8/6b7fef71-3444-4c8f-b2e2-502774ba9b51/2542314c-0b08-493b-856b-65d680d18812"
-					(reference "#PWR0502")
+					(reference "#PWR0504")
 					(unit 1)
 				)
@@
 			)
 		)
-		(property "Footprint" "AGQ200A12_footprint"
+		(property "Footprint" "AGQ:RELAY_AGQ_A_PAN"
 			(at 129.54 150.8 0)
 			(effects
