File: PCB/Main Board/Resistors.kicad_sch (KiCad schematic)
At the start: 17 parts, among them K501 AGQ200A12, K502 AGQ200A12, K503 AGQ200A12, K504 AGQ200A12, K505 AGQ200A12

Commit message: fb capacitances for abb
Parts:
- C501: value 100n -> 16n
- C502: value 100n -> 1.6n
- C503, C506: value 100n -> 160p
- C504, C505: value 100n -> 330p
Connections:
- no-connect marks 12 -> 15
Other:
- note added: "fb=100k"
- note added: "fb=1M"
- note added: "fb=500k"
- moved on the sheet: C501, C502, C503, C504, C505, C506, K501, K502, K503, K504, K505, R501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

Commit message: checkpoint
Parts:
- C506: value 160p -> 56p
Changed lines of the file:
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@@
 			)
 		)
-		(property "Value" "160p"
+		(property "Value" "56p"
 			(at 43.18 176.53 90)
 			(effects

Commit message: resistor footprints changed
Parts:
- removed R501: 10, Resistor_THT:R_Axial_DIN0516_L15.5mm_D5.0mm_P20.32mm_Horizontal, symbol Device:R
- added R? (x4): 10, Resistor_SMD:R_2512_6332Metric, symbol Device:R
Connections:
- net IN: now also R?.1, R?.1
- net at C501.2, K505.3: now also R?.2, R?.2
- new net: R?.1, R?.2 (x2)
Other:
- note removed: "RS02B10R00FE70"

Commit message: merge 2.0
Parts:
- gave numbers to parts that had none: 4
- renumbered R502 to R503, R503 to R504, R504 to R505, R505 to R506, R506 to R507
Changed lines of the file:
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@@
 		(dnp no)
 		(fields_autoplaced yes)
-		(property "Reference" "R503"
+		(property "Reference" "R504"
 			(at 43.18 80.01 90)
 			(effects
@@
 			(project "Main Board"
 				(path "/20aae4b7-3fb8-4924-82e8-1e7a29a313f8/6b7fef71-3444-4c8f-b2e2-502774ba9b51/2542314c-0b08-493b-856b-65d680d18812"
-					(reference "R503")
+					(reference "R504")
 					(unit 1)
 				)
@@
 		(dnp no)
 		(fields_autoplaced yes)
-		(property "Reference" "R?"
+		(property "Reference" "R501"
 			(at 39.37 24.13 90)
 			(effects
@@
 			(project "Main Board"
 				(path "/20aae4b7-3fb8-4924-82e8-1e7a29a313f8/6b7fef71-3444-4c8f-b2e2-502774ba9b51/2542314c-0b08-493b-856b-65d680d18812"
-					(reference "R?")
+					(reference "R501")
 					(unit 1)
 				)
@@
 		(on_board yes)
 		(dnp no)
-		(property "Reference" "R?"
+		(property "Reference" "R509"
 			(at 46.99 41.91 90)
 			(effects
@@
 			(project "Main Board"
 				(path "/20aae4b7-3fb8-4924-82e8-1e7a29a313f8/6b7fef71-3444-4c8f-b2e2-502774ba9b51/2542314c-0b08-493b-856b-65d680d18812"
-					(reference "R?")
+					(reference "R509")
 					(unit 1)
 				)
@@
 		(dnp no)
 		(fields_autoplaced yes)
-		(property "Reference" "R?"
+		(property "Reference" "R508"
 			(at 46.99 24.13 90)
 			(effects
@@
 			(project "Main Board"
 				(path "/20aae4b7-3fb8-4924-82e8-1e7a29a313f8/6b7fef71-3444-4c8f-b2e2-502774ba9b51/2542314c-0b08-493b-856b-65d680d18812"
-					(reference "R?")
+					(reference "R508")
 					(unit 1)
 				)
@@
 		(dnp no)
 		(fields_autoplaced yes)
-		(property "Reference" "R505"
+		(property "Reference" "R506"
 			(at 43.18 133.35 90)
 			(effects
@@
 			(project "Main Board"
 				(path "/20aae4b7-3fb8-4924-82e8-1e7a29a313f8/6b7fef71-3444-4c8f-b2e2-502774ba9b51/2542314c-0b08-493b-856b-65d680d18812"
-					(reference "R505")
+					(reference "R506")
 					(unit 1)
 				)
@@
 		(on_board yes)
 		(dnp no)
-		(property "Reference" "R?"
+		(property "Reference" "R502"
 			(at 39.37 41.91 90)
 			(effects
@@
 			(project "Main Board"
 				(path "/20aae4b7-3fb8-4924-82e8-1e7a29a313f8/6b7fef71-3444-4c8f-b2e2-502774ba9b51/2542314c-0b08-493b-856b-65d680d18812"
-					(reference "R?")
+					(reference "R502")
 					(unit 1)
 				)
@@
 		(dnp no)
 		(fields_autoplaced yes)
-		(property "Reference" "R502"
+		(property "Reference" "R503"
 			(at 43.18 57.15 90)
 			(effects
@@
 			(project "Main Board"
 				(path "/20aae4b7-3fb8-4924-82e8-1e7a29a313f8/6b7fef71-3444-4c8f-b2e2-502774ba9b51/2542314c-0b08-493b-856b-65d680d18812"
-					(reference "R502")
+					(reference "R503")
 					(unit 1)
 				)
@@
 		(dnp no)
 		(fields_autoplaced yes)
-		(property "Reference" "R504"
+		(property "Reference" "R505"
 			(at 43.18 102.87 90)
 			(effects
@@
 			(project "Main Board"
 				(path "/20aae4b7-3fb8-4924-82e8-1e7a29a313f8/6b7fef71-3444-4c8f-b2e2-502774ba9b51/2542314c-0b08-493b-856b-65d680d18812"
-					(reference "R504")
+					(reference "R505")
 					(unit 1)
 				)
@@
 		(on_board yes)
 		(dnp no)
-		(property "Reference" "R506"
+		(property "Reference" "R507"
 			(at 43.18 157.48 90)
 			(effects
@@
 			(project "Main Board"
 				(path "/20aae4b7-3fb8-4924-82e8-1e7a29a313f8/6b7fef71-3444-4c8f-b2e2-502774ba9b51/2542314c-0b08-493b-856b-65d680d18812"
-					(reference "R506")
-					(unit 1)
-				)
+					(reference "R507")
+					(unit 1)
+				)

Commit message: sig source finished
Parts:
- renumbered K505 to K501, K504 to K502, K502 to K504, K501 to K505, R508 to R502, R502 to R503, R509 to R504, R503 to R505, R504 to R506, R505 to R507, R506 to R508, R507 to R509
Other:
- moved on the sheet: C501, K501, R501, R502, R503, R504

Commit message: hello
Parts:
- added R501, R511, R512: 100, Resistor_SMD:R_0805_2012Metric, symbol Device:R
- renumbered K505 to K501, K504 to K502, K502 to K504, K501 to K505, R505 to R502, R501 to R503, R503 to R504, R506 to R505, R507 to R506, R508 to R507, R509 to R508, R502 to R509, R504 to R510
Connections:
- net IN: now also R501.1
- net at C502.2, K504.3: now also R511.2, R512.2; no longer R502.2
- new net: R502.2, R512.1
- new net: R501.2, R511.1
Other:
- moved on the sheet: R502

Commit message: please be nice
Parts:
- renumbered K505 to K501, K504 to K502, K502 to K504, K501 to K505, R503 to R501, R509 to R502, R504 to R503, R510 to R504, R501 to R505, R511 to R506, R502 to R507, R512 to R508, R505 to R509, R506 to R510, R507 to R511, R508 to R512
Changed lines of the file:
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@@
 		(dnp no)
 		(fields_autoplaced yes)
-		(property "Reference" "R505"
+		(property "Reference" "R509"
 			(at 43.18 80.01 90)
 			(effects
@@
 			(project "Main Board"
 				(path "/20aae4b7-3fb8-4924-82e8-1e7a29a313f8/6b7fef71-3444-4c8f-b2e2-502774ba9b51/2542314c-0b08-493b-856b-65d680d18812"
-					(reference "R505")
+					(reference "R509")
 					(unit 1)
 				)
@@
 		(dnp no)
 		(fields_autoplaced yes)
-		(property "Reference" "R503"
+		(property "Reference" "R501"
 			(at 39.37 17.78 90)
 			(effects
@@
 			(project "Main Board"
 				(path "/20aae4b7-3fb8-4924-82e8-1e7a29a313f8/6b7fef71-3444-4c8f-b2e2-502774ba9b51/2542314c-0b08-493b-856b-65d680d18812"
-					(reference "R503")
+					(reference "R501")
 					(unit 1)
 				)
@@
 		(on_board yes)
 		(dnp no)
-		(property "Reference" "#PWR0502"
+		(property "Reference" "#PWR0504"
 			(at 111.76 99.06 0)
 			(effects
@@
 			(project "Main Board"
 				(path "/20aae4b7-3fb8-4924-82e8-1e7a29a313f8/6b7fef71-3444-4c8f-b2e2-502774ba9b51/2542314c-0b08-493b-856b-65d680d18812"
-					(reference "#PWR0502")
+					(reference "#PWR0504")
 					(unit 1)
 				)
@@
 		(on_board yes)
 		(dnp no)
-		(property "Reference" "R510"
+		(property "Reference" "R504"
 			(at 46.99 35.56 90)
 			(effects
@@
 			(project "Main Board"
 				(path "/20aae4b7-3fb8-4924-82e8-1e7a29a313f8/6b7fef71-3444-4c8f-b2e2-502774ba9b51/2542314c-0b08-493b-856b-65d680d18812"
-					(reference "R510")
+					(reference "R504")
 					(unit 1)
 				)
@@
 		(on_board yes)
 		(dnp no)
-		(property "Reference" "R512"
+		(property "Reference" "R508"
 			(at 50.8 57.15 90)
 			(effects
@@
 			(project "Main Board"
 				(path "/20aae4b7-3fb8-4924-82e8-1e7a29a313f8/6b7fef71-3444-4c8f-b2e2-502774ba9b51/2542314c-0b08-493b-856b-65d680d18812"
-					(reference "R512")
+					(reference "R508")
 					(unit 1)
 				)
@@
 		(on_board yes)
 		(dnp no)
-		(property "Reference" "#PWR0501"
+		(property "Reference" "#PWR0505"
 			(at 86.36 129.54 0)
 			(effects
@@
 			(project "Main Board"
 				(path "/20aae4b7-3fb8-4924-82e8-1e7a29a313f8/6b7fef71-3444-4c8f-b2e2-502774ba9b51/2542314c-0b08-493b-856b-65d680d18812"
-					(reference "#PWR0501")
+					(reference "#PWR0505")
 					(unit 1)
 				)
@@
 		(dnp no)
 		(fields_autoplaced yes)
-		(property "Reference" "K504"
+		(property "Reference" "K502"
 			(at 160.02 43.18 0)
 			(effects
@@
 			(project "Main Board"
 				(path "/20aae4b7-3fb8-4924-82e8-1e7a29a313f8/6b7fef71-3444-4c8f-b2e2-502774ba9b51/2542314c-0b08-493b-856b-65d680d18812"
-					(reference "K504")
+					(reference "K502")
 					(unit 1)
 				)
@@
 		(dnp no)
 		(fields_autoplaced yes)
-		(property "Reference" "R509"
+		(property "Reference" "R502"
 			(at 46.99 17.78 90)
 			(effects
@@
 			(project "Main Board"
 				(path "/20aae4b7-3fb8-4924-82e8-1e7a29a313f8/6b7fef71-3444-4c8f-b2e2-502774ba9b51/2542314c-0b08-493b-856b-65d680d18812"
-					(reference "R509")
+					(reference "R502")
 					(unit 1)
 				)
@@
 		(on_board yes)
 		(dnp no)
-		(property "Reference" "#PWR0505"
+		(property "Reference" "#PWR0501"
 			(at 189.23 24.13 0)
 			(effects
@@
 			(project "Main Board"
 				(path "/20aae4b7-3fb8-4924-82e8-1e7a29a313f8/6b7fef71-3444-4c8f-b2e2-502774ba9b51/2542314c-0b08-493b-856b-65d680d18812"
-					(reference "#PWR0505")
+					(reference "#PWR0501")
 					(unit 1)
 				)
@@
 		(dnp no)
 		(fields_autoplaced yes)
-		(property "Reference" "K501"
+		(property "Reference" "K505"
 			(at 82.55 119.38 0)
 			(effects
@@
 			(project "Main Board"
 				(path "/20aae4b7-3fb8-4924-82e8-1e7a29a313f8/6b7fef71-3444-4c8f-b2e2-502774ba9b51/2542314c-0b08-493b-856b-65d680d18812"
-					(reference "K501")
+					(reference "K505")
 					(unit 1)
 				)
@@
 		(dnp no)
 		(fields_autoplaced yes)
-		(property "Reference" "K505"
+		(property "Reference" "K501"
 			(at 185.42 13.97 0)
 			(effects
@@
 			(project ""
 				(path "/20aae4b7-3fb8-4924-82e8-1e7a29a313f8/6b7fef71-3444-4c8f-b2e2-502774ba9b51/2542314c-0b08-493b-856b-65d680d18812"
-					(reference "K505")
+					(reference "K501")
 					(unit 1)
 				)
@@
 		(dnp no)
 		(fields_autoplaced yes)
-		(property "Reference" "K502"
+		(property "Reference" "K504"
 			(at 107.95 88.9 0)
 			(effects
@@
 			(project "Main Board"
 				(path "/20aae4b7-3fb8-4924-82e8-1e7a29a313f8/6b7fef71-3444-4c8f-b2e2-502774ba9b51/2542314c-0b08-493b-856b-65d680d18812"
-					(reference "K502")
+					(reference "K504")
 					(unit 1)
 				)
@@
 		(dnp no)
 		(fields_autoplaced yes)
-		(property "Reference" "R507"
+		(property "Reference" "R511"
 			(at 43.18 133.35 90)
 			(effects
@@
 			(project "Main Board"
 				(path "/20aae4b7-3fb8-4924-82e8-1e7a29a313f8/6b7fef71-3444-4c8f-b2e2-502774ba9b51/2542314c-0b08-493b-856b-65d680d18812"
-					(reference "R507")
+					(reference "R511")
 					(unit 1)
 				)
@@
 		(on_board yes)
 		(dnp no)
-		(property "Reference" "R504"
+		(property "Reference" "R503"
 			(at 39.37 35.56 90)
 			(effects
@@
 			(project "Main Board"
 				(path "/20aae4b7-3fb8-4924-82e8-1e7a29a313f8/6b7fef71-3444-4c8f-b2e2-502774ba9b51/2542314c-0b08-493b-856b-65d680d18812"
-					(reference "R504")
+					(reference "R503")
 					(unit 1)
 				)
@@
 		(on_board yes)
 		(dnp no)
-		(property "Reference" "R511"
+		(property "Reference" "R506"
 			(at 50.8 48.26 90)
 			(effects
@@
 			(project "Main Board"
 				(path "/20aae4b7-3fb8-4924-82e8-1e7a29a313f8/6b7fef71-3444-4c8f-b2e2-502774ba9b51/2542314c-0b08-493b-856b-65d680d18812"
-					(reference "R511")
+					(reference "R506")
 					(unit 1)
 				)
@@
 		(on_board yes)
 		(dnp no)
-		(property "Reference" "R501"
+		(property "Reference" "R505"
 			(at 38.1 48.26 90)
 			(effects
@@
 			(project "Main Board"
 				(path "/20aae4b7-3fb8-4924-82e8-1e7a29a313f8/6b7fef71-3444-4c8f-b2e2-502774ba9b51/2542314c-0b08-493b-856b-65d680d18812"
-					(reference "R501")
+					(reference "R505")
 					(unit 1)
 				)
@@
 		(on_board yes)
 		(dnp no)
-		(property "Reference" "#PWR0504"
+		(property "Reference" "#PWR0502"
 			(at 163.83 53.34 0)
 			(effects
@@
 			(project "Main Board"
 				(path "/20aae4b7-3fb8-4924-82e8-1e7a29a313f8/6b7fef71-3444-4c8f-b2e2-502774ba9b51/2542314c-0b08-493b-856b-65d680d18812"
-					(reference "#PWR0504")
+					(reference "#PWR0502")
 					(unit 1)
 				)
@@
 		(on_board yes)
 		(dnp no)
-		(property "Reference" "R502"
+		(property "Reference" "R507"
 			(at 38.1 57.15 90)
 			(effects
@@
 			(project "Main Board"
 				(path "/20aae4b7-3fb8-4924-82e8-1e7a29a313f8/6b7fef71-3444-4c8f-b2e2-502774ba9b51/2542314c-0b08-493b-856b-65d680d18812"
-					(reference "R502")
+					(reference "R507")
 					(unit 1)
 				)
@@
 		(dnp no)
 		(fields_autoplaced yes)
-		(property "Reference" "R506"
+		(property "Reference" "R510"
 			(at 43.18 102.87 90)
 			(effects
@@
 			(project "Main Board"
 				(path "/20aae4b7-3fb8-4924-82e8-1e7a29a313f8/6b7fef71-3444-4c8f-b2e2-502774ba9b51/2542314c-0b08-493b-856b-65d680d18812"
-					(reference "R506")
+					(reference "R510")
 					(unit 1)
 				)
@@
 		(on_board yes)
 		(dnp no)
-		(property "Reference" "R508"
+		(property "Reference" "R512"
 			(at 43.18 157.48 90)
 			(effects
@@
 			(project "Main Board"
 				(path "/20aae4b7-3fb8-4924-82e8-1e7a29a313f8/6b7fef71-3444-4c8f-b2e2-502774ba9b51/2542314c-0b08-493b-856b-65d680d18812"
-					(reference "R508")
-					(unit 1)
-				)
+					(reference "R512")
+					(unit 1)
+				)

Commit message: Final Schematic
Parts:
- renumbered C501 to C33, C502 to C34, C503 to C35, C504 to C36, C505 to C37, C506 to C38, K505 to K3, K504 to K4, K503 to K5, K502 to K6, K501 to K7, R505 to R46, R507 to R47, R501 to R48, R503 to R49, R509 to R50, R510 to R51, R511 to R52, R512 to R53, R502 to R54, R504 to R55, R506 to R56, R508 to R57
Other:
- title: (none) -> Resistor Selector
