File: PCB/Main Board/currentamp.kicad_sch (KiCad schematic)
At the start: 51 parts, among them U10 OPA2197xD, U11 DG201, U7 DG201, U8 INA828D, U9 OPA2197xD

Commit message: footprints and stm wiring
Parts:
- removed C? (x2): 100n, symbol Device:C
- removed JP?: SolderJumper_2_Open, Jumper:SolderJumper-2_P1.3mm_Open_RoundedPad1.0x1.5mm, symbol Jumper:SolderJumper_2_Open
- added C? (x2): 100n, symbol Device:C
- added JP?: SolderJumper_2_Open, Jumper:SolderJumper-2_P1.3mm_Open_RoundedPad1.0x1.5mm, symbol Jumper:SolderJumper_2_Open
Connections:
- net +1.65VA: no longer R34.2, R35.2, U10.7, U9.3 (+)
- net +18V: now also C?.2
- net -18V: now also C?.2
- net GND: now also C?.1, C?.1
- new net 1.65VA_REF: R34.2, R35.2, U10.7, U9.3 (+)
Other:
- company: Harry and Yuki - EEE3 Instrumentation -> (none)
- title: Instrumentation Amplifier -> (none)

Commit message: relays and layout begin
Parts:
- C56: renamed from C23; footprint (none) -> Capacitor_SMD:C_0805_2012Metric
- C57: renamed from C24; footprint (none) -> Capacitor_SMD:C_0805_2012Metric
- C58, C61: renamed from C?; footprint (none) -> Capacitor_SMD:C_0805_2012Metric
- C59: renamed from C25; footprint (none) -> Capacitor_SMD:C_0805_2012Metric
- C60: renamed from C26; footprint (none) -> Capacitor_SMD:C_0805_2012Metric
- C62: renamed from C27; footprint (none) -> Capacitor_SMD:C_0805_2012Metric
- C63: renamed from C28; footprint (none) -> Capacitor_SMD:C_0805_2012Metric
- C64: renamed from C35; footprint (none) -> Capacitor_SMD:C_0805_2012Metric
- C65: renamed from C29; footprint (none) -> Capacitor_SMD:C_0805_2012Metric
- C66: renamed from C30; footprint (none) -> Capacitor_SMD:C_0805_2012Metric
- C67: renamed from C36; footprint (none) -> Capacitor_SMD:C_0805_2012Metric
- C68: renamed from C31; footprint (none) -> Capacitor_SMD:C_0805_2012Metric
- C69: renamed from C37; footprint (none) -> Capacitor_SMD:C_0805_2012Metric
- C70: renamed from C32; footprint (none) -> Capacitor_SMD:C_0805_2012Metric
- C71: renamed from C33; footprint (none) -> Capacitor_SMD:C_0805_2012Metric
- C72: renamed from C38; footprint (none) -> Capacitor_SMD:C_0805_2012Metric
- C73: renamed from C34; footprint (none) -> Capacitor_SMD:C_0805_2012Metric
- R73: renamed from R25; footprint (none) -> Resistor_SMD:R_0805_2012Metric
- R74: renamed from R26; footprint (none) -> Resistor_SMD:R_0805_2012Metric
- R75: renamed from R27; footprint (none) -> Resistor_SMD:R_0805_2012Metric
- R76: renamed from R28; footprint (none) -> Resistor_SMD:R_0805_2012Metric
- R77: renamed from R29; footprint (none) -> Resistor_SMD:R_0805_2012Metric
- R78: renamed from R30; footprint (none) -> Resistor_SMD:R_0805_2012Metric
- R79: renamed from R31; footprint (none) -> Resistor_SMD:R_0805_2012Metric
- R80: renamed from R32; footprint (none) -> Resistor_SMD:R_0805_2012Metric
- R81: renamed from R33; footprint (none) -> Resistor_SMD:R_0805_2012Metric
- R82: renamed from R36; footprint (none) -> Resistor_SMD:R_0805_2012Metric
- R83: renamed from R37; footprint (none) -> Resistor_SMD:R_0805_2012Metric
- R84: renamed from R38; footprint (none) -> Resistor_SMD:R_0805_2012Metric
- R85: renamed from R34; footprint (none) -> Resistor_SMD:R_0805_2012Metric
- R86: renamed from R35; footprint (none) -> Resistor_SMD:R_0805_2012Metric
- R87: renamed from R39; footprint (none) -> Resistor_SMD:R_0805_2012Metric
- R88: renamed from R40; footprint (none) -> Resistor_SMD:R_0805_2012Metric
- R89: renamed from R41; footprint (none) -> Resistor_SMD:R_0805_2012Metric
- R90: renamed from R42; footprint (none) -> Resistor_SMD:R_0805_2012Metric
- R91: renamed from R43; footprint (none) -> Resistor_SMD:R_0805_2012Metric
- R92: renamed from R44; footprint (none) -> Resistor_SMD:R_0805_2012Metric
- R93: renamed from R45; footprint (none) -> Resistor_SMD:R_0805_2012Metric
- gave numbers to parts that had none: 1
- renumbered JP8 to JP18, JP9 to JP19, JP10 to JP20, JP11 to JP21, JP12 to JP22, JP13 to JP23, U7 to U18, U8 to U19, U9 to U20, U10 to U21, U11 to U22

Commit message: minor and layout
Parts:
- removed C58, C61: 100n, Capacitor_SMD:C_0805_2012Metric, symbol Device:C
- removed C73: 5.6n, Capacitor_SMD:C_0805_2012Metric, symbol Device:C
- removed JP17: SolderJumper_2_Open, Jumper:SolderJumper-2_P1.3mm_Open_RoundedPad1.0x1.5mm, symbol Jumper:SolderJumper_2_Open
- removed JP20, JP23: SolderJumper_2_Bridged, Jumper:SolderJumper-2_P1.3mm_Bridged_RoundedPad1.0x1.5mm, symbol Jumper:SolderJumper_2_Bridged
- removed R85, R86, R87, R88: 10k, Resistor_SMD:R_0805_2012Metric, symbol Device:R
- removed R89: 2.7M, Resistor_SMD:R_0805_2012Metric, symbol Device:R
- removed R90: 10M, Resistor_SMD:R_0805_2012Metric, symbol Device:R
- removed R91: 300k, Resistor_SMD:R_0805_2012Metric, symbol Device:R
- removed R92: 27k, Resistor_SMD:R_0805_2012Metric, symbol Device:R
- removed R93: 2.7k, Resistor_SMD:R_0805_2012Metric, symbol Device:R
- removed unit 1 of U21
- removed unit 2 of U22
- removed unit 4 of U22
- removed unit 3 of U22
- removed unit 1 of U22
Connections:
- net +1.65VA: now also U20.3 (+), U21.5 (+)
- net at U21.6 (-): now also U21.7
- removed net 1.65VA_REF: U20.3 (+), U21.7
Other:
- note removed: "Cut if populating"
- note removed: "Cut to isolate"
- moved on the sheet: U20A, U21B

Commit message: :ghost:
Parts:
- renumbered C63 to C1001, C68 to C1002, C56 to C1003, C59 to C1004, C62 to C1005, C64 to C1006, C69 to C1007, C65 to C1008, C70 to C1009, C66 to C1010, C71 to C1011, C60 to C1012, C67 to C1013, C72 to C1014, C57 to C1015, JP18 to JP1001, JP21 to JP1002, JP19 to JP1003, JP22 to JP1004, R75 to R1001, R82 to R1002, R76 to R1003, R73 to R1004, R77 to R1005, R83 to R1006, R74 to R1007, R78 to R1008, R79 to R1009, R80 to R1010, R81 to R1011, R84 to R1012, U21 to U1001, U19 to U1002, U18 to U1003, U20 to U1004, U22 to U1005
Other:
- moved on the sheet: U1004A

Commit message: aaa
Parts:
- removed C1010, C1011: 100n, Capacitor_SMD:C_0805_2012Metric, symbol Device:C
- removed JP1001, JP1002: SolderJumper_2_Open, Jumper:SolderJumper-2_P1.3mm_Open_RoundedPad1.0x1.5mm, symbol Jumper:SolderJumper_2_Open
- removed JP1003, JP1004: SolderJumper_2_Bridged, Jumper:SolderJumper-2_P1.3mm_Bridged_RoundedPad1.0x1.5mm, symbol Jumper:SolderJumper_2_Bridged
- removed U1005: DG201, Package_SO:SOIC-16_3.9x9.9mm_P1.27mm, symbol More_symbols:DG201
- added JP1001, JP1002: SolderJumper_3_Bridged12, Jumper:SolderJumper-3_P1.3mm_Bridged123_RoundedPad1.0x1.5mm, symbol Jumper:SolderJumper_3_Bridged12
- renumbered C1012 to C1010, C1013 to C1011, C1014 to C1012, C1015 to C1013
Connections:
- net +18V: now also JP1001.3 (B)
- net +3.3VA: now also JP1001.1 (A)
- net -18V: now also JP1002.3 (B)
- net GND: now also JP1002.1 (A)
- net at C1002.2, U1004.4 (V-): now also JP1002.2 (C)
- net at C1001.1, U1004.8 (V+): now also JP1001.2 (C)

Commit message: progress
Parts:
- removed C1011, C1012: 100n, Capacitor_SMD:C_0805_2012Metric, symbol Device:C
- removed U1001, U1004: OPA2197xD, Package_SO:SOIC-8_3.9x4.9mm_P1.27mm, symbol Amplifier_Operational:OPA2197xD
- added U? (x3): OPA2376xxD, Package_SO:SOIC-8_3.9x4.9mm_P1.27mm, symbol Amplifier_Operational:OPA2376xxD
Connections:
- net +1.65VA: now also U?.3 (+)
- net Out: now also U?.7
- net at C1010.1, R1010.2: now also U?.5 (+)
- net at R1011.1, R1012.2: now also U?.6 (-)
- net at C1003.2, C1004.2, C1005.2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: now also U?.1
- net at C1005.1, R1002.2, R1006.2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: now also U?.2 (-)
- net at C1001.1, JP1001.2 (C): now also U?.8 (V+)
- net at C1002.2, JP1002.2 (C): now also U?.4 (V-)

Commit message: beep beep
Parts:
- gave numbers to parts that had none: 1
- renumbered C1013 to C1011, U1002 to U1001, U1003 to U1002
Changed lines of the file:
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@@
 		(on_board yes)
 		(dnp no)
-		(property "Reference" "U1002"
+		(property "Reference" "U1001"
 			(at 64.77 40.64 0)
 			(effects
@@
 			(project "Main Board"
 				(path "/20aae4b7-3fb8-4924-82e8-1e7a29a313f8/2e1ccfa8-8bce-4bb4-9d3d-716156df4d18"
-					(reference "U1002")
+					(reference "U1001")
 					(unit 1)
 				)
@@
 		(dnp no)
 		(fields_autoplaced yes)
-		(property "Reference" "U?"
+		(property "Reference" "U1003"
 			(at 152.4 69.85 0)
 			(effects
@@
 			(project ""
 				(path "/20aae4b7-3fb8-4924-82e8-1e7a29a313f8/2e1ccfa8-8bce-4bb4-9d3d-716156df4d18"
-					(reference "U?")
+					(reference "U1003")
 					(unit 1)
 				)
@@
 		(dnp no)
 		(fields_autoplaced yes)
-		(property "Reference" "U?"
+		(property "Reference" "U1003"
 			(at 238.76 40.64 0)
 			(effects
@@
 			(project ""
 				(path "/20aae4b7-3fb8-4924-82e8-1e7a29a313f8/2e1ccfa8-8bce-4bb4-9d3d-716156df4d18"
-					(reference "U?")
+					(reference "U1003")
 					(unit 2)
 				)
@@
 		(dnp no)
 		(fields_autoplaced yes)
-		(property "Reference" "#PWR01004"
+		(property "Reference" "#PWR01003"
 			(at 148.59 82.55 0)
 			(effects
@@
 			(project "Main Board"
 				(path "/20aae4b7-3fb8-4924-82e8-1e7a29a313f8/2e1ccfa8-8bce-4bb4-9d3d-716156df4d18"
-					(reference "#PWR01004")
+					(reference "#PWR01003")
 					(unit 1)
 				)
@@
 		(dnp no)
 		(fields_autoplaced yes)
-		(property "Reference" "#PWR01021"
+		(property "Reference" "#PWR01017"
 			(at 261.62 127 0)
 			(effects
@@
 			(project "Main Board"
 				(path "/20aae4b7-3fb8-4924-82e8-1e7a29a313f8/2e1ccfa8-8bce-4bb4-9d3d-716156df4d18"
-					(reference "#PWR01021")
+					(reference "#PWR01017")
 					(unit 1)
 				)
@@
 		(dnp no)
 		(fields_autoplaced yes)
-		(property "Reference" "#PWR01007"
+		(property "Reference" "#PWR01006"
 			(at 166.37 125.73 0)
 			(effects
@@
 			(project "Main Board"
 				(path "/20aae4b7-3fb8-4924-82e8-1e7a29a313f8/2e1ccfa8-8bce-4bb4-9d3d-716156df4d18"
-					(reference "#PWR01007")
+					(reference "#PWR01006")
 					(unit 1)
 				)
@@
 		(dnp no)
 		(fields_autoplaced yes)
-		(property "Reference" "#PWR01014"
+		(property "Reference" "#PWR01013"
 			(at 198.12 137.16 0)
 			(effects
@@
 			(project "Main Board"
 				(path "/20aae4b7-3fb8-4924-82e8-1e7a29a313f8/2e1ccfa8-8bce-4bb4-9d3d-716156df4d18"
-					(reference "#PWR01014")
+					(reference "#PWR01013")
 					(unit 1)
 				)
@@
 		(dnp no)
 		(fields_autoplaced yes)
-		(property "Reference" "#PWR01002"
+		(property "Reference" "#PWR01001"
 			(at 62.23 44.45 0)
 			(effects
@@
 			(project "Main Board"
 				(path "/20aae4b7-3fb8-4924-82e8-1e7a29a313f8/2e1ccfa8-8bce-4bb4-9d3d-716156df4d18"
-					(reference "#PWR01002")
+					(reference "#PWR01001")
 					(unit 1)
 				)
@@
 		(dnp no)
 		(fields_autoplaced yes)
-		(property "Reference" "#PWR01008"
+		(property "Reference" "#PWR01007"
 			(at 172.72 137.16 0)
 			(effects
@@
 			(project "Main Board"
 				(path "/20aae4b7-3fb8-4924-82e8-1e7a29a313f8/2e1ccfa8-8bce-4bb4-9d3d-716156df4d18"
-					(reference "#PWR01008")
+					(reference "#PWR01007")
 					(unit 1)
 				)
@@
 		(on_board yes)
 		(dnp no)
-		(property "Reference" "#PWR01023"
+		(property "Reference" "#PWR01019"
 			(at 264.16 144.78 0)
 			(effects
@@
 			(project "Main Board"
 				(path "/20aae4b7-3fb8-4924-82e8-1e7a29a313f8/2e1ccfa8-8bce-4bb4-9d3d-716156df4d18"
-					(reference "#PWR01023")
+					(reference "#PWR01019")
 					(unit 1)
 				)
@@
 		(dnp no)
 		(fields_autoplaced yes)
-		(property "Reference" "#PWR01003"
+		(property "Reference" "#PWR01002"
 			(at 62.23 52.07 0)
 			(effects
@@
 			(project "Main Board"
 				(path "/20aae4b7-3fb8-4924-82e8-1e7a29a313f8/2e1ccfa8-8bce-4bb4-9d3d-716156df4d18"
-					(reference "#PWR01003")
+					(reference "#PWR01002")
 					(unit 1)
 				)
@@
 		(dnp no)
 		(fields_autoplaced yes)
-		(property "Reference" "U1003"
+		(property "Reference" "U1002"
 			(at 143.51 53.34 0)
 			(effects
@@
 			(project "Main Board"
 				(path "/20aae4b7-3fb8-4924-82e8-1e7a29a313f8/2e1ccfa8-8bce-4bb4-9d3d-716156df4d18"
-					(reference "U1003")
+					(reference "U1002")
 					(unit 2)
 				)
@@
 		(dnp no)
 		(fields_autoplaced yes)
-		(property "Reference" "U1003"
+		(property "Reference" "U1002"
 			(at 269.24 134.6199 0)
 			(effects
@@
 			(project "Main Board"
 				(path "/20aae4b7-3fb8-4924-82e8-1e7a29a313f8/2e1ccfa8-8bce-4bb4-9d3d-716156df4d18"
-					(reference "U1003")
+					(reference "U1002")
 					(unit 5)
 				)
@@
 		(dnp no)
 		(fields_autoplaced yes)
-		(property "Reference" "#PWR01015"
+		(property "Reference" "#PWR01014"
 			(at 191.77 140.97 0)
 			(effects
@@
 			(project "Main Board"
 				(path "/20aae4b7-3fb8-4924-82e8-1e7a29a313f8/2e1ccfa8-8bce-4bb4-9d3d-716156df4d18"
-					(reference "#PWR01015")
+					(reference "#PWR01014")
 					(unit 1)
 				)
@@
 		(dnp no)
 		(fields_autoplaced yes)
-		(property "Reference" "#PWR01006"
+		(property "Reference" "#PWR01005"
 			(at 153.67 158.75 0)
 			(effects
@@
 			(project "Main Board"
 				(path "/20aae4b7-3fb8-4924-82e8-1e7a29a313f8/2e1ccfa8-8bce-4bb4-9d3d-716156df4d18"
-					(reference "#PWR01006")
+					(reference "#PWR01005")
 					(unit 1)
 				)
@@
 		(dnp no)
 		(fields_autoplaced yes)
-		(property "Reference" "#PWR01020"
+		(property "Reference" "#PWR01016"
 			(at 251.46 88.9 0)
 			(effects
@@
 			(project "Main Board"
 				(path "/20aae4b7-3fb8-4924-82e8-1e7a29a313f8/2e1ccfa8-8bce-4bb4-9d3d-716156df4d18"
-					(reference "#PWR01020")
+					(reference "#PWR01016")
 					(unit 1)
 				)
@@
 		(on_board yes)
 		(dnp no)
-		(property "Reference" "U1003"
+		(property "Reference" "U1002"
 			(at 255.27 78.7399 90)
 			(effects
@@
 			(project "Main Board"
 				(path "/20aae4b7-3fb8-4924-82e8-1e7a29a313f8/2e1ccfa8-8bce-4bb4-9d3d-716156df4d18"
-					(reference "U1003")
+					(reference "U1002")
 					(unit 4)
 				)
@@
 		(dnp no)
 		(fields_autoplaced yes)
-		(property "Reference" "#PWR01012"
+		(property "Reference" "#PWR01011"
 			(at 179.07 140.97 0)
 			(effects
@@
 			(project "Main Board"
 				(path "/20aae4b7-3fb8-4924-82e8-1e7a29a313f8/2e1ccfa8-8bce-4bb4-9d3d-716156df4d18"
-					(reference "#PWR01012")
+					(reference "#PWR01011")
 					(unit 1)
 				)
@@
 		(on_board yes)
 		(dnp no)
-		(property "Reference" "#PWR01022"
+		(property "Reference" "#PWR01018"
 			(at 261.62 154.94 0)
 			(effects
@@
 			(project "Main Board"
 				(path "/20aae4b7-3fb8-4924-82e8-1e7a29a313f8/2e1ccfa8-8bce-4bb4-9d3d-716156df4d18"
-					(reference "#PWR01022")
+					(reference "#PWR01018")
 					(unit 1)
 				)
@@
 		(dnp no)
 		(fields_autoplaced yes)
-		(property "Reference" "#PWR01011"
+		(property "Reference" "#PWR01010"
 			(at 185.42 137.16 0)
 			(effects
@@
 			(project "Main Board"
 				(path "/20aae4b7-3fb8-4924-82e8-1e7a29a313f8/2e1ccfa8-8bce-4bb4-9d3d-716156df4d18"
-					(reference "#PWR01011")
+					(reference "#PWR01010")
 					(unit 1)
 				)
@@
 		(on_board yes)
 		(dnp no)
-		(property "Reference" "#PWR01009"
+		(property "Reference" "#PWR01008"
 			(at 166.37 148.59 0)
 			(effects
@@
 			(project "Main Board"
 				(path "/20aae4b7-3fb8-4924-82e8-1e7a29a313f8/2e1ccfa8-8bce-4bb4-9d3d-716156df4d18"
-					(reference "#PWR01009")
+					(reference "#PWR01008")
 					(unit 1)
 				)
@@
 		(dnp no)
 		(fields_autoplaced yes)
-		(property "Reference" "#PWR01010"
+		(property "Reference" "#PWR01009"
 			(at 179.07 133.35 0)
 			(effects
@@
 			(project "Main Board"
 				(path "/20aae4b7-3fb8-4924-82e8-1e7a29a313f8/2e1ccfa8-8bce-4bb4-9d3d-716156df4d18"
-					(reference "#PWR01010")
+					(reference "#PWR01009")
 					(unit 1)
 				)
@@
 		(dnp no)
 		(fields_autoplaced yes)
-		(property "Reference" "#PWR01018"
+		(property "Reference" "#PWR01015"
 			(at 219.71 57.15 0)
 			(effects
@@
 			(project "Main Board"
 				(path "/20aae4b7-3fb8-4924-82e8-1e7a29a313f8/2e1ccfa8-8bce-4bb4-9d3d-716156df4d18"
-					(reference "#PWR01018")
+					(reference "#PWR01015")
 					(unit 1)
 				)
@@
 		(dnp no)
 		(fields_autoplaced yes)
-		(property "Reference" "#PWR01013"
+		(property "Reference" "#PWR01012"
 			(at 191.77 133.35 0)
 			(effects
@@
 			(project "Main Board"
 				(path "/20aae4b7-3fb8-4924-82e8-1e7a29a313f8/2e1ccfa8-8bce-4bb4-9d3d-716156df4d18"
-					(reference "#PWR01013")
+					(reference "#PWR01012")
 					(unit 1)
 				)
@@
 		(dnp no)
 		(fields_autoplaced yes)
-		(property "Reference" "U?"
+		(property "Reference" "U1003"
 			(at 154.94 135.8899 0)
 			(effects
@@
 			(project ""
 				(path "/20aae4b7-3fb8-4924-82e8-1e7a29a313f8/2e1ccfa8-8bce-4bb4-9d3d-716156df4d18"
-					(reference "U?")
+					(reference "U1003")
 					(unit 3)
 				)
@@
 		(dnp no)
 		(fields_autoplaced yes)
-		(property "Reference" "U1003"
+		(property "Reference" "U1002"
 			(at 118.11 53.34 0)
 			(effects
@@
 			(project "Main Board"
 				(path "/20aae4b7-3fb8-4924-82e8-1e7a29a313f8/2e1ccfa8-8bce-4bb4-9d3d-716156df4d18"
-					(reference "U1003")
+					(reference "U1002")
 					(unit 1)
 				)
@@
 		(dnp no)
 		(fields_autoplaced yes)
-		(property "Reference" "#PWR01005"
+		(property "Reference" "#PWR01004"
 			(at 153.67 125.73 0)
 			(effects
@@
 			(project "Main Board"
 				(path "/20aae4b7-3fb8-4924-82e8-1e7a29a313f8/2e1ccfa8-8bce-4bb4-9d3d-716156df4d18"
-					(reference "#PWR01005")
+					(reference "#PWR01004")
 					(unit 1)
 				)
@@
 		(dnp no)
 		(fields_autoplaced yes)
-		(property "Reference" "C1013"
+		(property "Reference" "C1011"
 			(at 232.41 27.94 90)
 			(effects
@@
 			(project "Main Board"
 				(path "/20aae4b7-3fb8-4924-82e8-1e7a29a313f8/2e1ccfa8-8bce-4bb4-9d3d-716156df4d18"
-					(reference "C1013")
+					(reference "C1011")
 					(unit 1)
 				)
@@
 		(dnp no)
 		(fields_autoplaced yes)
-		(property "Reference" "U1003"
+		(property "Reference" "U1002"
 			(at 143.51 34.29 0)
 			(effects
@@
 			(project "Main Board"
 				(path "/20aae4b7-3fb8-4924-82e8-1e7a29a313f8/2e1ccfa8-8bce-4bb4-9d3d-716156df4d18"
-					(reference "U1003")
+					(reference "U1002")
 					(unit 3)
 				)
