File: PCB/Main Board/currentamp.kicad_sch (KiCad schematic)
At the start: 28 parts, among them U1001 INA828D, U1002 DG201, U1003 OPA2376xxD

Commit message: :-1:
Parts:
- renumbered C1001 to C701, C1002 to C702, C1003 to C703, C1004 to C704, C1005 to C705, C1006 to C706, C1007 to C707, C1008 to C708, C1009 to C709, C1010 to C710, C1011 to C711, JP1001 to JP701, JP1002 to JP702, R1001 to R701, R1002 to R702, R1003 to R703, R1004 to R704, R1005 to R705, R1006 to R706, R1007 to R707, R1008 to R708, R1009 to R709, R1010 to R710, R1011 to R711, R1012 to R712, U1001 to U701, U1002 to U702, U1003 to U703
Connections:
- net +1.65VA: now also U702.11; no longer U702.15
- net x1: now also U702.16; no longer U702.9
- net x3: now also U702.1; no longer U702.8
- net /4: now also U702.8; no longer U702.1
- net ~{x100}: now also U702.9; no longer U702.16
- net at C704.1, R705.2: now also U702.2; no longer U702.6
- net at C705.1, R702.2, R706.2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: now also U702.14, U702.3, U702.6; no longer U702.11, U702.2, U702.7
- net at C703.1, R704.2: now also U702.15; no longer U702.10
- net at R703.2: now also U702.7; no longer U702.3
- net at R712.1: now also U702.10; no longer U702.14
Other:
- moved on the sheet: U702A, U702B, U702C, U702D

Commit message: changed to multiple feedback and minor error correction
Connections:
- no-connect marks 2 -> 3
Other:
- moved on the sheet: R701, R702, R703
Changed lines of the file:
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@@
+	)
+	(no_connect
+		(at 67.31 55.88)
 	)
 	(no_connect
@@
 	(wire
 		(pts
-			(xy 80.01 67.31) (xy 88.9 67.31)
+			(xy 80.01 67.31) (xy 90.17 67.31)
 		)
 		(stroke
@@
 	(wire
 		(pts
-			(xy 102.87 48.26) (xy 110.49 48.26)
+			(xy 104.14 48.26) (xy 110.49 48.26)
 		)
 		(stroke
@@
 	(wire
 		(pts
-			(xy 96.52 67.31) (xy 130.81 67.31)
+			(xy 97.79 67.31) (xy 130.81 67.31)
 		)
 		(stroke
@@
 	(wire
 		(pts
-			(xy 80.01 48.26) (xy 82.55 48.26)
+			(xy 80.01 48.26) (xy 83.82 48.26)
 		)
 		(stroke
@@
 	(wire
 		(pts
-			(xy 90.17 48.26) (xy 95.25 48.26)
+			(xy 91.44 48.26) (xy 96.52 48.26)
 		)
 		(stroke
@@
 	(symbol
 		(lib_id "Device:R")
-		(at 92.71 67.31 90)
+		(at 93.98 67.31 90)
 		(unit 1)
 		(exclude_from_sim no)
@@
 		(dnp no)
 		(property "Reference" "R702"
-			(at 92.71 60.96 90)
+			(at 93.98 60.96 90)
 			(effects
 				(font
@@
 		)
 		(property "Value" "39k"
-			(at 92.71 63.5 90)
+			(at 93.98 63.5 90)
 			(effects
 				(font
@@
 		)
 		(property "Footprint" "Resistor_SMD:R_0805_2012Metric"
-			(at 92.71 69.088 90)
+			(at 93.98 69.088 90)
 			(effects
 				(font
@@
 		)
 		(property "Datasheet" "~"
-			(at 92.71 67.31 0)
+			(at 93.98 67.31 0)
 			(effects
 				(font
@@
 		)
 		(property "Description" "Resistor"
-			(at 92.71 67.31 0)
+			(at 93.98 67.31 0)
 			(effects
 				(font
@@
 	(symbol
 		(lib_id "Device:R")
-		(at 86.36 48.26 90)
+		(at 87.63 48.26 90)
 		(unit 1)
 		(exclude_from_sim no)
@@
 		(fields_autoplaced yes)
 		(property "Reference" "R701"
-			(at 86.36 41.91 90)
+			(at 87.63 41.91 90)
 			(effects
 				(font
@@
 		)
 		(property "Value" "12k"
-			(at 86.36 44.45 90)
+			(at 87.63 44.45 90)
 			(effects
 				(font
@@
 		)
 		(property "Footprint" "Resistor_SMD:R_0805_2012Metric"
-			(at 86.36 50.038 90)
+			(at 87.63 50.038 90)
 			(effects
 				(font
@@
 		)
 		(property "Datasheet" "~"
-			(at 86.36 48.26 0)
+			(at 87.63 48.26 0)
 			(effects
 				(font
@@
 		)
 		(property "Description" "Resistor"
-			(at 86.36 48.26 0)
+			(at 87.63 48.26 0)
 			(effects
 				(font
@@
 	(symbol
 		(lib_id "Device:R")
-		(at 99.06 48.26 90)
+		(at 100.33 48.26 90)
 		(unit 1)
 		(exclude_from_sim no)
@@
 		(fields_autoplaced yes)
 		(property "Reference" "R703"
-			(at 99.06 41.91 90)
+			(at 100.33 41.91 90)
 			(effects
 				(font
@@
 		)
 		(property "Value" "1.5k"
-			(at 99.06 44.45 90)
+			(at 100.33 44.45 90)
 			(effects
 				(font
@@
 		)
 		(property "Footprint" "Resistor_SMD:R_0805_2012Metric"
-			(at 99.06 50.038 90)
+			(at 100.33 50.038 90)
 			(effects
 				(font
@@
 		)
 		(property "Datasheet" "~"
-			(at 99.06 48.26 0)
+			(at 100.33 48.26 0)
 			(effects
 				(font
@@
 		)
 		(property "Description" "Resistor"
-			(at 99.06 48.26 0)
-			(effects
-				(font
+			(at 100.33 48.26 0)
+			(effects
+				(font

Commit message: sorry i fell asleep b4 layout
Parts:
- renumbered C703 to C701, C711 to C702, C704 to C703, C710 to C704, C701 to C706, C706 to C707, C702 to C709, C707 to C710, C709 to C711, R704 to R701, R707 to R702, R701 to R703, R703 to R704, R708 to R706, R709 to R707, R710 to R708, R711 to R709, R702 to R710, R706 to R711, U702 to U701, U701 to U702

Commit message: HI
Parts:
- renumbered C706 to C701, C709 to C702, C701 to C703, C703 to C704, C707 to C706, C710 to C707, C711 to C709, C704 to C710, C702 to C711, R703 to R701, R710 to R702, R704 to R703, R701 to R704, R711 to R706, R702 to R707, R706 to R708, R707 to R709, R708 to R710, R709 to R711, U702 to U701, U701 to U702

Commit message: sig source finished
Parts:
- renumbered C703 to C701, C711 to C702, C704 to C703, C710 to C704, C701 to C706, C706 to C707, C702 to C709, C707 to C710, C709 to C711, R704 to R701, R707 to R702, R701 to R703, R703 to R704, R708 to R706, R709 to R707, R710 to R708, R711 to R709, R702 to R710, R706 to R711, U702 to U701, U701 to U702

Commit message: hello
Parts:
- JP701, JP702: footprint Jumper:SolderJumper-3_P1.3mm_Bridged123_RoundedPad1.0x1.5mm -> Jumper:SolderJumper-3_P1.3mm_Bridged12_RoundedPad1.0x1.5mm
- renumbered C706 to C701, C709 to C702, C701 to C703, C703 to C704, C707 to C706, C710 to C707, C711 to C709, C704 to C710, C702 to C711, R703 to R701, R710 to R702, R704 to R703, R701 to R704, R711 to R706, R702 to R707, R706 to R708, R707 to R709, R708 to R710, R709 to R711, U702 to U701, U701 to U702

Commit message: please be nice
Parts:
- renumbered C703 to C701, C711 to C702, C704 to C703, C710 to C704, C701 to C706, C706 to C707, C702 to C709, C707 to C710, C709 to C711, R704 to R701, R707 to R702, R701 to R703, R703 to R704, R708 to R706, R709 to R707, R710 to R708, R711 to R709, R702 to R710, R706 to R711, U702 to U701, U701 to U702

Commit message: sleepdrunk
Parts:
- removed C708, C711: 100n, Capacitor_SMD:C_0805_2012Metric, symbol Device:C
