File: PCB/Main Board/currentamp.kicad_sch (KiCad schematic)
At the start: 26 parts, among them U701 DG201, U702 INA828D, U703 OPA2376xxD

Commit message: Final Schematic
Parts:
- renumbered C706 to C51, C709 to C52, C701 to C53, C703 to C54, C705 to C55, C707 to C56, C710 to C57, C704 to C58, C702 to C59, JP701 to JP13, JP702 to JP14, R703 to R78, R710 to R79, R704 to R80, R701 to R81, R705 to R82, R711 to R83, R702 to R84, R706 to R85, R707 to R86, R708 to R87, R709 to R88, R712 to R89, U702 to U17, U701 to U18, U703 to U19
Other:
- note removed: "Falstad"
- note removed: "unity gain"
- company: (none) -> Harry and Yuki - EEE3 Instrumentation
- title: (none) -> Current Amplifier
- moved on the sheet: C51, C52, C53, C54, C55, C56, C57, C58, C59, JP13, JP14, R78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

Commit message: minor cleanup from the party
Parts:
- renumbered C53 to C701, C59 to C702, C54 to C703, C58 to C704, C55 to C705, C51 to C706, C56 to C707, C52 to C708, C57 to C709, JP13 to JP701, JP14 to JP702, R81 to R701, R84 to R702, R78 to R703, R80 to R704, R82 to R705, R85 to R706, R86 to R707, R87 to R708, R88 to R709, R79 to R710, R83 to R711, R89 to R712, U18 to U701, U17 to U702, U19 to U703

Commit message: :(
Parts:
- renumbered C701 to C51, C703 to C52, C705 to C53, C704 to C54, C702 to C55, C706 to C56, C708 to C57, C707 to C58, C709 to C59, JP701 to JP12, JP702 to JP13, R703 to R78, R710 to R79, R704 to R80, R701 to R81, R705 to R82, R711 to R83, R702 to R84, R706 to R85, R707 to R86, R708 to R87, R709 to R88, R712 to R89, U702 to U17, U701 to U18, U703 to U19
Connections:
- net In+: now also U17.2 (-); no longer U17.3 (+)
- net In-: now also U17.3 (+); no longer U17.2 (-)

Commit message: edits
Parts:
- removed C55: 47p, Capacitor_SMD:C_0805_2012Metric, symbol Device:C
- removed R86: 4.85k, Resistor_SMD:R_0805_2012Metric, symbol Device:R
Connections:
- net at C51.2, C52.2, C53.2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: now also R87.1
Changed lines of the file:
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@@
 	)
 	(junction
-		(at 234.95 50.8)
-		(diameter 0)
-		(color 0 0 0 0)
-	)
-	(junction
 		(at 228.6 140.97)
 		(diameter 0)
@@
 	)
 	(junction
-		(at 190.5 50.8)
-		(diameter 0)
-		(color 0 0 0 0)
-	)
-	(junction
 		(at 234.95 63.5)
 		(diameter 0)
@@
 	(wire
 		(pts
-			(xy 212.09 38.1) (xy 190.5 38.1)
-		)
-		(stroke
-			(width 0)
-			(type default)
-		)
-	)
-	(wire
-		(pts
 			(xy 152.4 31.75) (xy 152.4 44.45)
 		)
@@
 	(wire
 		(pts
-			(xy 219.71 38.1) (xy 234.95 38.1)
-		)
-		(stroke
-			(width 0)
-			(type default)
-		)
-	)
-	(wire
-		(pts
 			(xy 234.95 63.5) (xy 234.95 66.04)
 		)
@@
 	(wire
 		(pts
-			(xy 190.5 50.8) (xy 193.04 50.8)
-		)
-		(stroke
-			(width 0)
-			(type default)
-		)
-	)
-	(wire
-		(pts
 			(xy 127 44.45) (xy 127 50.8)
 		)
@@
 	(wire
 		(pts
-			(xy 187.96 50.8) (xy 190.5 50.8)
-		)
-		(stroke
-			(width 0)
-			(type default)
-		)
-	)
-	(wire
-		(pts
 			(xy 152.4 25.4) (xy 152.4 31.75)
 		)
@@
 	(wire
 		(pts
-			(xy 234.95 38.1) (xy 234.95 50.8)
-		)
-		(stroke
-			(width 0)
-			(type default)
-		)
-	)
-	(wire
-		(pts
 			(xy 234.95 50.8) (xy 234.95 53.34)
 		)
@@
 	(wire
 		(pts
-			(xy 152.4 50.8) (xy 180.34 50.8)
+			(xy 152.4 50.8) (xy 193.04 50.8)
 		)
 		(stroke
@@
 	(wire
 		(pts
-			(xy 190.5 38.1) (xy 190.5 50.8)
-		)
-		(stroke
-			(width 0)
-			(type default)
-		)
-	)
-	(wire
-		(pts
 			(xy 87.63 44.45) (xy 88.9 44.45)
 		)
@@
 	)
 	(symbol
-		(lib_id "Device:R")
-		(at 184.15 50.8 90)
-		(unit 1)
-		(exclude_from_sim no)
-		(in_bom yes)
-		(on_board yes)
-		(dnp no)
-		(fields_autoplaced yes)
-		(property "Reference" "R86"
-			(at 184.15 44.45 90)
-			(effects
-				(font
-					(size 1.27 1.27)
-				)
-			)
-		)
-		(property "Value" "4.85k"
-			(at 184.15 46.99 90)
-			(effects
-				(font
-					(size 1.27 1.27)
-				)
-			)
-		)
-		(property "Footprint" "Resistor_SMD:R_0805_2012Metric"
-			(at 184.15 52.578 90)
-			(effects
-				(font
-					(size 1.27 1.27)
-				)
-				(hide yes)
-			)
-		)
-		(property "Datasheet" "~"
-			(at 184.15 50.8 0)
-			(effects
-				(font
-					(size 1.27 1.27)
-				)
-				(hide yes)
-			)
-		)
-		(property "Description" "Resistor"
-			(at 184.15 50.8 0)
-			(effects
-				(font
-					(size 1.27 1.27)
-				)
-				(hide yes)
-			)
-		)
-		(pin "2"
-		)
-		(pin "1"
-		)
-		(instances
-			(project "Main Board"
-				(path "/20aae4b7-3fb8-4924-82e8-1e7a29a313f8/2e1ccfa8-8bce-4bb4-9d3d-716156df4d18"
-					(reference "R86")
-					(unit 1)
-				)
-			)
-		)
-	)
-	(symbol
 		(lib_id "Amplifier_Operational:OPA2376xxD")
 		(at 222.25 53.34 0)
@@
 					(unit 1)
 				)
-			)
-		)
-	)
-	(symbol
-		(lib_id "Device:C")
-		(at 215.9 38.1 90)
-		(unit 1)
-		(exclude_from_sim no)
-		(in_bom yes)
-		(on_board yes)
-		(dnp no)
-		(fields_autoplaced yes)
-		(property "Reference" "C55"
-			(at 215.9 30.48 90)
-			(effects
-				(font
-					(size 1.27 1.27)
-				)
-			)
-		)
-		(property "Value" "47p"
-			(at 215.9 33.02 90)
-			(effects
-				(font
-					(size 1.27 1.27)
-				)
-			)
-		)
-		(property "Footprint" "Capacitor_SMD:C_0805_2012Metric"
-			(at 219.71 37.1348 0)
-			(effects
-				(font
-					(size 1.27 1.27)
-				)
-				(hide yes)
-			)
-		)
-		(property "Datasheet" "~"
-			(at 215.9 38.1 0)
-			(effects
-				(font
-					(size 1.27 1.27)
-				)
-				(hide yes)
-			)
-		)
-		(property "Description" "Unpolarized capacitor"
-			(at 215.9 38.1 0)
-			(effects
-				(font
-					(size 1.27 1.27)
-				)
-				(hide yes)
-			)
-		)
-		(pin "1"
-		)
-		(pin "2"
-		)
-		(instances
-			(project "Main Board"
-				(path "/20aae4b7-3fb8-4924-82e8-1e7a29a313f8/2e1ccfa8-8bce-4bb4-9d3d-716156df4d18"
-					(reference "C55")
-					(unit 1)
-				)

Commit message: minor
Changed lines of the file:
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@@
 	(wire
 		(pts
-			(xy 234.95 50.8) (xy 247.65 50.8)
+			(xy 234.95 53.34) (xy 247.65 53.34)
 		)
 		(stroke
@@
 		(pts
 			(xy 152.4 50.8) (xy 152.4 44.45)
-		)
-		(stroke
-			(width 0)
-			(type default)
-		)
-	)
-	(wire
-		(pts
-			(xy 234.95 50.8) (xy 234.95 53.34)
 		)
 		(stroke
@@
 	(hierarchical_label "Out"
 		(shape output)
-		(at 247.65 50.8 0)
+		(at 247.65 53.34 0)
 		(effects
 			(font

Commit message: BLEH
Parts:
- renumbered C51 to C50, C52 to C51, C53 to C52, C54 to C53, C56 to C54, C57 to C55, C58 to C56, C59 to C57, JP13 to JP10, JP12 to JP9, R78 to R75, R79 to R76, R80 to R77, R81 to R78, R82 to R79, R83 to R80, R84 to R81, R85 to R82, R87 to R83, R88 to R84, R89 to R85, U17 to U16, U18 to U17, U19 to U18

Commit message: minor
Connections:
- net In+: now also U16.3 (+); no longer U16.2 (-)
- net In-: now also U16.2 (-); no longer U16.3 (+)
Changed lines of the file:
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@@
+		)
+	)
+	(hierarchical_label "In-"
+		(shape input)
+		(at 25.4 55.88 180)
+		(effects
+			(font
+				(size 1.27 1.27)
+			)
+			(justify right)
 		)
 	)
@@
 		)
 	)
-	(hierarchical_label "In-"
+	(hierarchical_label "x1"
 		(shape input)
-		(at 25.4 45.72 180)
+		(at 113.03 25.4 180)
 		(effects
 			(font
@@
 		)
 	)
-	(hierarchical_label "x1"
+	(hierarchical_label "In+"
 		(shape input)
-		(at 113.03 25.4 180)
+		(at 25.4 45.72 180)
 		(effects
 			(font
@@
 		(effects
 			(font
-				(size 1.27 1.27)
-			)
-			(justify right)
-		)
-	)
-	(hierarchical_label "In+"
-		(shape input)
-		(at 25.4 55.88 180)
-		(effects
-			(font

Commit message: sims?
Connections:
- net +1.65VA: now also U16.5 (Ref)
- no-connect marks 3 -> 2
Changed lines of the file:
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@@
-	)
-	(no_connect
-		(at 38.1 58.42)
 	)
 	(no_connect
@@
 	)
 	(symbol
+		(lib_id "More_power:+1.65VA")
+		(at 38.1 58.42 180)
+		(unit 1)
+		(exclude_from_sim no)
+		(in_bom yes)
+		(on_board yes)
+		(dnp no)
+		(property "Reference" "#PWR06"
+			(at 38.1 54.61 0)
+			(effects
+				(font
+					(size 1.27 1.27)
+				)
+				(hide yes)
+			)
+		)
+		(property "Value" "+1.65VA"
+			(at 38.1 65.532 90)
+			(effects
+				(font
+					(size 1.27 1.27)
+				)
+			)
+		)
+		(property "Footprint" ""
+			(at 38.1 58.42 0)
+			(effects
+				(font
+					(size 1.27 1.27)
+				)
+				(hide yes)
+			)
+		)
+		(property "Datasheet" ""
+			(at 38.1 58.42 0)
+			(effects
+				(font
+					(size 1.27 1.27)
+				)
+				(hide yes)
+			)
+		)
+		(property "Description" "Power symbol creates a global label with name \"+1.65VA\""
+			(at 38.1 58.42 0)
+			(effects
+				(font
+					(size 1.27 1.27)
+				)
+				(hide yes)
+			)
+		)
+		(pin "1"
+		)
+		(instances
+			(project "Main Board"
+				(path "/20aae4b7-3fb8-4924-82e8-1e7a29a313f8/2e1ccfa8-8bce-4bb4-9d3d-716156df4d18"
+					(reference "#PWR06")
+					(unit 1)
+				)
+			)
+		)
+	)
+	(symbol
 		(lib_id "Device:C")
 		(at 203.2 57.15 0)
@@
 		(on_board yes)
 		(dnp no)
-		(fields_autoplaced yes)
 		(property "Reference" "#PWR0127"
 			(at 33.02 54.61 0)
@@
 		)
 		(property "Value" "-18V"
-			(at 33.02 63.5 0)
-			(effects
-				(font
+			(at 33.02 64.008 90)
+			(effects
+				(font
