File: PCB/Main Board/dac.kicad_sch (KiCad schematic)
At the start: 0 parts

Commit message: changed to multiple feedback and minor error correction
Parts:
- added C1, C2: 100n, Capacitor_SMD:C_0805_2012Metric, symbol Device:C
- added U2, U4: OPA2376xxD, Package_SO:SOIC-8_3.9x4.9mm_P1.27mm, symbol Amplifier_Operational:OPA2376xxD
- added U3: OPA2197xD, Package_SO:SOIC-8_3.9x4.9mm_P1.27mm, symbol Amplifier_Operational:OPA2197xD
Connections:
- new net +18V: C1.1, U3.8 (V+)
- new net -18V: C2.2, U2.3 (+), U3.4 (V-)
- new net GND: C1.2, C2.1

Commit message: minor schematic changes
Parts:
- added RN?: R_Network09, Resistor_THT:R_Array_SIP10, symbol Device:R_Network09
Connections:
- net at U2.1: now also RN?.2 (R1)
- net at U2.2 (-): now also RN?.1 (common)
Other:
- moved on the sheet: U2A
Changed lines of the file:
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@@
+	(wire
+		(pts
+			(xy 102.87 96.52) (xy 102.87 99.06)
+		)
+		(stroke
+			(width 0)
+			(type default)
+		)
+	)
+	(wire
+		(pts
+			(xy 123.19 99.06) (xy 123.19 96.52)
+		)
+		(stroke
+			(width 0)
+			(type default)
+		)
+	)
+	(wire
+		(pts
+			(xy 144.78 115.57) (xy 142.24 115.57)
+		)
+		(stroke
+			(width 0)
+			(type default)
+		)
+	)
+	(wire
+		(pts
+			(xy 110.49 96.52) (xy 110.49 99.06)
+		)
+		(stroke
+			(width 0)
+			(type default)
+		)
+	)
 	(wire
 		(pts
@@
 	(wire
 		(pts
+			(xy 118.11 96.52) (xy 118.11 99.06)
+		)
+		(stroke
+			(width 0)
+			(type default)
+		)
+	)
+	(wire
+		(pts
+			(xy 115.57 96.52) (xy 115.57 99.06)
+		)
+		(stroke
+			(width 0)
+			(type default)
+		)
+	)
+	(wire
+		(pts
 			(xy 177.8 146.05) (xy 190.5 146.05)
 		)
@@
 	(wire
 		(pts
-			(xy 133.35 113.03) (xy 129.54 113.03)
-		)
-		(stroke
-			(width 0)
-			(type default)
-		)
-	)
-	(wire
-		(pts
-			(xy 129.54 101.6) (xy 129.54 113.03)
-		)
-		(stroke
-			(width 0)
-			(type default)
-		)
-	)
-	(wire
-		(pts
-			(xy 130.81 118.11) (xy 133.35 118.11)
+			(xy 144.78 96.52) (xy 144.78 115.57)
+		)
+		(stroke
+			(width 0)
+			(type default)
+		)
+	)
+	(wire
+		(pts
+			(xy 113.03 96.52) (xy 113.03 99.06)
+		)
+		(stroke
+			(width 0)
+			(type default)
+		)
+	)
+	(wire
+		(pts
+			(xy 107.95 96.52) (xy 107.95 99.06)
+		)
+		(stroke
+			(width 0)
+			(type default)
+		)
+	)
+	(wire
+		(pts
+			(xy 123.19 96.52) (xy 144.78 96.52)
+		)
+		(stroke
+			(width 0)
+			(type default)
+		)
+	)
+	(wire
+		(pts
+			(xy 127 113.03) (xy 123.19 113.03)
+		)
+		(stroke
+			(width 0)
+			(type default)
+		)
+	)
+	(wire
+		(pts
+			(xy 123.19 109.22) (xy 123.19 113.03)
+		)
+		(stroke
+			(width 0)
+			(type default)
+		)
+	)
+	(wire
+		(pts
+			(xy 105.41 96.52) (xy 105.41 99.06)
+		)
+		(stroke
+			(width 0)
+			(type default)
+		)
+	)
+	(wire
+		(pts
+			(xy 124.46 118.11) (xy 127 118.11)
+		)
+		(stroke
+			(width 0)
+			(type default)
+		)
+	)
+	(wire
+		(pts
+			(xy 120.65 99.06) (xy 120.65 96.52)
 		)
 		(stroke
@@
 	(symbol
 		(lib_id "More_power:-18V")
-		(at 130.81 118.11 90)
+		(at 124.46 118.11 90)
 		(unit 1)
 		(exclude_from_sim no)
@@
 		(fields_autoplaced yes)
 		(property "Reference" "#PWR07"
-			(at 134.62 118.11 0)
+			(at 128.27 118.11 0)
 			(effects
 				(font
@@
 		)
 		(property "Value" "-18V"
-			(at 127 118.1099 90)
+			(at 120.65 118.1099 90)
 			(effects
 				(font
@@
 		)
 		(property "Footprint" ""
-			(at 130.81 118.11 0)
+			(at 124.46 118.11 0)
 			(effects
 				(font
@@
 		)
 		(property "Datasheet" ""
-			(at 130.81 118.11 0)
+			(at 124.46 118.11 0)
 			(effects
 				(font
@@
 		)
 		(property "Description" "Power symbol creates a global label with name \"-18V\""
-			(at 130.81 118.11 0)
+			(at 124.46 118.11 0)
 			(effects
 				(font
@@
 	)
 	(symbol
+		(lib_id "Device:R_Network09")
+		(at 113.03 104.14 180)
+		(unit 1)
+		(exclude_from_sim no)
+		(in_bom yes)
+		(on_board yes)
+		(dnp no)
+		(fields_autoplaced yes)
+		(property "Reference" "RN?"
+			(at 100.33 102.6159 0)
+			(effects
+				(font
+					(size 1.27 1.27)
+				)
+				(justify left)
+			)
+		)
+		(property "Value" "R_Network09"
+			(at 100.33 105.1559 0)
+			(effects
+				(font
+					(size 1.27 1.27)
+				)
+				(justify left)
+			)
+		)
+		(property "Footprint" "Resistor_THT:R_Array_SIP10"
+			(at 98.425 104.14 90)
+			(effects
+				(font
+					(size 1.27 1.27)
+				)
+				(hide yes)
+			)
+		)
+		(property "Datasheet" "http://www.vishay.com/docs/31509/csc.pdf"
+			(at 113.03 104.14 0)
+			(effects
+				(font
+					(size 1.27 1.27)
+				)
+				(hide yes)
+			)
+		)
+		(property "Description" "9 resistor network, star topology, bussed resistors, small symbol"
+			(at 113.03 104.14 0)
+			(effects
+				(font
+					(size 1.27 1.27)
+				)
+				(hide yes)
+			)
+		)
+		(pin "10"
+		)
+		(pin "2"
+		)
+		(pin "7"
+		)
+		(pin "9"
+		)
+		(pin "5"
+		)
+		(pin "3"
+		)
+		(pin "8"
+		)
+		(pin "1"
+		)
+		(pin "6"
+		)
+		(pin "4"
+		)
+		(instances
+			(project ""
+				(path "/20aae4b7-3fb8-4924-82e8-1e7a29a313f8/3b141455-3ffc-4caf-b236-781e4c798512"
+					(reference "RN?")
+					(unit 1)
+				)
+			)
+		)
+	)
+	(symbol
 		(lib_id "Amplifier_Operational:OPA2376xxD")
-		(at 140.97 115.57 0)
+		(at 134.62 115.57 0)
 		(mirror x)
 		(unit 1)
@@
 		(dnp no)
 		(property "Reference" "U2"
-			(at 140.97 105.41 0)
+			(at 134.62 105.41 0)
 			(effects
 				(font
@@
 		)
 		(property "Value" "OPA2376xxD"
-			(at 140.97 107.95 0)
+			(at 134.62 107.95 0)
 			(effects
 				(font
@@
 		)
 		(property "Footprint" "Package_SO:SOIC-8_3.9x4.9mm_P1.27mm"
-			(at 140.97 115.57 0)
+			(at 134.62 115.57 0)
 			(effects
 				(font
@@
 		)
 		(property "Datasheet" "http://www.ti.com/lit/ds/symlink/opa376.pdf"
-			(at 140.97 115.57 0)
+			(at 134.62 115.57 0)
 			(effects
 				(font
@@
 		)
 		(property "Description" "Dual Low-Noise, Low Quiescent Current, Precision Operational Amplifier e-trim Series, SOIC-8"
-			(at 140.97 115.57 0)
-			(effects
-				(font
+			(at 134.62 115.57 0)
+			(effects
+				(font
