File: PCB/Main Board/Processor.kicad_sch (KiCad schematic)
At the start: 21 parts, among them J901 USB_C_Receptacle_USB2.0_16P, U901 USBLC6-2SC6

Commit message: footprints and minor
Parts:
- gave numbers to parts that had none: 19
- renumbered J901 to J5, U901 to U1

Commit message: footprints and stm wiring
Connections:
- net IAmp.AC_100: now also U3.2 (PC13)
- net IAmp.AC_10k: now also U3.4 (PC15)
- net IAmp.AC_1k: now also U3.3 (PC14)
- net IAmp.AC_EN: now also U3.53 (PC12)
- net IAmp.x1: now also U3.40 (PC9)
- net IAmp.x3: now also U3.51 (PC10)
- net IAmp./4: now also U3.39 (PC8)
- net IAmp.~{x100}: now also U3.52 (PC11)
- net Source./10: now also U3.57 (PB5)
- net Source.~{x4}: now also U3.56 (PB4)
- net VAmp.AC_100: now also U3.25 (PC5)
- net VAmp.AC_10k: now also U3.38 (PC7)
- net VAmp.AC_1k: now also U3.37 (PC6)
- net VAmp.AC_EN: now also U3.24 (PC4)
- net VAmp.x1: now also U3.9 (PC1)
- net VAmp.x3: now also U3.10 (PC2)
- net VAmp./4: now also U3.8 (PC0)
- net VAmp.~{x100}: now also U3.11 (PC3)
- net at U3.29 (PB10): now also U2.3 (I3)
- net at U3.33 (PB12): now also U2.4 (I4)
- net at U3.34 (PB13): now also U2.5 (I5)
- net at U3.35 (PB14): now also U2.6 (I6)
- net at U3.36 (PB15): now also U2.7 (I7)
- net R_SEL_432k: now reaches U3.58 (PB6)
- net R_SEL_100k: now reaches U3.59 (PB7)
- net at U3.61 (PB8): now also U2.1 (I1)
- net at U3.62 (PB9): now also U2.2 (I2)
- net SIG_SOURCE: now reaches U2.11 (O6)
- net DC_INT_ISO: now reaches U2.12 (O5)
- net R_SEL_10: now reaches U2.13 (O4)
- net R_SEL_100: now reaches U2.14 (O3)
- net R_SEL_1k: now reaches U2.15 (O2)
- net R_SEL_10k: now reaches U2.16 (O1)
- no-connect marks 3 -> 20
Other:
- note added: "can shufffle these after layout starts"
- moved on the sheet: C1, C2, C3, C4, C5, C6, C7, C8, C9, JP1, R1, R2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

Commit message: relays and layout begin
Parts:
- added FL1: Filter_EMI_CommonMode, Inductor_SMD:L_CommonModeChoke_Coilcraft_0603USB, symbol Device:Filter_EMI_CommonMode
- added JP25, JP26: SolderJumper_2_Open, Jumper:SolderJumper-2_P1.3mm_Open_RoundedPad1.0x1.5mm, symbol Jumper:SolderJumper_2_Open
- C1, C2, C3, C4, C5, C6, C7, C8, C9: footprint (none) -> Capacitor_SMD:C_0805_2012Metric
- R1, R2, R3, R4: footprint (none) -> Resistor_SMD:R_0805_2012Metric
- R5: footprint Resistor_SMD:R_0603_1608Metric -> Resistor_SMD:R_0805_2012Metric
- R6, R7: footprint Capacitor_SMD:C_0603_1608Metric -> Resistor_SMD:R_0805_2012Metric
- U3: renamed from U2; footprint (none) -> Package_SO:SOIC-16_3.9x9.9mm_P1.27mm
- renumbered U3 to U2
Connections:
- net USB_DN: now also FL1.2, JP25.2 (B); no longer U1.6 (I/O1)
- net USB_DP: now also FL1.4, JP26.2 (B); no longer U1.4 (I/O2)
- new net: FL1.1, JP25.1 (A), U1.6 (I/O1)
- new net: FL1.3, JP26.1 (A), U1.4 (I/O2)
Other:
- note added: "flyback included on psu"
- note added: "no crystal?"

Commit message: minor and layout
Parts:
- added C? (x2): 33p, Capacitor_SMD:C_0805_2012Metric, symbol Device:C
- added Y1: 8MHz, Crystal:Crystal_SMD_5032-2Pin_5.0x3.2mm, symbol Device:Crystal
Connections:
- net GND: now also C?.2, C?.2
- net XTAL1: now reaches U2.5 (PH0)
- net XTAL1: now also C?.1, Y1.2
- net XTAL2: now reaches U2.6 (PH1)
- net XTAL2: now also C?.1, Y1.1
- no-connect marks 20 -> 23
Other:
- note removed: "can shufffle these after layout starts"
- note removed: "no crystal?"

Commit message: amplifer floorplan and relay footprint + minor
Parts:
- removed JP1: SolderJumper_2_Bridged, symbol Jumper:SolderJumper_2_Bridged
- added JP?: SolderJumper_2_Bridged, Jumper:SolderJumper-2_P1.3mm_Bridged_RoundedPad1.0x1.5mm, symbol Jumper:SolderJumper_2_Bridged
- gave numbers to parts that had none: 2
Connections:
- net BOOT0: now also JP?.1 (A)
- net at U2.60 (BOOT0): now also JP?.2 (B)
Other:
- moved on the sheet: C1, C2, C3, C4, C40, C43, C5, C6, C7, C8, C9, R1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

Commit message: :ghost:
Parts:
- gave numbers to parts that had none: 1
- renumbered C40 to C201, C43 to C202, C3 to C203, C2 to C204, C4 to C205, C5 to C206, C6 to C207, C7 to C208, C1 to C209, C8 to C210, C9 to C211, FL1 to FL201, J5 to J201, JP25 to JP201, JP26 to JP202, R5 to R201, R6 to R202, R7 to R203, R1 to R204, R2 to R205, R3 to R206, R4 to R207, U1 to U201, U2 to U202, U3 to U203, Y1 to Y201

Commit message: Layout progress
Connections:
- net IAmp.In renamed IAmp.Out
- net VAmp.In renamed VAmp.Out
Changed lines of the file:
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@@
 		)
 	)
-	(hierarchical_label "VAmp.In"
+	(hierarchical_label "VAmp.Out"
 		(shape input)
 		(at 207.01 40.64 0)
@@
 		)
 	)
-	(hierarchical_label "IAmp.In"
+	(hierarchical_label "IAmp.Out"
 		(shape input)
 		(at 207.01 43.18 0)

Commit message: :-1:
Connections:
- net DC_INT_ISO: now also U203.11 (O6); no longer U203.12 (O5)
- net R_SEL_10: now also U203.12 (O5); no longer U203.13 (O4)
- net R_SEL_100: now also U203.13 (O4); no longer U203.14 (O3)
- net R_SEL_100k: now also U203.16 (O1); no longer U202.59 (PB7)
- net R_SEL_10k: now also U203.15 (O2); no longer U203.16 (O1)
- net R_SEL_1k: now also U203.14 (O3); no longer U203.15 (O2)
- net SIG_SOURCE: now also U203.10 (O7); no longer U203.11 (O6)
- no-connect marks 23 -> 22
Changed lines of the file:
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@@
-	)
-	(no_connect
-		(at 243.84 119.38)
 	)
 	(no_connect
@@
 	(wire
 		(pts
+			(xy 243.84 119.38) (xy 245.11 119.38)
+		)
+		(stroke
+			(width 0)
+			(type default)
+		)
+	)
+	(wire
+		(pts
 			(xy 245.11 111.76) (xy 243.84 111.76)
 		)
@@
 		(pts
 			(xy 110.49 140.97) (xy 110.49 138.43)
-		)
-		(stroke
-			(width 0)
-			(type default)
-		)
-	)
-	(wire
-		(pts
-			(xy 208.28 101.6) (xy 207.01 101.6)
 		)
 		(stroke
@@
 	(hierarchical_label "R_SEL_10k"
 		(shape output)
-		(at 245.11 104.14 0)
+		(at 245.11 106.68 0)
 		(effects
 			(font
@@
 	(hierarchical_label "R_SEL_100"
 		(shape output)
-		(at 245.11 109.22 0)
+		(at 245.11 111.76 0)
 		(effects
 			(font
@@
 	(hierarchical_label "SIG_SOURCE"
 		(shape output)
-		(at 245.11 116.84 0)
+		(at 245.11 119.38 0)
 		(effects
 			(font
@@
 	(hierarchical_label "R_SEL_100k"
 		(shape output)
-		(at 208.28 101.6 0)
+		(at 245.11 104.14 0)
 		(effects
 			(font
@@
 	(hierarchical_label "R_SEL_1k"
 		(shape output)
-		(at 245.11 106.68 0)
+		(at 245.11 109.22 0)
 		(effects
 			(font
@@
 	(hierarchical_label "DC_INT_ISO"
 		(shape output)
+		(at 245.11 116.84 0)
+		(effects
+			(font
+				(size 1.27 1.27)
+			)
+			(justify left)
+		)
+	)
+	(hierarchical_label "R_SEL_10"
+		(shape output)
 		(at 245.11 114.3 0)
 		(effects
 			(font
-				(size 1.27 1.27)
-			)
-			(justify left)
-		)
-	)
-	(hierarchical_label "R_SEL_10"
-		(shape output)
-		(at 245.11 111.76 0)
-		(effects
-			(font
