File: PCB/Main Board/Processor.kicad_sch (KiCad schematic)
At the start: 27 parts, among them J201 USB_C_Receptacle_USB2.0_16P, U201 USBLC6-2SC6, U202 STM32F446RETx, U203 ULN2003, Y201 8MHz

Commit message: minor schematic changes
Parts:
- added R?: 10k, Resistor_SMD:R_0805_2012Metric, symbol Device:R
- added SW? (x2): SW_Push, Button_Switch_THT:SW_PUSH_6mm, symbol Switch:SW_Push
Connections:
- net +3.3V: now also SW?.2, SW?.2
- net BOOT0: now also SW?.1
- net GND: now also R?.2
- net SW1: now reaches U202.16 (PA2)
- net SW1: now also R?.1, SW?.1
- net DAC_0: now reaches U202.22 (PA6)
- net DAC_1: now reaches U202.23 (PA7)
- net DAC_2: now reaches U202.41 (PA8)
- net DAC_3: now reaches U202.42 (PA9)
- net DAC_4: now reaches U202.43 (PA10)
- net DAC_5: now reaches U202.44 (PA11)
- net DAC_6: now reaches U202.45 (PA12)
- net DAC_7: now reaches U202.46 (PA13)
- net R_SEL_432k: no longer names the net of U202.58 (PB6)
- no-connect marks 22 -> 13

Commit message: sorry i fell asleep b4 layout
Parts:
- gave numbers to parts that had none: 3
- renumbered C209 to C201, C204 to C202, C201 to C203, C202 to C204, C203 to C205, C205 to C206, C206 to C207, C207 to C208, C208 to C209, JP203 to JP202, JP202 to JP203
Connections:
- no-connect marks 13 -> 15
Other:
- moved on the sheet: C203, C204, C205, C206, C207, C208, C209, C210, C211, JP202, U202, U203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

Commit message: HI
Parts:
- renumbered C203 to C201, C204 to C202, C205 to C203, C202 to C204, C206 to C205, C207 to C206, C208 to C207, C209 to C208, C201 to C209, JP203 to JP202, JP202 to JP203, R208 to R204, R204 to R205, R205 to R206, R206 to R207, R207 to R208, SW202 to SW201, SW201 to SW202

Commit message: yup
Parts:
- removed U203: ULN2003, Package_SO:SOIC-16_3.9x9.9mm_P1.27mm, symbol Transistor_Array:ULN2003
Connections:
- net DC_INT_ISO: now also U202.35 (PB14)
- net R_SEL_10: now also U202.34 (PB13)
- net R_SEL_100: now also U202.33 (PB12)
- net R_SEL_100k: now also U202.61 (PB8)
- net R_SEL_10k: now also U202.62 (PB9)
- net R_SEL_1k: now also U202.29 (PB10)
- net SIG_SOURCE: now also U202.36 (PB15)
- no-connect marks 15 -> 14
Other:
- note removed: "flyback included on psu"

Commit message: sig source finished
Parts:
- renumbered C209 to C201, C204 to C202, C201 to C203, C202 to C204, C203 to C205, C205 to C206, C206 to C207, C207 to C208, C208 to C209, JP203 to JP202, JP202 to JP203, R205 to R204, R206 to R205, R207 to R206, R208 to R207, R204 to R208, SW202 to SW201, SW201 to SW202

Commit message: hello
Parts:
- renumbered C203 to C201, C204 to C202, C205 to C203, C202 to C204, C206 to C205, C207 to C206, C208 to C207, C209 to C208, C201 to C209, JP203 to JP202, JP202 to JP203, R208 to R204, R204 to R205, R205 to R206, R206 to R207, R207 to R208, SW202 to SW201, SW201 to SW202
Connections:
- net DC_INT_ISO: now also U202.56 (PB4); no longer U202.35 (PB14)
- net IAmp.AC_100: no longer U202.2 (PC13)
- net IAmp.AC_10k: no longer U202.4 (PC15)
- net IAmp.AC_1k: no longer U202.3 (PC14)
- net IAmp.AC_EN: no longer U202.53 (PC12)
- net IAmp.Out: now also U202.9 (PC1); no longer U202.15 (PA1)
- net IAmp.x1: no longer U202.40 (PC9)
- net IAmp.x3: no longer U202.51 (PC10)
- net IAmp./4: no longer U202.39 (PC8)
- net IAmp.~{x100}: no longer U202.52 (PC11)
- net R_SEL_10: now also U202.62 (PB9); no longer U202.34 (PB13)
- net R_SEL_100: now also U202.61 (PB8); no longer U202.33 (PB12)
- net R_SEL_100k: now also U202.57 (PB5); no longer U202.61 (PB8)
- net R_SEL_10k: now also U202.59 (PB7); no longer U202.62 (PB9)
- net R_SEL_1k: now also U202.58 (PB6); no longer U202.29 (PB10)
- net SIG_SOURCE: no longer U202.36 (PB15)
- net SW1: no longer U202.16 (PA2)
- net Source./10: no longer U202.57 (PB5)
- net Source.~{x4}: no longer U202.56 (PB4)
- net VAmp.AC_100: no longer U202.25 (PC5)
- net VAmp.AC_10k: no longer U202.38 (PC7)
- net VAmp.AC_1k: no longer U202.37 (PC6)
- net VAmp.AC_EN: no longer U202.24 (PC4)
- net VAmp.Out: now also U202.17 (PA3); no longer U202.14 (PA0)
- net VAmp.x1: no longer U202.9 (PC1)
- net VAmp.x3: no longer U202.10 (PC2)
- net VAmp./4: no longer U202.8 (PC0)
- net VAmp.~{x100}: no longer U202.11 (PC3)
- no-connect marks 14 -> 11
Other:
- note added: "ADC1_IN11"
- note added: "ADC2_IN3"
- note removed: "ADC1_IN0"
- note removed: "ADC2_IN1"

Commit message: :(
Connections:
- net DC_INT_ISO: now also U202.49 (PA14); no longer U202.56 (PB4)
- net IAmp.AC_100: now also U202.58 (PB6)
- net IAmp.AC_10k: now also U202.56 (PB4)
- net IAmp.AC_1k: now also U202.57 (PB5)
- net IAmp.AC_EN: now also U202.55 (PB3)
- net R_SEL_10: now also U202.54 (PD2); no longer U202.62 (PB9)
- net R_SEL_100: now also U202.53 (PC12); no longer U202.61 (PB8)
- net R_SEL_100k: now also U202.50 (PA15); no longer U202.57 (PB5)
- net R_SEL_10k: now also U202.52 (PC11); no longer U202.59 (PB7)
- net R_SEL_1k: now also U202.51 (PC10); no longer U202.58 (PB6)
- no-connect marks 11 -> 4

Commit message: asdfjkhhjk
Connections:
- net IAmp.x1: now also U202.61 (PB8)
- net IAmp.x3: now also U202.59 (PB7)
- net IAmp./4: now also U202.8 (PC0)
- net IAmp.~{x100}: now also U202.62 (PB9)
Changed lines of the file:
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@@
 	(hierarchical_label "IAmp.x1"
 		(shape output)
-		(at 119.38 88.9 180)
-		(effects
-			(font
-				(size 1.27 1.27)
-			)
-			(justify right)
+		(at 190.5 104.14 0)
+		(effects
+			(font
+				(size 1.27 1.27)
+			)
+			(justify left)
 		)
 	)
@@
 	(hierarchical_label "IAmp.{slash}4"
 		(shape output)
-		(at 119.38 86.36 180)
+		(at 142.24 63.5 180)
 		(effects
 			(font
@@
 	(hierarchical_label "IAmp.x3"
 		(shape output)
-		(at 119.38 91.44 180)
-		(effects
-			(font
-				(size 1.27 1.27)
-			)
-			(justify right)
+		(at 190.5 101.6 0)
+		(effects
+			(font
+				(size 1.27 1.27)
+			)
+			(justify left)
 		)
 	)
@@
 	(hierarchical_label "IAmp.~{x100}"
 		(shape output)
-		(at 119.38 93.98 180)
-		(effects
-			(font
-				(size 1.27 1.27)
-			)
-			(justify right)
-		)
-	)
+		(at 190.5 106.68 0)
+		(effects
+			(font
+				(size 1.27 1.27)
+			)
+			(justify left)
+		)
+	)
