File: PCB/Main Board/Processor.kicad_sch (KiCad schematic)
At the start: 25 parts, among them J6 USB_C_Receptacle_USB2.0_16P, J7 Conn_01x05_Pin, SW1 SW_Push, U1 USBLC6-2SC6, U2 STM32F446RETx, Y1 8MHz

Commit message: bleh
Other:
- note added: "FIX IBIASMON"
Changed lines of the file:
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@@
+		)
+	)
+	(text "FIX IBIASMON\n"
+		(exclude_from_sim no)
+		(at 114.3 76.2 0)
+		(effects
+			(font
+				(size 1.27 1.27)
+			)
 		)
 	)

Commit message: :(
Parts:
- removed FL1: Filter_EMI_CommonMode, Inductor_SMD:L_CommonModeChoke_Coilcraft_0603USB, symbol Device:Filter_EMI_CommonMode
- removed JP1, JP2, JP3: SolderJumper_2_Open, Jumper:SolderJumper-2_P1.3mm_Open_RoundedPad1.0x1.5mm, symbol Jumper:SolderJumper_2_Open
- removed U1: USBLC6-2SC6, Package_TO_SOT_SMD:SOT-23-6, symbol Power_Protection:USBLC6-2SC6
Connections:
- net GND: now also J6.S1 (SHIELD)
- net IAmp.AC_100: now also U2.8 (PC0); no longer U2.59 (PB7)
- net IAmp.AC_10k: now also U2.3 (PC14); no longer U2.57 (PB5)
- net IAmp.AC_1k: now also U2.4 (PC15); no longer U2.58 (PB6)
- net IAmp.AC_EN: now also U2.2 (PC13); no longer U2.56 (PB4)
- net IAmp.x1: now also U2.56 (PB4); no longer U2.2 (PC13)
- net IAmp.x3: now also U2.57 (PB5); no longer U2.3 (PC14)
- net IAmp./4: now also U2.58 (PB6); no longer U2.4 (PC15)
- net IAmp.~{x100}: now also U2.59 (PB7); no longer U2.8 (PC0)
- net Source./10: now also U2.27 (PB1); no longer U2.26 (PB0)
- net Source.~{x4}: now also U2.26 (PB0); no longer U2.27 (PB1)
- net USB_DN: now also J6.A7 (D-), J6.B7 (D-)
- net USB_DP: now also J6.A6 (D+), J6.B6 (D+)
- no-connect marks 14 -> 13

Commit message: :(
Parts:
- added J?: Conn_01x03_Pin, Connector_PinHeader_2.54mm:PinHeader_1x03_P2.54mm_Vertical, symbol Connector:Conn_01x03_Pin
Connections:
- net GND: now also J?.1 (Pin_1)
- net IAmp./4: now also U2.61 (PB8); no longer U2.58 (PB6)
- net IAmp.~{x100}: now also U2.62 (PB9); no longer U2.59 (PB7)
- new net USART_RX: J?.3 (Pin_3), U2.59 (PB7)
- new net USART_TX: J?.2 (Pin_2), U2.58 (PB6)
- no-connect marks 13 -> 11
Changed lines of the file:
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@@
-	)
-	(no_connect
-		(at 186.69 106.68)
 	)
 	(no_connect
@@
 		(at 161.29 33.02)
 	)
-	(no_connect
-		(at 186.69 104.14)
-	)
 	(wire
 		(pts
@@
 		)
 	)
+	(label "USART_RX"
+		(at 177.8 144.78 180)
+		(effects
+			(font
+				(size 1.27 1.27)
+			)
+			(justify right)
+		)
+	)
 	(label "USB_CC2"
 		(at 52.07 80.01 0)
@@
 		)
 	)
+	(label "USART_RX"
+		(at 186.69 101.6 0)
+		(effects
+			(font
+				(size 1.27 1.27)
+			)
+			(justify left)
+		)
+	)
+	(label "USART_TX"
+		(at 186.69 99.06 0)
+		(effects
+			(font
+				(size 1.27 1.27)
+			)
+			(justify left)
+		)
+	)
 	(label "USB_DP"
 		(at 26.67 92.71 180)
@@
 		)
 	)
+	(label "USART_TX"
+		(at 177.8 147.32 180)
+		(effects
+			(font
+				(size 1.27 1.27)
+			)
+			(justify right)
+		)
+	)
 	(hierarchical_label "R_SEL_10k"
 		(shape output)
@@
 	(hierarchical_label "IAmp.{slash}4"
 		(shape output)
-		(at 186.69 99.06 0)
+		(at 186.69 104.14 0)
 		(effects
 			(font
@@
 	(hierarchical_label "IAmp.~{x100}"
 		(shape output)
-		(at 186.69 101.6 0)
+		(at 186.69 106.68 0)
 		(effects
 			(font
@@
 				(path "/20aae4b7-3fb8-4924-82e8-1e7a29a313f8/e5018641-2f50-45af-a491-5d0cd121e7a0"
 					(reference "#PWR024")
+					(unit 1)
+				)
+			)
+		)
+	)
+	(symbol
+		(lib_id "power:GND")
+		(at 177.8 149.86 270)
+		(unit 1)
+		(exclude_from_sim no)
+		(in_bom yes)
+		(on_board yes)
+		(dnp no)
+		(property "Reference" "#PWR09"
+			(at 171.45 149.86 0)
+			(effects
+				(font
+					(size 1.27 1.27)
+				)
+				(hide yes)
+			)
+		)
+		(property "Value" "GND"
+			(at 172.72 149.86 90)
+			(effects
+				(font
+					(size 1.27 1.27)
+				)
+			)
+		)
+		(property "Footprint" ""
+			(at 177.8 149.86 0)
+			(effects
+				(font
+					(size 1.27 1.27)
+				)
+				(hide yes)
+			)
+		)
+		(property "Datasheet" ""
+			(at 177.8 149.86 0)
+			(effects
+				(font
+					(size 1.27 1.27)
+				)
+				(hide yes)
+			)
+		)
+		(property "Description" ""
+			(at 177.8 149.86 0)
+			(effects
+				(font
+					(size 1.27 1.27)
+				)
+				(hide yes)
+			)
+		)
+		(pin "1"
+		)
+		(instances
+			(project "Main Board"
+				(path "/20aae4b7-3fb8-4924-82e8-1e7a29a313f8/e5018641-2f50-45af-a491-5d0cd121e7a0"
+					(reference "#PWR09")
 					(unit 1)
 				)
@@
 					(unit 1)
 				)
+			)
+		)
+	)
+	(symbol
+		(lib_id "Connector:Conn_01x03_Pin")
+		(at 182.88 147.32 180)
+		(unit 1)
+		(exclude_from_sim no)
+		(in_bom yes)
+		(on_board yes)
+		(dnp no)
+		(fields_autoplaced yes)
+		(property "Reference" "J?"
+			(at 184.15 146.0499 0)
+			(effects
+				(font
+					(size 1.27 1.27)
+				)
+				(justify right)
+			)
+		)
+		(property "Value" "Conn_01x03_Pin"
+			(at 184.15 148.5899 0)
+			(effects
+				(font
+					(size 1.27 1.27)
+				)
+				(justify right)
+			)
+		)
+		(property "Footprint" "Connector_PinHeader_2.54mm:PinHeader_1x03_P2.54mm_Vertical"
+			(at 182.88 147.32 0)
+			(effects
+				(font
+					(size 1.27 1.27)
+				)
+				(hide yes)
+			)
+		)
+		(property "Datasheet" "~"
+			(at 182.88 147.32 0)
+			(effects
+				(font
+					(size 1.27 1.27)
+				)
+				(hide yes)
+			)
+		)
+		(property "Description" "Generic connector, single row, 01x03, script generated"
+			(at 182.88 147.32 0)
+			(effects
+				(font
+					(size 1.27 1.27)
+				)
+				(hide yes)
+			)
+		)
+		(pin "1"
+		)
+		(pin "2"
+		)
+		(pin "3"
+		)
+		(instances
+			(project ""
+				(path "/20aae4b7-3fb8-4924-82e8-1e7a29a313f8/e5018641-2f50-45af-a491-5d0cd121e7a0"
+					(reference "J?")
+					(unit 1)
+				)

Commit message: ready to krill myself
Parts:
- gave numbers to parts that had none: 1
Connections:
- net USB_DN: now also U2.35 (PB14)
- net USB_DP: now also U2.36 (PB15)
- no-connect marks 11 -> 9
Changed lines of the file:
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@@
 	)
 	(no_connect
-		(at 186.69 116.84)
-	)
-	(no_connect
-		(at 186.69 119.38)
-	)
-	(no_connect
 		(at 186.69 109.22)
 	)
@@
 		)
 	)
+	(label "USB_DP"
+		(at 186.69 119.38 0)
+		(effects
+			(font
+				(size 1.27 1.27)
+			)
+			(justify left)
+		)
+	)
+	(label "USB_DN"
+		(at 186.69 116.84 0)
+		(effects
+			(font
+				(size 1.27 1.27)
+			)
+			(justify left)
+		)
+	)
 	(label "XTAL1"
 		(at 146.05 50.8 180)
@@
 		(dnp no)
 		(fields_autoplaced yes)
-		(property "Reference" "J?"
+		(property "Reference" "J10"
 			(at 184.15 146.0499 0)
 			(effects
@@
 			(project ""
 				(path "/20aae4b7-3fb8-4924-82e8-1e7a29a313f8/e5018641-2f50-45af-a491-5d0cd121e7a0"
-					(reference "J?")
+					(reference "J10")
 					(unit 1)
 				)

Commit message: minor
Parts:
- added J?: Conn_01x03_Pin, Connector_PinHeader_2.54mm:PinHeader_1x03_P2.54mm_Vertical, symbol Connector:Conn_01x03_Pin
Connections:
- net GND: now also J?.1 (Pin_1)
- net USB_DN: now also J?.2 (Pin_2)
- net USB_DP: now also J?.3 (Pin_3)
Changed lines of the file:
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@@
 	(wire
 		(pts
+			(xy 77.47 40.64) (xy 82.55 40.64)
+		)
+		(stroke
+			(width 0)
+			(type default)
+		)
+	)
+	(wire
+		(pts
 			(xy 49.53 43.18) (xy 49.53 45.72)
 		)
@@
 	(wire
 		(pts
+			(xy 82.55 45.72) (xy 80.01 45.72)
+		)
+		(stroke
+			(width 0)
+			(type default)
+		)
+	)
+	(wire
+		(pts
 			(xy 60.96 167.64) (xy 63.5 167.64)
 		)
@@
 	(wire
 		(pts
+			(xy 77.47 43.18) (xy 82.55 43.18)
+		)
+		(stroke
+			(width 0)
+			(type default)
+		)
+	)
+	(wire
+		(pts
 			(xy 72.39 130.81) (xy 72.39 128.27)
 		)
@@
 	(wire
 		(pts
+			(xy 80.01 45.72) (xy 80.01 48.26)
+		)
+		(stroke
+			(width 0)
+			(type default)
+		)
+	)
+	(wire
+		(pts
 			(xy 97.79 128.27) (xy 97.79 130.81)
 		)
@@
 		)
 	)
+	(label "USB_DN"
+		(at 77.47 43.18 180)
+		(effects
+			(font
+				(size 1.27 1.27)
+			)
+			(justify right bottom)
+		)
+	)
 	(label "~{RST}"
 		(at 142.24 152.4 180)
@@
 		)
 	)
+	(label "USB_DP"
+		(at 77.47 40.64 180)
+		(effects
+			(font
+				(size 1.27 1.27)
+			)
+			(justify right bottom)
+		)
+	)
 	(label "BOOT0"
 		(at 116.84 128.27 0)
@@
 	)
 	(symbol
+		(lib_id "Connector:Conn_01x03_Pin")
+		(at 87.63 43.18 180)
+		(unit 1)
+		(exclude_from_sim no)
+		(in_bom yes)
+		(on_board yes)
+		(dnp no)
+		(property "Reference" "J?"
+			(at 88.9 43.1799 0)
+			(effects
+				(font
+					(size 1.27 1.27)
+				)
+				(justify right)
+			)
+		)
+		(property "Value" "Conn_01x03_Pin"
+			(at 88.9 44.4499 0)
+			(effects
+				(font
+					(size 1.27 1.27)
+				)
+				(justify right)
+				(hide yes)
+			)
+		)
+		(property "Footprint" "Connector_PinHeader_2.54mm:PinHeader_1x03_P2.54mm_Vertical"
+			(at 87.63 43.18 0)
+			(effects
+				(font
+					(size 1.27 1.27)
+				)
+				(hide yes)
+			)
+		)
+		(property "Datasheet" "~"
+			(at 87.63 43.18 0)
+			(effects
+				(font
+					(size 1.27 1.27)
+				)
+				(hide yes)
+			)
+		)
+		(property "Description" "Generic connector, single row, 01x03, script generated"
+			(at 87.63 43.18 0)
+			(effects
+				(font
+					(size 1.27 1.27)
+				)
+				(hide yes)
+			)
+		)
+		(pin "1"
+		)
+		(pin "2"
+		)
+		(pin "3"
+		)
+		(instances
+			(project "Main Board"
+				(path "/20aae4b7-3fb8-4924-82e8-1e7a29a313f8/e5018641-2f50-45af-a491-5d0cd121e7a0"
+					(reference "J?")
+					(unit 1)
+				)
+			)
+		)
+	)
+	(symbol
 		(lib_id "power:+3.3V")
 		(at 88.9 168.91 0)
@@
 		(on_board yes)
 		(dnp no)
-		(fields_autoplaced yes)
 		(property "Reference" "J10"
-			(at 184.15 146.0499 0)
+			(at 184.15 147.3199 0)
 			(effects
 				(font
@@
 				)
 				(justify right)
+				(hide yes)
 			)
 		)
@@
 					(unit 1)
 				)
+			)
+		)
+	)
+	(symbol
+		(lib_name "GND_1")
+		(lib_id "power:GND")
+		(at 80.01 48.26 0)
+		(unit 1)
+		(exclude_from_sim no)
+		(in_bom yes)
+		(on_board yes)
+		(dnp no)
+		(fields_autoplaced yes)
+		(property "Reference" "#PWR0201"
+			(at 80.01 54.61 0)
+			(effects
+				(font
+					(size 1.27 1.27)
+				)
+				(hide yes)
+			)
+		)
+		(property "Value" "GND"
+			(at 80.01 53.34 0)
+			(effects
+				(font
+					(size 1.27 1.27)
+				)
+			)
+		)
+		(property "Footprint" ""
+			(at 80.01 48.26 0)
+			(effects
+				(font
+					(size 1.27 1.27)
+				)
+				(hide yes)
+			)
+		)
+		(property "Datasheet" ""
+			(at 80.01 48.26 0)
+			(effects
+				(font
+					(size 1.27 1.27)
+				)
+				(hide yes)
+			)
+		)
+		(property "Description" "Power symbol creates a global label with name \"GND\" , ground"
+			(at 80.01 48.26 0)
+			(effects
+				(font
+					(size 1.27 1.27)
+				)
+				(hide yes)
+			)
+		)
+		(pin "1"
+		)
+		(instances
+			(project "Main Board"
+				(path "/20aae4b7-3fb8-4924-82e8-1e7a29a313f8/e5018641-2f50-45af-a491-5d0cd121e7a0"
+					(reference "#PWR0201")
+					(unit 1)
+				)

Commit message: BLEH
Parts:
- removed J6: USB_C_Receptacle_USB2.0_16P, Connector_USB:USB_C_Receptacle_GCT_USB4110, symbol Connector:USB_C_Receptacle_USB2.0_16P
- removed R2, R3: 5.1k, Resistor_SMD:R_0805_2012Metric, symbol Device:R
- gave numbers to parts that had none: 1
- renumbered J7 to J8, J10 to J9, U2 to U1
Connections:
- no-connect marks 9 -> 6

Commit message: tired
Connections:
- net VAmp.AC_100: now also U1.14 (PA0); no longer U1.11 (PC3)
- net VAmp.AC_10k: now also U1.15 (PA1); no longer U1.14 (PA0)
- net VAmp.AC_EN: now also U1.16 (PA2); no longer U1.15 (PA1)
- new net I_B_MON: U1.11 (PC3)
- no-connect marks 6 -> 5
Other:
- moved on the sheet: J7, R1
Changed lines of the file:
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@@
 	)
 	(no_connect
-		(at 186.69 45.72)
-	)
-	(no_connect
 		(at 161.29 33.02)
 	)
 	(wire
 		(pts
-			(xy 77.47 40.64) (xy 82.55 40.64)
+			(xy 83.82 41.91) (xy 88.9 41.91)
 		)
 		(stroke
@@
 	(wire
 		(pts
-			(xy 82.55 45.72) (xy 80.01 45.72)
+			(xy 88.9 46.99) (xy 86.36 46.99)
 		)
 		(stroke
@@
 	(wire
 		(pts
-			(xy 26.67 90.17) (xy 26.67 92.71)
+			(xy 63.5 48.26) (xy 63.5 50.8)
 		)
 		(stroke
@@
 	(wire
 		(pts
-			(xy 26.67 82.55) (xy 26.67 80.01)
+			(xy 63.5 40.64) (xy 63.5 38.1)
 		)
 		(stroke
@@
 	(wire
 		(pts
-			(xy 77.47 43.18) (xy 82.55 43.18)
+			(xy 83.82 44.45) (xy 88.9 44.45)
 		)
 		(stroke
@@
 	(wire
 		(pts
-			(xy 80.01 45.72) (xy 80.01 48.26)
+			(xy 86.36 46.99) (xy 86.36 49.53)
 		)
 		(stroke
@@
 	)
 	(label "USB_DN"
-		(at 77.47 43.18 180)
+		(at 83.82 44.45 180)
 		(effects
 			(font
@@
 	)
 	(label "USB_DP"
-		(at 26.67 92.71 180)
+		(at 63.5 50.8 180)
 		(effects
 			(font
@@
 	)
 	(label "USB_DP"
-		(at 77.47 40.64 180)
+		(at 83.82 41.91 180)
 		(effects
 			(font
@@
 	(hierarchical_label "VAmp.AC_10k"
 		(shape output)
-		(at 186.69 40.64 0)
+		(at 186.69 43.18 0)
 		(effects
 			(font
@@
 		)
 	)
+	(hierarchical_label "I_B_MON"
+		(shape input)
+		(at 146.05 71.12 180)
+		(effects
+			(font
+				(size 1.27 1.27)
+			)
+			(justify right)
+		)
+	)
 	(hierarchical_label "IAmp.AC_1k"
 		(shape output)
@@
 	(hierarchical_label "VAmp.AC_100"
 		(shape output)
-		(at 146.05 71.12 180)
+		(at 186.69 40.64 0)
 		(effects
 			(font
 				(size 1.27 1.27)
 			)
-			(justify right)
+			(justify left)
 		)
 	)
@@
 	(hierarchical_label "VAmp.AC_EN"
 		(shape output)
-		(at 186.69 43.18 0)
+		(at 186.69 45.72 0)
 		(effects
 			(font
@@
 	(symbol
 		(lib_id "Connector:Conn_01x03_Pin")
-		(at 87.63 43.18 180)
+		(at 93.98 44.45 180)
 		(unit 1)
 		(exclude_from_sim no)
@@
 		(dnp no)
 		(property "Reference" "J7"
-			(at 88.9 43.1799 0)
+			(at 95.25 44.4499 0)
 			(effects
 				(font
@@
 		)
 		(property "Value" "Conn_01x03_Pin"
-			(at 88.9 44.4499 0)
+			(at 95.25 45.7199 0)
 			(effects
 				(font
@@
 		)
 		(property "Footprint" "Connector_PinHeader_2.54mm:PinHeader_1x03_P2.54mm_Vertical"
-			(at 87.63 43.18 0)
+			(at 93.98 44.45 0)
 			(effects
 				(font
@@
 		)
 		(property "Datasheet" "~"
-			(at 87.63 43.18 0)
+			(at 93.98 44.45 0)
 			(effects
 				(font
@@
 		)
 		(property "Description" "Generic connector, single row, 01x03, script generated"
-			(at 87.63 43.18 0)
+			(at 93.98 44.45 0)
 			(effects
 				(font
@@
 	(symbol
 		(lib_id "power:+3.3V")
-		(at 26.67 80.01 0)
+		(at 63.5 38.1 0)
 		(unit 1)
 		(exclude_from_sim no)
@@
 		(fields_autoplaced yes)
 		(property "Reference" "#PWR04"
-			(at 26.67 83.82 0)
+			(at 63.5 41.91 0)
 			(effects
 				(font
@@
 		)
 		(property "Value" "+3.3V"
-			(at 26.67 74.93 0)
+			(at 63.5 33.02 0)
 			(effects
 				(font
@@
 		)
 		(property "Footprint" ""
-			(at 26.67 80.01 0)
+			(at 63.5 38.1 0)
 			(effects
 				(font
@@
 		)
 		(property "Datasheet" ""
-			(at 26.67 80.01 0)
+			(at 63.5 38.1 0)
 			(effects
 				(font
@@
 		)
 		(property "Description" "Power symbol creates a global label with name \"+3.3V\""
-			(at 26.67 80.01 0)
+			(at 63.5 38.1 0)
 			(effects
 				(font
@@
 	(symbol
 		(lib_id "Device:R")
-		(at 26.67 86.36 0)
+		(at 63.5 44.45 0)
 		(unit 1)
 		(exclude_from_sim no)
@@
 		(fields_autoplaced yes)
 		(property "Reference" "R1"
-			(at 29.21 85.0899 0)
+			(at 66.04 43.1799 0)
 			(effects
 				(font
@@
 		)
 		(property "Value" "1.5k"
-			(at 29.21 87.6299 0)
+			(at 66.04 45.7199 0)
 			(effects
 				(font
@@
 		)
 		(property "Footprint" "Resistor_SMD:R_0805_2012Metric"
-			(at 24.892 86.36 90)
+			(at 61.722 44.45 90)
 			(effects
 				(font
@@
 		)
 		(property "Datasheet" "~"
-			(at 26.67 86.36 0)
+			(at 63.5 44.45 0)
 			(effects
 				(font
@@
 		)
 		(property "Description" "Resistor"
-			(at 26.67 86.36 0)
+			(at 63.5 44.45 0)
 			(effects
 				(font
@@
 		(lib_name "GND_1")
 		(lib_id "power:GND")
-		(at 80.01 48.26 0)
+		(at 86.36 49.53 0)
 		(unit 1)
 		(exclude_from_sim no)
@@
 		(fields_autoplaced yes)
 		(property "Reference" "#PWR012"
-			(at 80.01 54.61 0)
+			(at 86.36 55.88 0)
 			(effects
 				(font
@@
 		)
 		(property "Value" "GND"
-			(at 80.01 53.34 0)
+			(at 86.36 54.61 0)
 			(effects
 				(font
@@
 		)
 		(property "Footprint" ""
-			(at 80.01 48.26 0)
+			(at 86.36 49.53 0)
 			(effects
 				(font
@@
 		)
 		(property "Datasheet" ""
-			(at 80.01 48.26 0)
+			(at 86.36 49.53 0)
 			(effects
 				(font
@@
 		)
 		(property "Description" "Power symbol creates a global label with name \"GND\" , ground"
-			(at 80.01 48.26 0)
+			(at 86.36 49.53 0)
 			(effects
 				(font

Commit message: minor
Connections:
- no-connect marks 5 -> 6
Changed lines of the file:
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@@
+	)
+	(no_connect
+		(at 146.05 78.74)
 	)
 	(no_connect
