File: PCB/Main Board/voltageamp.kicad_sch (KiCad schematic)
At the start: 51 parts, among them U10 OPA2197xD, U11 DG201, U7 DG201, U8 INA828D, U9 OPA2197xD

Commit message: footprints and stm wiring
Connections:
- net +1.65VA: no longer R34.2, R35.2, U10.7, U9.3 (+)
- new net 1.65VA_REF: R34.2, R35.2, U10.7, U9.3 (+)
Other:
- company: Harry and Yuki - EEE3 Instrumentation -> (none)
- title: Instrumentation Amplifier -> (none)
- moved on the sheet: C23, C24, C25, C26, C27, C28, C29, C30, C31, C32, C33, C34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

Commit message: relays and layout begin
Parts:
- C38: renamed from C23; footprint (none) -> Capacitor_SMD:C_0805_2012Metric
- C39: renamed from C24; footprint (none) -> Capacitor_SMD:C_0805_2012Metric
- C40, C43: renamed from C?; footprint (none) -> Capacitor_SMD:C_0805_2012Metric
- C41: renamed from C25; footprint (none) -> Capacitor_SMD:C_0805_2012Metric
- C42: renamed from C26; footprint (none) -> Capacitor_SMD:C_0805_2012Metric
- C44: renamed from C27; footprint (none) -> Capacitor_SMD:C_0805_2012Metric
- C45: renamed from C28; footprint (none) -> Capacitor_SMD:C_0805_2012Metric
- C46: renamed from C35; footprint (none) -> Capacitor_SMD:C_0805_2012Metric
- C47: renamed from C29; footprint (none) -> Capacitor_SMD:C_0805_2012Metric
- C48: renamed from C30; footprint (none) -> Capacitor_SMD:C_0805_2012Metric
- C49: renamed from C36; footprint (none) -> Capacitor_SMD:C_0805_2012Metric
- C50: renamed from C31; footprint (none) -> Capacitor_SMD:C_0805_2012Metric
- C51: renamed from C37; footprint (none) -> Capacitor_SMD:C_0805_2012Metric
- C52: renamed from C32; footprint (none) -> Capacitor_SMD:C_0805_2012Metric
- C53: renamed from C33; footprint (none) -> Capacitor_SMD:C_0805_2012Metric
- C54: renamed from C38; footprint (none) -> Capacitor_SMD:C_0805_2012Metric
- C55: renamed from C34; footprint (none) -> Capacitor_SMD:C_0805_2012Metric
- R52: renamed from R25; footprint (none) -> Resistor_SMD:R_0805_2012Metric
- R53: renamed from R26; footprint (none) -> Resistor_SMD:R_0805_2012Metric
- R54: renamed from R27; footprint (none) -> Resistor_SMD:R_0805_2012Metric
- R55: renamed from R28; footprint (none) -> Resistor_SMD:R_0805_2012Metric
- R56: renamed from R29; footprint (none) -> Resistor_SMD:R_0805_2012Metric
- R57: renamed from R30; footprint (none) -> Resistor_SMD:R_0805_2012Metric
- R58: renamed from R31; footprint (none) -> Resistor_SMD:R_0805_2012Metric
- R59: renamed from R32; footprint (none) -> Resistor_SMD:R_0805_2012Metric
- R60: renamed from R33; footprint (none) -> Resistor_SMD:R_0805_2012Metric
- R61: renamed from R36; footprint (none) -> Resistor_SMD:R_0805_2012Metric
- R62: renamed from R37; footprint (none) -> Resistor_SMD:R_0805_2012Metric
- R63: renamed from R38; footprint (none) -> Resistor_SMD:R_0805_2012Metric
- R64: renamed from R34; footprint (none) -> Resistor_SMD:R_0805_2012Metric
- R65: renamed from R35; footprint (none) -> Resistor_SMD:R_0805_2012Metric
- R66: renamed from R39; footprint (none) -> Resistor_SMD:R_0805_2012Metric
- R67: renamed from R40; footprint (none) -> Resistor_SMD:R_0805_2012Metric
- R68: renamed from R41; footprint (none) -> Resistor_SMD:R_0805_2012Metric
- R69: renamed from R42; footprint (none) -> Resistor_SMD:R_0805_2012Metric
- R70: renamed from R43; footprint (none) -> Resistor_SMD:R_0805_2012Metric
- R71: renamed from R44; footprint (none) -> Resistor_SMD:R_0805_2012Metric
- R72: renamed from R45; footprint (none) -> Resistor_SMD:R_0805_2012Metric
- gave numbers to parts that had none: 1
- renumbered JP8 to JP11, JP9 to JP12, JP10 to JP13, JP11 to JP14, JP12 to JP15, JP13 to JP16, U7 to U13, U8 to U14, U9 to U15, U10 to U16, U11 to U17

Commit message: minor and layout
Parts:
- removed C40, C43: 100n, Capacitor_SMD:C_0805_2012Metric, symbol Device:C
- removed JP10: SolderJumper_2_Open, Jumper:SolderJumper-2_P1.3mm_Open_RoundedPad1.0x1.5mm, symbol Jumper:SolderJumper_2_Open
- removed R65: 10k, Resistor_SMD:R_0805_2012Metric, symbol Device:R
Connections:
- net 1.65VA_REF is gone; now on net +1.65VA: R64.2, U15.3 (+), U16.7
Other:
- moved on the sheet: R64, R66, R67, U16B

Commit message: :ghost:
Parts:
- renumbered C55 to C901, C45 to C902, C50 to C903, C38 to C904, C41 to C905, C44 to C906, C46 to C907, C51 to C908, C47 to C909, C52 to C910, C48 to C911, C53 to C912, C42 to C913, C49 to C914, C54 to C915, C39 to C916, JP13 to JP901, JP16 to JP902, JP11 to JP903, JP14 to JP904, JP12 to JP905, JP15 to JP906, R66 to R901, R67 to R902, R64 to R903, R54 to R904, R61 to R905, R69 to R906, R55 to R907, R70 to R908, R71 to R909, R72 to R910, R68 to R911, R52 to R912, R56 to R913, R62 to R914, R53 to R915, R57 to R916, R58 to R917, R59 to R918, R60 to R919, R63 to R920, U16 to U901, U14 to U902, U17 to U903, U13 to U904, U15 to U905
Other:
- moved on the sheet: U905A

Commit message: Layout progress
Parts:
- removed JP902, JP905, JP906: SolderJumper_2_Bridged, Jumper:SolderJumper-2_P1.3mm_Bridged_RoundedPad1.0x1.5mm, symbol Jumper:SolderJumper_2_Bridged
- removed JP903, JP904: SolderJumper_2_Open, Jumper:SolderJumper-2_P1.3mm_Open_RoundedPad1.0x1.5mm, symbol Jumper:SolderJumper_2_Open
- removed unit 2 of U901
- removed unit 2 of U905
- removed unit 3 of U905
- added JP902: SolderJumper_2_Open, Jumper:SolderJumper-2_P1.3mm_Open_RoundedPad1.0x1.5mm, symbol Jumper:SolderJumper_2_Open
- added JP903, JP904: SolderJumper_3_Bridged12, Jumper:SolderJumper-3_P1.3mm_Bridged123_RoundedPad1.0x1.5mm, symbol Jumper:SolderJumper_3_Bridged12
- added U905: OPA2376xxD, Package_SO:SOIC-8_3.9x4.9mm_P1.27mm, symbol Amplifier_Operational:OPA2376xxD
- renumbered C904 to C902, C905 to C903, C906 to C904, C902 to C905, C903 to C906, C916 to C914, C914 to C915, C915 to C916, R904 to R901, R905 to R902, R906 to R903, R907 to R904, R908 to R905, R909 to R906, R910 to R907, R911 to R908, R912 to R909, R913 to R910, R914 to R911, R915 to R912, R916 to R913, R901 to R914, R902 to R915, R917 to R916, R918 to R917, R903 to R918, U902 to U901, U903 to U902, U901 to U903, U905 to U903
Connections:
- net +1.65VA: now also U903.5 (+), JP902.2 (B), U905.1; no longer U903.3 (+)
- net +18V: now also JP903.3 (B)
- net +3.3VA: now also JP903.1 (A)
- net -18V: now also JP904.3 (B)
- net GND: now also JP904.1 (A)
- net Out: now also U905.7
- net x1: now also U904.1; no longer U904.9
- net /4: now also U904.9; no longer U904.1
- net at C901.2, R903.2, R905.1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: now also U902.15; no longer U902.14
- net at C901.1, JP901.2 (B), R903.1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: now also U902.14; no longer U902.15
- net at C904.1, R902.2, R911.2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: now also U903.6 (-), U904.3; no longer U903.2 (-), U904.2
- net at C902.2, C903.2, C904.2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: now also U903.7; no longer U903.1
- net at R904.2: now also U904.10; no longer U904.3
- net at C906.2: now also JP904.2 (C), U905.4 (V-)
- net at C902.1, R909.2: now also U904.2; no longer U904.10
- net at R919.1, R920.2: now also U905.6 (-)
- net at R914.1, R915.2: now also U905.3 (+)
- net at R918.1: now also U905.2 (-)
- net at C913.1, R917.2: now also U905.5 (+)
- net at JP901.1 (A), U901.5 (Ref): now also JP902.1 (A)
- net at C905.1: now also JP903.2 (C), U905.8 (V+)
Other:
- note added: "Short if populating"
- note removed: "Cut if populating"
- moved on the sheet: C901, C902, C903, C904, C913, C914, JP901, R901, R902, R903, R904, R905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

Commit message: :-1:
Parts:
- renumbered C901 to C601, C902 to C602, C903 to C603, C904 to C604, C905 to C605, C906 to C606, C907 to C607, C908 to C608, C909 to C609, C910 to C610, C911 to C611, C912 to C612, C913 to C613, C914 to C614, C915 to C615, C916 to C616, JP901 to JP601, JP902 to JP602, JP903 to JP603, JP904 to JP604, R901 to R601, R902 to R602, R903 to R603, R904 to R604, R905 to R605, R906 to R606, R907 to R607, R908 to R608, R909 to R609, R910 to R610, R911 to R611, R912 to R612, R913 to R613, R914 to R614, R915 to R615, R916 to R616, R917 to R617, R918 to R618, R919 to R619, R920 to R620, U901 to U601, U902 to U602, U903 to U603, U904 to U604, U905 to U605
Connections:
- net x1: now also U604.8; no longer U604.1
- net x3: now also U604.1; no longer U604.8
- net at C602.1, R609.2: now also U604.6; no longer U604.2
- net at C603.1, R610.2: now also U604.2; no longer U604.6
Other:
- moved on the sheet: U604A, U604B
