File: PCB/Main Board/voltageamp.kicad_sch (KiCad schematic)
At the start: 45 parts, among them U601 INA828D, U602 DG201, U603 OPA2197xD, U604 DG201, U605 OPA2376xxD

Commit message: changed to multiple feedback and minor error correction
Parts:
- R618: value 10k -> 5k
Other:
- moved on the sheet: R614, R615
Changed lines of the file:
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@@
 	)
 	(junction
-		(at 185.42 97.79)
+		(at 184.15 97.79)
 		(diameter 0)
 		(color 0 0 0 0)
@@
 	(wire
 		(pts
-			(xy 185.42 97.79) (xy 195.58 97.79)
+			(xy 184.15 97.79) (xy 195.58 97.79)
 		)
 		(stroke
@@
 	(wire
 		(pts
-			(xy 185.42 96.52) (xy 185.42 97.79)
+			(xy 184.15 96.52) (xy 184.15 97.79)
 		)
 		(stroke
@@
 	(wire
 		(pts
-			(xy 185.42 97.79) (xy 185.42 99.06)
+			(xy 184.15 97.79) (xy 184.15 99.06)
 		)
 		(stroke
@@
 	(symbol
 		(lib_id "Device:R")
-		(at 185.42 92.71 180)
+		(at 184.15 92.71 180)
 		(unit 1)
 		(exclude_from_sim no)
@@
 		(fields_autoplaced yes)
 		(property "Reference" "R614"
-			(at 187.96 91.4399 0)
+			(at 186.69 91.4399 0)
 			(effects
 				(font
@@
 		)
 		(property "Value" "10k"
-			(at 187.96 93.9799 0)
+			(at 186.69 93.9799 0)
 			(effects
 				(font
@@
 		)
 		(property "Footprint" "Resistor_SMD:R_0805_2012Metric"
-			(at 187.198 92.71 90)
+			(at 185.928 92.71 90)
 			(effects
 				(font
@@
 		)
 		(property "Datasheet" "~"
-			(at 185.42 92.71 0)
+			(at 184.15 92.71 0)
 			(effects
 				(font
@@
 		)
 		(property "Description" "Resistor"
-			(at 185.42 92.71 0)
+			(at 184.15 92.71 0)
 			(effects
 				(font
@@
 	(symbol
 		(lib_id "power:GND")
-		(at 185.42 106.68 0)
+		(at 184.15 106.68 0)
 		(unit 1)
 		(exclude_from_sim no)
@@
 		(fields_autoplaced yes)
 		(property "Reference" "#PWR0614"
-			(at 185.42 113.03 0)
+			(at 184.15 113.03 0)
 			(effects
 				(font
@@
 		)
 		(property "Value" "GND"
-			(at 185.42 111.76 0)
+			(at 184.15 111.76 0)
 			(effects
 				(font
@@
 		)
 		(property "Footprint" ""
-			(at 185.42 106.68 0)
+			(at 184.15 106.68 0)
 			(effects
 				(font
@@
 		)
 		(property "Datasheet" ""
-			(at 185.42 106.68 0)
+			(at 184.15 106.68 0)
 			(effects
 				(font
@@
 		)
 		(property "Description" "Power symbol creates a global label with name \"GND\" , ground"
-			(at 185.42 106.68 0)
+			(at 184.15 106.68 0)
 			(effects
 				(font
@@
 			)
 		)
-		(property "Value" "10k"
+		(property "Value" "5k"
 			(at 203.2 82.55 90)
 			(effects
@@
 	(symbol
 		(lib_id "power:+3.3VA")
-		(at 185.42 88.9 0)
+		(at 184.15 88.9 0)
 		(unit 1)
 		(exclude_from_sim no)
@@
 		(fields_autoplaced yes)
 		(property "Reference" "#PWR0613"
-			(at 185.42 92.71 0)
+			(at 184.15 92.71 0)
 			(effects
 				(font
@@
 		)
 		(property "Value" "+3.3VA"
-			(at 185.42 83.82 0)
+			(at 184.15 83.82 0)
 			(effects
 				(font
@@
 		)
 		(property "Footprint" ""
-			(at 185.42 88.9 0)
+			(at 184.15 88.9 0)
 			(effects
 				(font
@@
 		)
 		(property "Datasheet" ""
-			(at 185.42 88.9 0)
+			(at 184.15 88.9 0)
 			(effects
 				(font
@@
 		)
 		(property "Description" "Power symbol creates a global label with name \"+3.3VA\""
-			(at 185.42 88.9 0)
+			(at 184.15 88.9 0)
 			(effects
 				(font
@@
 	(symbol
 		(lib_id "Device:R")
-		(at 185.42 102.87 180)
+		(at 184.15 102.87 180)
 		(unit 1)
 		(exclude_from_sim no)
@@
 		(fields_autoplaced yes)
 		(property "Reference" "R615"
-			(at 187.96 101.5999 0)
+			(at 186.69 101.5999 0)
 			(effects
 				(font
@@
 		)
 		(property "Value" "10k"
-			(at 187.96 104.1399 0)
+			(at 186.69 104.1399 0)
 			(effects
 				(font
@@
 		)
 		(property "Footprint" "Resistor_SMD:R_0805_2012Metric"
-			(at 187.198 102.87 90)
+			(at 185.928 102.87 90)
 			(effects
 				(font
@@
 		)
 		(property "Datasheet" "~"
-			(at 185.42 102.87 0)
+			(at 184.15 102.87 0)
 			(effects
 				(font
@@
 		)
 		(property "Description" "Resistor"
-			(at 185.42 102.87 0)
+			(at 184.15 102.87 0)
 			(effects
 				(font

Commit message: sorry i fell asleep b4 layout
Parts:
- renumbered C602 to C601, C614 to C602, C613 to C604, C604 to C605, C605 to C606, C609 to C608, C611 to C609, C615 to C610, C606 to C611, C608 to C612, C610 to C613, C612 to C614, C616 to C615, C601 to C616, JP603 to JP601, JP604 to JP602, JP601 to JP603, JP602 to JP604, R609 to R601, R612 to R602, R601 to R603, R610 to R605, R613 to R606, R616 to R607, R617 to R608, R619 to R609, R602 to R610, R620 to R612, R618 to R613, R608 to R616, R603 to R617, R605 to R618, R606 to R619, R607 to R620, U604 to U601, U601 to U602, U605 to U603, U603 to U604, U602 to U605

Commit message: HI
Parts:
- renumbered C616 to C601, C601 to C602, C605 to C604, C606 to C605, C611 to C606, C612 to C608, C608 to C609, C613 to C610, C609 to C611, C614 to C612, C604 to C613, C602 to C614, C610 to C615, C615 to C616, JP603 to JP601, JP604 to JP602, JP601 to JP603, JP602 to JP604, R603 to R601, R610 to R602, R617 to R603, R618 to R605, R619 to R606, R620 to R607, R616 to R608, R601 to R609, R605 to R610, R602 to R612, R606 to R613, R607 to R616, R608 to R617, R613 to R618, R609 to R619, R612 to R620, U602 to U601, U605 to U602, U604 to U603, U601 to U604, U603 to U605

Commit message: checkpoint
Changed lines of the file:
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@@
 		(at 29.21 45.72)
+	)
+	(bus_entry
+		(at -66.04 149.86)
+		(size 2.54 2.54)
+		(stroke
+			(width 0)
+			(type default)
+		)
 	)
 	(wire

Commit message: please be nice
Parts:
- renumbered C602 to C601, C614 to C602, C613 to C604, C604 to C605, C605 to C606, C609 to C608, C611 to C609, C615 to C610, C606 to C611, C608 to C612, C610 to C613, C612 to C614, C616 to C615, C601 to C616, JP603 to JP601, JP604 to JP602, JP601 to JP603, JP602 to JP604, R609 to R601, R612 to R602, R601 to R603, R610 to R605, R613 to R606, R616 to R607, R617 to R608, R619 to R609, R602 to R610, R620 to R612, R618 to R613, R608 to R616, R603 to R617, R605 to R618, R606 to R619, R607 to R620, U604 to U601, U601 to U602, U605 to U603, U603 to U604, U602 to U605

Commit message: hello
Parts:
- renumbered C616 to C601, C601 to C602, C605 to C604, C606 to C605, C611 to C606, C612 to C608, C608 to C609, C613 to C610, C609 to C611, C614 to C612, C604 to C613, C602 to C614, C610 to C615, C615 to C616, JP603 to JP601, JP604 to JP602, JP601 to JP603, JP602 to JP604, R603 to R601, R610 to R602, R617 to R603, R618 to R605, R619 to R606, R620 to R607, R616 to R608, R601 to R609, R605 to R610, R602 to R612, R606 to R613, R607 to R616, R608 to R617, R613 to R618, R609 to R619, R612 to R620, U602 to U601, U605 to U602, U604 to U603, U601 to U604, U603 to U605
