File: PCB/Main Board/voltageamp.kicad_sch (KiCad schematic)
At the start: 41 parts, among them U601 DG201, U602 INA828D, U603 OPA2376xxD, U604 OPA2197xD, U605 DG201

Commit message: Final Schematic
Parts:
- renumbered C616 to C39, C601 to C40, C603 to C41, C605 to C42, C606 to C43, C611 to C44, C607 to C45, C612 to C46, C604 to C47, C602 to C48, C610 to C49, C615 to C50, JP604 to JP10, JP601 to JP11, JP602 to JP12, JP603 to JP9, R603 to R58, R610 to R59, R617 to R60, R604 to R61, R618 to R62, R619 to R63, R620 to R64, R616 to R65, R601 to R66, R605 to R67, R611 to R68, R602 to R69, R606 to R70, R614 to R71, R615 to R72, R607 to R73, R608 to R74, R613 to R75, R609 to R76, R612 to R77, U602 to U12, U605 to U13, U604 to U14, U601 to U15, U603 to U16
Other:
- note added: "AC coupling Optional"
- note removed: "Falstad"
- note removed: "unity gain"
- company: (none) -> Harry and Yuki - EEE3 Instrumentation
- title: (none) -> Voltage Amplifier
- moved on the sheet: C39, C40, C41, C42, C43, C44, C45, C46, C47, C48, JP10, JP11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

Commit message: cryingggggg
Parts:
- JP11, JP12: footprint Jumper:SolderJumper-3_P1.3mm_Bridged123_RoundedPad1.0x1.5mm -> Jumper:SolderJumper-3_P1.3mm_Bridged12_RoundedPad1.0x1.5mm_NumberLabels
Changed lines of the file:
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@@
 			)
 		)
-		(property "Footprint" "Jumper:SolderJumper-3_P1.3mm_Bridged123_RoundedPad1.0x1.5mm"
+		(property "Footprint" "Jumper:SolderJumper-3_P1.3mm_Bridged12_RoundedPad1.0x1.5mm_NumberLabels"
 			(at 184.15 125.73 0)
 			(effects
@@
 			)
 		)
-		(property "Footprint" "Jumper:SolderJumper-3_P1.3mm_Bridged123_RoundedPad1.0x1.5mm"
+		(property "Footprint" "Jumper:SolderJumper-3_P1.3mm_Bridged12_RoundedPad1.0x1.5mm_NumberLabels"
 			(at 184.15 148.59 0)
 			(effects

Commit message: minor cleanup from the party
Parts:
- renumbered C40 to C601, C48 to C602, C41 to C603, C47 to C604, C42 to C605, C43 to C606, C45 to C607, C49 to C608, C44 to C609, C46 to C610, C50 to C611, C39 to C612, JP11 to JP601, JP12 to JP602, JP9 to JP603, JP10 to JP604, R66 to R601, R69 to R602, R58 to R603, R61 to R604, R67 to R605, R70 to R606, R73 to R607, R74 to R608, R76 to R609, R59 to R610, R68 to R611, R77 to R612, R65 to R613, R75 to R614, R71 to R615, R60 to R616, R62 to R617, R72 to R618, R63 to R619, R64 to R620, U15 to U601, U12 to U602, U16 to U603, U14 to U604, U13 to U605

Commit message: footprints and tps
Parts:
- added TP?: +1.65VA, TestPoint:TestPoint_Pad_2.0x2.0mm, symbol Connector:TestPoint
Connections:
- net +1.65VA: now also TP?.1
Changed lines of the file:
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@@
+	)
+	(junction
+		(at 162.56 139.7)
+		(diameter 0)
+		(color 0 0 0 0)
 	)
 	(junction
@@
 		(pts
 			(xy 203.2 60.96) (xy 203.2 63.5)
+		)
+		(stroke
+			(width 0)
+			(type default)
+		)
+	)
+	(wire
+		(pts
+			(xy 162.56 142.24) (xy 162.56 139.7)
 		)
 		(stroke
@@
 				)
 			)
+		)
+	)
+	(symbol
+		(lib_id "Connector:TestPoint")
+		(at 162.56 142.24 0)
+		(mirror x)
+		(unit 1)
+		(exclude_from_sim no)
+		(in_bom yes)
+		(on_board yes)
+		(dnp no)
+		(property "Reference" "TP?"
+			(at 165.1 146.8121 0)
+			(effects
+				(font
+					(size 1.27 1.27)
+				)
+				(justify left)
+			)
+		)
+		(property "Value" "+1.65VA"
+			(at 165.1 144.2721 0)
+			(effects
+				(font
+					(size 1.27 1.27)
+				)
+				(justify left)
+			)
+		)
+		(property "Footprint" "TestPoint:TestPoint_Pad_2.0x2.0mm"
+			(at 167.64 142.24 0)
+			(effects
+				(font
+					(size 1.27 1.27)
+				)
+				(hide yes)
+			)
+		)
+		(property "Datasheet" "~"
+			(at 167.64 142.24 0)
+			(effects
+				(font
+					(size 1.27 1.27)
+				)
+				(hide yes)
+			)
+		)
+		(property "Description" "test point"
+			(at 162.56 142.24 0)
+			(effects
+				(font
+					(size 1.27 1.27)
+				)
+				(hide yes)
+			)
+		)
+		(pin "1"
+		)
+		(instances
+			(project "Main Board"
+				(path "/20aae4b7-3fb8-4924-82e8-1e7a29a313f8/95088de2-bf01-4c0a-bbbc-d1b3fecbe0ad"
+					(reference "TP?")
+					(unit 1)
+				)
+			)

Commit message: :(
Parts:
- removed JP603: SolderJumper_2_Bridged, Jumper:SolderJumper-2_P1.3mm_Bridged_RoundedPad1.0x1.5mm, symbol Jumper:SolderJumper_2_Bridged
- removed JP604: SolderJumper_2_Open, Jumper:SolderJumper-2_P1.3mm_Open_RoundedPad1.0x1.5mm, symbol Jumper:SolderJumper_2_Open
- added JP9: SolderJumper_3_Bridged12, Jumper:SolderJumper-3_P1.3mm_Bridged12_RoundedPad1.0x1.5mm_NumberLabels, symbol Jumper:SolderJumper_3_Bridged12
- gave numbers to parts that had none: 1
- renumbered C612 to C39, C601 to C40, C603 to C41, C605 to C42, C606 to C43, C609 to C44, C604 to C45, C607 to C46, C610 to C47, C602 to C48, C608 to C49, C611 to C50, JP601 to JP10, JP602 to JP11, R603 to R58, R610 to R59, R616 to R60, R604 to R61, R617 to R62, R619 to R63, R620 to R64, R613 to R65, R601 to R66, R605 to R67, R615 to R68, R618 to R69, R611 to R70, R602 to R71, R606 to R72, R614 to R73, R607 to R74, R608 to R75, R609 to R76, R612 to R77, U602 to U12, U605 to U13, U604 to U14, U601 to U15, U603 to U16
Connections:
- net +1.65VA: now also JP9.3 (B)
- net at C39.1, R60.1, U13.14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: now also JP9.1 (A)
- net at U12.5 (Ref): now also JP9.2 (C)
Other:
- note removed: "Cut to isolate"
- note removed: "Short if populating"

Commit message: edits
Parts:
- removed C48: 47p, Capacitor_SMD:C_0805_2012Metric, symbol Device:C
- removed R74: 4.85k, Resistor_SMD:R_0805_2012Metric, symbol Device:R
Connections:
- net at C40.2, C41.2, C42.2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: now also R75.1
Changed lines of the file:
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@@
 	)
 	(junction
-		(at 190.5 50.8)
-		(diameter 0)
-		(color 0 0 0 0)
-	)
-	(junction
 		(at 234.95 63.5)
 		(diameter 0)
@@
 	)
 	(junction
-		(at 234.95 50.8)
-		(diameter 0)
-		(color 0 0 0 0)
-	)
-	(junction
 		(at 110.49 127)
 		(diameter 0)
@@
 	(wire
 		(pts
-			(xy 219.71 38.1) (xy 234.95 38.1)
-		)
-		(stroke
-			(width 0)
-			(type default)
-		)
-	)
-	(wire
-		(pts
 			(xy 152.4 25.4) (xy 143.51 25.4)
 		)
@@
 	(wire
 		(pts
-			(xy 234.95 38.1) (xy 234.95 50.8)
-		)
-		(stroke
-			(width 0)
-			(type default)
-		)
-	)
-	(wire
-		(pts
 			(xy 144.78 137.16) (xy 142.24 137.16)
 		)
@@
 	(wire
 		(pts
-			(xy 190.5 38.1) (xy 190.5 50.8)
-		)
-		(stroke
-			(width 0)
-			(type default)
-		)
-	)
-	(wire
-		(pts
 			(xy 121.92 50.8) (xy 127 50.8)
 		)
@@
 	(wire
 		(pts
-			(xy 190.5 50.8) (xy 193.04 50.8)
-		)
-		(stroke
-			(width 0)
-			(type default)
-		)
-	)
-	(wire
-		(pts
 			(xy 76.2 139.7) (xy 76.2 152.4)
 		)
@@
 	(wire
 		(pts
-			(xy 187.96 50.8) (xy 190.5 50.8)
-		)
-		(stroke
-			(width 0)
-			(type default)
-		)
-	)
-	(wire
-		(pts
 			(xy 177.8 121.92) (xy 177.8 125.73)
 		)
@@
 	(wire
 		(pts
-			(xy 212.09 38.1) (xy 190.5 38.1)
-		)
-		(stroke
-			(width 0)
-			(type default)
-		)
-	)
-	(wire
-		(pts
 			(xy 127 44.45) (xy 127 50.8)
 		)
@@
 	(wire
 		(pts
-			(xy 152.4 50.8) (xy 180.34 50.8)
+			(xy 152.4 50.8) (xy 193.04 50.8)
 		)
 		(stroke
@@
 	(symbol
 		(lib_id "Device:C")
-		(at 215.9 38.1 90)
-		(unit 1)
-		(exclude_from_sim no)
-		(in_bom yes)
-		(on_board yes)
-		(dnp no)
-		(fields_autoplaced yes)
-		(property "Reference" "C48"
-			(at 215.9 30.48 90)
-			(effects
-				(font
-					(size 1.27 1.27)
-				)
-			)
-		)
-		(property "Value" "47p"
-			(at 215.9 33.02 90)
-			(effects
-				(font
-					(size 1.27 1.27)
-				)
-			)
-		)
-		(property "Footprint" "Capacitor_SMD:C_0805_2012Metric"
-			(at 219.71 37.1348 0)
-			(effects
-				(font
-					(size 1.27 1.27)
-				)
-				(hide yes)
-			)
-		)
-		(property "Datasheet" "~"
-			(at 215.9 38.1 0)
-			(effects
-				(font
-					(size 1.27 1.27)
-				)
-				(hide yes)
-			)
-		)
-		(property "Description" "Unpolarized capacitor"
-			(at 215.9 38.1 0)
-			(effects
-				(font
-					(size 1.27 1.27)
-				)
-				(hide yes)
-			)
-		)
-		(pin "1"
-		)
-		(pin "2"
-		)
-		(instances
-			(project "Main Board"
-				(path "/20aae4b7-3fb8-4924-82e8-1e7a29a313f8/95088de2-bf01-4c0a-bbbc-d1b3fecbe0ad"
-					(reference "C48")
-					(unit 1)
-				)
-			)
-		)
-	)
-	(symbol
-		(lib_id "Device:C")
 		(at 228.6 133.35 0)
 		(unit 1)
@@
 					(unit 1)
 				)
-			)
-		)
-	)
-	(symbol
-		(lib_id "Device:R")
-		(at 184.15 50.8 90)
-		(unit 1)
-		(exclude_from_sim no)
-		(in_bom yes)
-		(on_board yes)
-		(dnp no)
-		(fields_autoplaced yes)
-		(property "Reference" "R74"
-			(at 184.15 44.45 90)
-			(effects
-				(font
-					(size 1.27 1.27)
-				)
-			)
-		)
-		(property "Value" "4.85k"
-			(at 184.15 46.99 90)
-			(effects
-				(font
-					(size 1.27 1.27)
-				)
-			)
-		)
-		(property "Footprint" "Resistor_SMD:R_0805_2012Metric"
-			(at 184.15 52.578 90)
-			(effects
-				(font
-					(size 1.27 1.27)
-				)
-				(hide yes)
-			)
-		)
-		(property "Datasheet" "~"
-			(at 184.15 50.8 0)
-			(effects
-				(font
-					(size 1.27 1.27)
-				)
-				(hide yes)
-			)
-		)
-		(property "Description" "Resistor"
-			(at 184.15 50.8 0)
-			(effects
-				(font
-					(size 1.27 1.27)
-				)
-				(hide yes)
-			)
-		)
-		(pin "2"
-		)
-		(pin "1"
-		)
-		(instances
-			(project "Main Board"
-				(path "/20aae4b7-3fb8-4924-82e8-1e7a29a313f8/95088de2-bf01-4c0a-bbbc-d1b3fecbe0ad"
-					(reference "R74")
-					(unit 1)
-				)

Commit message: minor
Parts:
- added C?: 100n, Capacitor_SMD:C_0805_2012Metric, symbol Device:C
- R60: now fitted
Connections:
- net GND: now also C?.2
- net at R68.1, R69.2, U16.3 (+): now also C?.1
Changed lines of the file:
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@@
 	(wire
 		(pts
-			(xy 234.95 50.8) (xy 247.65 50.8)
+			(xy 234.95 53.34) (xy 247.65 53.34)
 		)
 		(stroke
@@
 	(wire
 		(pts
+			(xy 121.92 143.51) (xy 121.92 142.24)
+		)
+		(stroke
+			(width 0)
+			(type default)
+		)
+	)
+	(wire
+		(pts
 			(xy 67.31 152.4) (xy 76.2 152.4)
 		)
@@
 	(wire
 		(pts
-			(xy 234.95 50.8) (xy 234.95 53.34)
+			(xy 86.36 165.1) (xy 90.17 165.1)
 		)
 		(stroke
@@
 	(wire
 		(pts
-			(xy 86.36 165.1) (xy 90.17 165.1)
+			(xy 45.72 50.8) (xy 50.8 50.8)
 		)
 		(stroke
@@
 	(wire
 		(pts
-			(xy 45.72 50.8) (xy 50.8 50.8)
+			(xy 156.21 130.81) (xy 162.56 130.81)
 		)
 		(stroke
@@
 	(wire
 		(pts
-			(xy 156.21 130.81) (xy 162.56 130.81)
+			(xy 76.2 165.1) (xy 78.74 165.1)
 		)
 		(stroke
@@
 	(wire
 		(pts
-			(xy 76.2 165.1) (xy 78.74 165.1)
+			(xy 121.92 142.24) (xy 133.35 142.24)
 		)
 		(stroke
@@
 	(hierarchical_label "Out"
 		(shape output)
-		(at 247.65 50.8 0)
+		(at 247.65 53.34 0)
 		(effects
 			(font
@@
 	)
 	(symbol
+		(lib_id "Device:C")
+		(at 121.92 147.32 0)
+		(unit 1)
+		(exclude_from_sim no)
+		(in_bom yes)
+		(on_board yes)
+		(dnp no)
+		(fields_autoplaced yes)
+		(property "Reference" "C?"
+			(at 125.73 146.0499 0)
+			(effects
+				(font
+					(size 1.27 1.27)
+				)
+				(justify left)
+			)
+		)
+		(property "Value" "100n"
+			(at 125.73 148.5899 0)
+			(effects
+				(font
+					(size 1.27 1.27)
+				)
+				(justify left)
+			)
+		)
+		(property "Footprint" "Capacitor_SMD:C_0805_2012Metric"
+			(at 122.8852 151.13 0)
+			(effects
+				(font
+					(size 1.27 1.27)
+				)
+				(hide yes)
+			)
+		)
+		(property "Datasheet" "~"
+			(at 121.92 147.32 0)
+			(effects
+				(font
+					(size 1.27 1.27)
+				)
+				(hide yes)
+			)
+		)
+		(property "Description" "Unpolarized capacitor"
+			(at 121.92 147.32 0)
+			(effects
+				(font
+					(size 1.27 1.27)
+				)
+				(hide yes)
+			)
+		)
+		(pin "1"
+		)
+		(pin "2"
+		)
+		(instances
+			(project "Main Board"
+				(path "/20aae4b7-3fb8-4924-82e8-1e7a29a313f8/95088de2-bf01-4c0a-bbbc-d1b3fecbe0ad"
+					(reference "C?")
+					(unit 1)
+				)
+			)
+		)
+	)
+	(symbol
 		(lib_id "More_symbols:DG201")
 		(at 88.9 50.8 0)
@@
 		(in_bom yes)
 		(on_board yes)
-		(dnp yes)
+		(dnp no)
 		(property "Reference" "R60"
 			(at 63.5 133.35 90)
@@
 					(unit 1)
 				)
+			)
+		)
+	)
+	(symbol
+		(lib_id "power:GND")
+		(at 121.92 151.13 0)
+		(unit 1)
+		(exclude_from_sim no)
+		(in_bom yes)
+		(on_board yes)
+		(dnp no)
+		(fields_autoplaced yes)
+		(property "Reference" "#PWR0601"
+			(at 121.92 157.48 0)
+			(effects
+				(font
+					(size 1.27 1.27)
+				)
+				(hide yes)
+			)
+		)
+		(property "Value" "GND"
+			(at 121.92 156.21 0)
+			(effects
+				(font
+					(size 1.27 1.27)
+				)
+			)
+		)
+		(property "Footprint" ""
+			(at 121.92 151.13 0)
+			(effects
+				(font
+					(size 1.27 1.27)
+				)
+				(hide yes)
+			)
+		)
+		(property "Datasheet" ""
+			(at 121.92 151.13 0)
+			(effects
+				(font
+					(size 1.27 1.27)
+				)
+				(hide yes)
+			)
+		)
+		(property "Description" "Power symbol creates a global label with name \"GND\" , ground"
+			(at 121.92 151.13 0)
+			(effects
+				(font
+					(size 1.27 1.27)
+				)
+				(hide yes)
+			)
+		)
+		(pin "1"
+		)
+		(instances
+			(project "Main Board"
+				(path "/20aae4b7-3fb8-4924-82e8-1e7a29a313f8/95088de2-bf01-4c0a-bbbc-d1b3fecbe0ad"
+					(reference "#PWR0601")
+					(unit 1)
+				)

Commit message: BLEH
Parts:
- gave numbers to parts that had none: 1
- renumbered C39 to C38, C49 to C48, C50 to C49, JP9 to JP6, JP10 to JP7, JP11 to JP8, R58 to R56, R59 to R57, R60 to R58, R61 to R59, R62 to R60, R63 to R61, R64 to R62, R65 to R63, R66 to R64, R67 to R65, R68 to R66, R69 to R67, R70 to R68, R71 to R69, R72 to R70, R73 to R71, R75 to R72, R76 to R73, R77 to R74, TP9 to TP8, U12 to U11, U13 to U12, U14 to U13, U15 to U14, U16 to U15
