File: PCB/Main Board/Bridge.kicad_sch (KiCad schematic)
At the start: 48 parts, among them K3 AGQ200A12, Q3 2N4401, Q4 2N4401, Q5 2N4403, Q6 2N4403, U10 DG201, U7 OPA2197xD, U8 OPA2197xD, U9 OPA2197xD

Commit message: amplifer floorplan and relay footprint + minor
Parts:
- K3: footprint AGQ200A03X -> AGQ200A12_footprint
Changed lines of the file:
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@@
 			)
 		)
-		(property "Footprint" "AGQ200A03X"
+		(property "Footprint" "AGQ200A12_footprint"
 			(at 158.75 135.56 0)
 			(effects

Commit message: :ghost:
Parts:
- removed D2, D3: BAV99, Package_TO_SOT_SMD:SOT-363_SC-70-6, symbol Diode:BAV99
- added D701, D703: BAV99, Package_TO_SOT_SMD:SOT-23, symbol Diode:BAV99
- added JP702: SolderJumper_2_Bridged, Jumper:SolderJumper-2_P1.3mm_Bridged_RoundedPad1.0x1.5mm, symbol Jumper:SolderJumper_2_Bridged
- renumbered C25 to C701, C26 to C702, C29 to C703, C30 to C704, C34 to C705, C31 to C706, C35 to C707, C23 to C708, C24 to C709, C27 to C710, C28 to C711, C32 to C712, C36 to C713, C33 to C714, C37 to C715, D4 to D702, JP8 to JP701, K3 to K701, Q4 to Q701, Q6 to Q702, Q3 to Q703, Q5 to Q704, R34 to R701, R33 to R702, R38 to R703, R25 to R704, R32 to R705, R39 to R706, R26 to R707, R28 to R708, R35 to R709, R41 to R710, R27 to R711, R29 to R712, R40 to R713, R42 to R714, R43 to R715, R44 to R716, R31 to R717, R36 to R718, R30 to R719, R37 to R720, U9 to U701, U10 to U702, U8 to U703, U7 to U704
Connections:
- net GND: now also JP702.1 (A); no longer K701.2
- net at Q703.2 (B), R717.2: now also D703.1 (K)
- net at Q701.2 (B), R702.2: now also D701.1 (K)
- net at Q702.2 (B), R703.1: now also D701.2 (A)
- net at U701.1: now also D701.3 (K)
- net at U704.1: now also D703.3 (K)
- net at Q704.2 (B), R718.1: now also D703.2 (A)
- new net GUARD: JP702.2 (B), K701.2

Commit message: Layout progress
Parts:
- removed JP701: SolderJumper_2_Open, Jumper:SolderJumper-2_P1.3mm_Open_RoundedPad1.0x1.5mm, symbol Jumper:SolderJumper_2_Open
Other:
- note removed: "i removed the guarding here"
Changed lines of the file:
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@@
-		)
-	)
-	(text "i removed the guarding here"
-		(exclude_from_sim no)
-		(at 156.21 49.53 0)
-		(effects
-			(font
-				(size 1.27 1.27)
-			)
 		)
 	)
@@
 	)
 	(junction
-		(at 160.02 90.17)
-		(diameter 0)
-		(color 0 0 0 0)
-	)
-	(junction
 		(at 149.86 115.57)
 		(diameter 0)
@@
 	(junction
 		(at 66.04 60.96)
-		(diameter 0)
-		(color 0 0 0 0)
-	)
-	(junction
-		(at 134.62 87.63)
 		(diameter 0)
 		(color 0 0 0 0)
@@
 	(wire
 		(pts
-			(xy 160.02 96.52) (xy 160.02 90.17)
-		)
-		(stroke
-			(width 0)
-			(type default)
-		)
-	)
-	(wire
-		(pts
 			(xy 57.15 95.25) (xy 57.15 96.52)
 		)
@@
 	(wire
 		(pts
-			(xy 134.62 96.52) (xy 143.51 96.52)
-		)
-		(stroke
-			(width 0)
-			(type default)
-		)
-	)
-	(wire
-		(pts
 			(xy 119.38 82.55) (xy 110.49 82.55)
 		)
@@
 	(wire
 		(pts
-			(xy 134.62 87.63) (xy 134.62 96.52)
-		)
-		(stroke
-			(width 0)
-			(type default)
-		)
-	)
-	(wire
-		(pts
 			(xy 146.05 115.57) (xy 149.86 115.57)
 		)
@@
 		(pts
 			(xy 105.41 109.22) (xy 105.41 110.49)
-		)
-		(stroke
-			(width 0)
-			(type default)
-		)
-	)
-	(wire
-		(pts
-			(xy 151.13 96.52) (xy 160.02 96.52)
 		)
 		(stroke
@@
 					(unit 1)
 				)
-			)
-		)
-	)
-	(symbol
-		(lib_id "Jumper:SolderJumper_2_Open")
-		(at 147.32 96.52 180)
-		(unit 1)
-		(exclude_from_sim no)
-		(in_bom no)
-		(on_board yes)
-		(dnp no)
-		(property "Reference" "JP701"
-			(at 146.05 92.71 0)
-			(effects
-				(font
-					(size 1.27 1.27)
-				)
-				(justify right)
-			)
-		)
-		(property "Value" "SolderJumper_2_Open"
-			(at 146.0501 99.06 90)
-			(effects
-				(font
-					(size 1.27 1.27)
-				)
-				(justify left)
-				(hide yes)
-			)
-		)
-		(property "Footprint" "Jumper:SolderJumper-2_P1.3mm_Open_RoundedPad1.0x1.5mm"
-			(at 147.32 96.52 0)
-			(effects
-				(font
-					(size 1.27 1.27)
-				)
-				(hide yes)
-			)
-		)
-		(property "Datasheet" "~"
-			(at 147.32 96.52 0)
-			(effects
-				(font
-					(size 1.27 1.27)
-				)
-				(hide yes)
-			)
-		)
-		(property "Description" "Solder Jumper, 2-pole, open"
-			(at 147.32 96.52 0)
-			(effects
-				(font
-					(size 1.27 1.27)
-				)
-				(hide yes)
-			)
-		)
-		(pin "1"
-		)
-		(pin "2"
-		)
-		(instances
-			(project "Main Board"
-				(path "/20aae4b7-3fb8-4924-82e8-1e7a29a313f8/6b7fef71-3444-4c8f-b2e2-502774ba9b51"
-					(reference "JP701")
-					(unit 1)
-				)

Commit message: aaa
Parts:
- renumbered JP702 to JP701
Changed lines of the file:
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@@
 		(on_board yes)
 		(dnp no)
-		(property "Reference" "JP702"
+		(property "Reference" "JP701"
 			(at 232.41 125.73 0)
 			(effects
@@
 			(project "Main Board"
 				(path "/20aae4b7-3fb8-4924-82e8-1e7a29a313f8/6b7fef71-3444-4c8f-b2e2-502774ba9b51"
-					(reference "JP702")
+					(reference "JP701")
 					(unit 1)
 				)

Commit message: beep beep
Parts:
- added C716, C717: 100n, Capacitor_SMD:C_0805_2012Metric, symbol Device:C
- added unit 3 of U704
- added unit 1 of U704
- Q701, Q702, Q703, Q704: footprint Package_TO_SOT_THT:TO-92_Inline -> Package_TO_SOT_THT:TO-220-3_Horizontal_TabDown
- R709: value 1 -> 50
- renumbered C712 to C708, C713 to C709, C708 to C710, C709 to C711, C710 to C712, C711 to C713, U703 to U701, U704 to U701, U704 to U703, U701 to U703
Connections:
- net +18V: now also C716.1, U704.8 (V+)
- net -18V: now also C717.2, U704.4 (V-)
- net GND: now also U701.3 (+), U701.5 (+), U704.5 (+), C716.2, C717.1, U704.3 (+); no longer U701.3 (+), U701.5 (+), U704.3 (+)
- net In: now also U704.6 (-); no longer U704.2 (-)
- net at C705.2, R710.2, R713.1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: now also U701.6 (-); no longer U701.6 (-)
- net at D703.3 (K): now also U704.7; no longer U704.1
- net at C705.1, R701.1, R710.1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: now also U701.7; no longer U701.7
- net at D701.3 (K): now also U701.1; no longer U701.1
- net at R701.2, R704.1: now also U701.2 (-); no longer U701.2 (-)
- net at K701.3, R709.2: now also U703.3 (+); no longer U703.5 (+)
- new net: R712.2, U703.1, U703.2 (-)
- new net: U704.1, U704.2 (-)
Other:
- note removed: "changed these values and removed the opamp if the resistor values are big its not needed"
- moved on the sheet: C706, C707, C708, C709, C714, C715, JP701, K701, U701A, U701B, U701C, U702E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

Commit message: :-1:
Parts:
- removed D702: BAV199, Package_TO_SOT_SMD:SOT-363_SC-70-6, symbol Diode:BAV99
- added D402: BAV199, Package_TO_SOT_SMD:SOT-23, symbol Diode:BAV99
- renumbered C701 to C401, C702 to C402, C703 to C403, C704 to C404, C705 to C405, C706 to C406, C707 to C407, C708 to C408, C709 to C409, C710 to C410, C711 to C411, C712 to C412, C713 to C413, C714 to C414, C715 to C415, C716 to C416, C717 to C417, D701 to D401, D703 to D403, JP701 to JP401, K701 to K401, Q701 to Q401, Q702 to Q402, Q703 to Q403, Q704 to Q404, R701 to R401, R702 to R402, R703 to R403, R704 to R404, R705 to R405, R706 to R406, R707 to R407, R708 to R408, R709 to R409, R710 to R410, R711 to R411, R712 to R412, R713 to R413, R714 to R414, R715 to R415, R716 to R416, R717 to R417, R718 to R418, R719 to R419, R720 to R420, U701 to U401, U702 to U402, U703 to U403, U704 to U404
Connections:
- net GND: now also D402.1 (K), D402.2 (A)
- net In: now also D402.3 (K)

Commit message: changed to multiple feedback and minor error correction
Parts:
- removed R405, R406, R419, R420: 100m, Resistor_SMD:R_0805_2012Metric, symbol Device:R
Connections:
- net +18V: now also Q401.3 (C), Q403.3 (C)
- net -18V: now also Q402.3 (C), Q404.3 (C)
Other:
- moved on the sheet: K401
