File: PCB/Main Board/Bridge.kicad_sch (KiCad schematic)
At the start: 46 parts, among them K401 AGQ200A12, Q401 2N4401, Q402 2N4403, Q403 2N4401, Q404 2N4403, U401 OPA2197xD, U402 DG201, U403 OPA2197xD, U404 OPA2197xD

Commit message: minor schematic changes
Parts:
- added C?: 100n, Capacitor_SMD:C_0805_2012Metric, symbol Device:C
- added J?: Conn_01x01_Pin, Connector_PinHeader_2.54mm:PinHeader_1x01_P2.54mm_Horizontal, symbol Connector:Conn_01x01_Pin
- added JP?: SolderJumper_3_Open, symbol Jumper:SolderJumper_3_Open
- added R?: 20k, Resistor_SMD:R_0805_2012Metric, symbol Device:R
- added RN?: 4610X-R2R-103LF, SIP249W51P254L2535H508Q10P, symbol 4610X-R2R-103LF:4610X-R2R-103LF
Connections:
- net -18V: now also JP?.3 (B)
- net GND: now also C?.2, JP?.1 (A); no longer U404.3 (+)
- net at U404.2 (-): now also R?.1, RN?.1; no longer U404.1
- new net: JP?.2 (C), RN?.10, U404.3 (+)
- new net: C?.1, J?.1 (Pin_1), R?.2, U404.1
- new net DAC_0: RN?.2
- new net DAC_1: RN?.3
- new net DAC_2: RN?.4
- new net DAC_3: RN?.5
- new net DAC_4: RN?.6
- new net DAC_5: RN?.7
- new net DAC_6: RN?.8
- new net DAC_7: RN?.9
Other:
- note added: "10k R/2R IC"
- note added: "LSB"
- note added: "MSB"
- note added: "SUM"
- moved on the sheet: C401, C402, C403, C404, C405, C406, C407, C408, C409, C414, C415, C416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

Commit message: sorry i fell asleep b4 layout
Parts:
- removed C?: 100n, Capacitor_SMD:C_0805_2012Metric, symbol Device:C
- removed J?: Conn_01x01_Pin, Connector_PinHeader_2.54mm:PinHeader_1x01_P2.54mm_Horizontal, symbol Connector:Conn_01x01_Pin
- removed JP?: SolderJumper_3_Open, symbol Jumper:SolderJumper_3_Open
- removed R?: 20k, Resistor_SMD:R_0805_2012Metric, symbol Device:R
- removed RN?: 4610X-R2R-103LF, SIP249W51P254L2535H508Q10P, symbol 4610X-R2R-103LF:4610X-R2R-103LF
- renumbered C410 to C403, C411 to C404, C403 to C405, C404 to C406, C412 to C407, C413 to C408, C405 to C409, C406 to C410, C408 to C411, C414 to C412, C416 to C413, C407 to C414, C409 to C415, C415 to C416, D403 to D402, D402 to D403, Q403 to Q402, Q402 to Q403, R404 to R401, R407 to R402, R411 to R403, R408 to R404, R412 to R405, R402 to R406, R417 to R407, R401 to R408, R403 to R410, R413 to R411, R418 to R412, R410 to R413, U403 to U401, U401 to U402, U404 to U403, U402 to U404
Connections:
- net GUARD: now also U403.1, U403.2 (-); no longer JP401.2 (B)
- net at U403.3 (+): now also JP401.2 (B)
Other:
- note removed: "10k R/2R IC"
- note removed: "LSB"
- note removed: "MSB"
- note removed: "SUM"
- moved on the sheet: JP401, U403A

Commit message: HI
Parts:
- removed JP401: SolderJumper_2_Bridged, Jumper:SolderJumper-2_P1.3mm_Bridged_RoundedPad1.0x1.5mm, symbol Jumper:SolderJumper_2_Bridged
- added JP401: SolderJumper_3_Bridged12, Jumper:SolderJumper-3_P1.3mm_Bridged123_RoundedPad1.0x1.5mm, symbol Jumper:SolderJumper_3_Bridged12
- K401: footprint AGQ200A12_footprint -> AGQ:RELAY_AGQ_A_PAN
- renumbered C405 to C403, C406 to C404, C409 to C405, C410 to C406, C414 to C407, C411 to C408, C415 to C409, C403 to C410, C404 to C411, C407 to C412, C408 to C413, C412 to C414, C416 to C415, C413 to C416, D403 to D402, D402 to D403, Q403 to Q402, Q402 to Q403, R408 to R401, R406 to R402, R410 to R403, R401 to R404, R413 to R405, R402 to R406, R404 to R407, R409 to R408, R411 to R409, R414 to R410, R415 to R411, R416 to R412, R403 to R413, R405 to R414, R407 to R415, R412 to R416, U402 to U401, U404 to U402, U401 to U403, U403 to U404
Connections:
- net GND: now also U404.3 (+), JP401.3 (B)
- net GUARD: now also JP401.2 (C); no longer U404.1, U404.2 (-)
- new net: JP401.1 (A), U404.1, U404.2 (-)
Other:
- moved on the sheet: U404A

Commit message: footprints
Parts:
- removed Q401, Q403: 2N4401, Package_TO_SOT_THT:TO-220-3_Horizontal_TabDown, symbol Transistor_BJT:2N2219
- removed Q402, Q404: 2N4403, Package_TO_SOT_THT:TO-220-3_Horizontal_TabDown, symbol Transistor_BJT:2N3906
- added Q? (x2): TIP41C, Package_TO_SOT_THT:TO-220-3_Vertical, symbol Transistor_BJT:TIP41C
- added Q? (x2): TIP42C, Package_TO_SOT_THT:TO-220-3_Vertical, symbol Transistor_BJT:TIP42C
Connections:
- net +18V: now also Q?.3 (E), Q?.3 (E)
- net -18V: now also Q?.3 (E), Q?.3 (E)
- net Resistor Selector/I_OUT: now also Q?.2 (C), Q?.2 (C)
- net at D403.1 (K), R415.2: now also Q?.1 (B)
- net at R404.2, R407.2, R408.1: now also Q?.2 (C), Q?.2 (C)
- net at D401.2 (A), R403.1: now also Q?.1 (B)
- net at D403.2 (A), R416.1: now also Q?.1 (B)
- net at D401.1 (K), R402.2: now also Q?.1 (B)

Commit message: checkpoint
Parts:
- added R405, R406, R419, R420: 100m, Resistor_SMD:R_0805_2012Metric, symbol Device:R
- Q401, Q402, Q403, Q404: renamed from Q?; footprint Package_TO_SOT_THT:TO-220-3_Vertical -> Package_TO_SOT_THT:TO-220-3_Horizontal_TabDown
- renumbered C404 to C402, C402 to C403, C403 to C404, C413 to C411, C411 to C412, C412 to C413, R405 to R407, R406 to R408, R407 to R409, R408 to R410, R409 to R411, R410 to R412, R411 to R413, R412 to R414, R413 to R415, R414 to R416, R415 to R417, R416 to R418
Connections:
- net +18V: now also Q401.2 (C), Q403.2 (C); no longer Q402.3 (E), Q404.3 (E)
- net -18V: now also Q402.2 (C), Q404.2 (C); no longer Q401.3 (E), Q403.3 (E)
- net Resistor Selector/I_OUT: now also U402.14, R419.2, R420.1; no longer Q403.2 (C), Q404.2 (C), U402.15
- net at D403.2 (A), R418.1: now also Q404.1 (B); no longer Q403.1 (B)
- net at D403.1 (K), R417.2: now also Q403.1 (B); no longer Q404.1 (B)
- net at R411.2: now also U402.15; no longer U402.14
- net at D401.1 (K), R402.2: now also Q401.1 (B); no longer Q402.1 (B)
- net at R404.2, R409.2, R410.1: now also R405.2, R406.1; no longer Q401.2 (C), Q402.2 (C)
- net at D401.2 (A), R403.1: now also Q402.1 (B); no longer Q401.1 (B)
- new net: Q403.3 (E), R419.1
- new net: Q404.3 (E), R420.2
- new net: Q401.3 (E), R405.1
- new net: Q402.3 (E), R406.2
Other:
- moved on the sheet: C401, C402, C403, C404, C410, C411, C412, C413, Q401, Q402, Q403, Q404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

Commit message: Cryiunbg
Connections:
- net GUARD: now also K401.7; no longer K401.2
- net In: now also K401.5; no longer K401.4
- net at R410.2, U403.3 (+): now also K401.6; no longer K401.3
Other:
- moved on the sheet: K401
Changed lines of the file:
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@@
 	)
 	(no_connect
-		(at 153.67 86.36)
+		(at 153.67 66.04)
 	)
 	(no_connect
-		(at 138.43 83.82)
+		(at 138.43 63.5)
 	)
 	(no_connect
-		(at 153.67 81.28)
+		(at 153.67 60.96)
 	)
 	(wire
@@
 	(hierarchical_label "DC_INT_ISO"
 		(shape input)
-		(at 138.43 63.5 180)
+		(at 138.43 53.34 180)
 		(effects
 			(font
@@
 	(symbol
 		(lib_id "More_power:+18V")
-		(at 153.67 63.5 270)
+		(at 153.67 53.34 270)
 		(unit 1)
 		(exclude_from_sim no)
@@
 		(fields_autoplaced yes)
 		(property "Reference" "#PWR0411"
-			(at 149.86 63.5 0)
+			(at 149.86 53.34 0)
 			(effects
 				(font
@@
 		)
 		(property "Value" "+12V"
-			(at 157.48 63.4999 90)
+			(at 157.48 53.3399 90)
 			(effects
 				(font
@@
 		)
 		(property "Footprint" ""
-			(at 153.67 63.5 0)
+			(at 153.67 53.34 0)
 			(effects
 				(font
@@
 		)
 		(property "Datasheet" ""
-			(at 153.67 63.5 0)
+			(at 153.67 53.34 0)
 			(effects
 				(font
@@
 		)
 		(property "Description" "Power symbol creates a global label with name \"+18V\""
-			(at 153.67 63.5 0)
+			(at 153.67 53.34 0)
 			(effects
 				(font
@@
 	(symbol
 		(lib_id "AGQ200A12:AGQ200A12")
-		(at 146.05 72.39 0)
+		(at 146.05 62.23 0)
 		(unit 1)
 		(exclude_from_sim no)
@@
 		(fields_autoplaced yes)
 		(property "Reference" "K401"
-			(at 146.05 53.34 0)
+			(at 146.05 43.18 0)
 			(effects
 				(font
@@
 		)
 		(property "Value" "AGQ200A12"
-			(at 146.05 55.88 0)
+			(at 146.05 45.72 0)
 			(effects
 				(font
@@
 		)
 		(property "Footprint" "AGQ:RELAY_AGQ_A_PAN"
-			(at 157.48 136.83 0)
+			(at 157.48 126.67 0)
 			(effects
 				(font
@@
 		)
 		(property "Datasheet" "https://industry.panasonic.com/ac/cdn/e/control/relay/signal/catalog/mech_eng_gq.pdf"
-			(at 157.48 236.83 0)
+			(at 157.48 226.67 0)
 			(effects
 				(font
@@
 		)
 		(property "Description" "High sensitivity, 100 mW operating power, 2 Form C, 2 A, compact size and flat relays"
-			(at 154.178 71.374 0)
+			(at 154.178 61.214 0)
 			(effects
 				(font
@@
 		)
 		(property "Height" "5.4"
-			(at 157.48 436.83 0)
+			(at 157.48 426.67 0)
 			(effects
 				(font
@@
 		)
 		(property "Mouser Part Number" "769-AGQ200A12"
-			(at 157.48 536.83 0)
+			(at 157.48 526.67 0)
 			(effects
 				(font
@@
 		)
 		(property "Mouser Price/Stock" "https://www.mouser.co.uk/ProductDetail/Panasonic-Industrial-Devices/AGQ200A12?qs=HLLy2pIPwutAjJTGv7DYvA%3D%3D"
-			(at 157.48 636.83 0)
+			(at 157.48 626.67 0)
 			(effects
 				(font
@@
 		)
 		(property "Manufacturer_Name" "Panasonic"
-			(at 157.48 736.83 0)
+			(at 157.48 726.67 0)
 			(effects
 				(font
@@
 		)
 		(property "Manufacturer_Part_Number" "AGQ200A12"
-			(at 157.48 836.83 0)
+			(at 157.48 826.67 0)
 			(effects
 				(font

Commit message: merge 2.0
Parts:
- removed C402, C403, C411, C412: 100n, Capacitor_SMD:C_0805_2012Metric, symbol Device:C
Other:
- moved on the sheet: C401, C410, C413
