File: PCB/Main Board/Bridge.kicad_sch (KiCad schematic)
At the start: 46 parts, among them K401 AGQ200A12, Q401 TIP41C, Q402 TIP42C, Q403 TIP41C, Q404 TIP42C, U401 OPA2197xD, U402 DG201, U403 OPA2197xD, U404 OPA2197xD

Commit message: yup
Parts:
- added U402: ULN2003, Package_SO:SOIC-16_3.9x9.9mm_P1.27mm, symbol Transistor_Array:ULN2003
- renumbered C404 to C402, C405 to C403, C406 to C404, C407 to C405, C408 to C406, C409 to C407, C410 to C408, C413 to C409, C414 to C410, C415 to C411, C416 to C412, C417 to C413, U402 to U403, U403 to U404, U404 to U405
Connections:
- net +12V: now also U402.9 (COM)
- net DC_INT_ISO: now also U402.6 (I6); no longer K401.8
- net GND: now also U402.8 (GND)
- net R_SEL_10: now also U402.1 (I1)
- net R_SEL_100: now also U402.2 (I2)
- net R_SEL_100k: now also U402.5 (I5)
- net R_SEL_10k: now also U402.4 (I4)
- net R_SEL_1k: now also U402.3 (I3)
- new net DC_ISO: K401.8, U402.11 (O6)
- new net SEL_10: U402.13 (O4)
- new net SEL_100: U402.14 (O3)
- new net SEL_100k: U402.12 (O5)
- new net SEL_10k: U402.16 (O1)
- new net SEL_1k: U402.15 (O2)
- no-connect marks 3 -> 5

Commit message: sig source finished
Parts:
- removed C408, C409: 10µ, Capacitor_SMD:C_0805_2012Metric, symbol Device:C
- removed R405, R406, R419, R420: 100m, Resistor_SMD:R_0805_2012Metric, symbol Device:R
- added C403, C404: 1u, Capacitor_SMD:C_0805_2012Metric, symbol Device:C
- added C405, C406: 10µ, Capacitor_SMD:C_0805_2012Metric, symbol Device:C
- renumbered C403 to C407, C404 to C408, C406 to C409, C412 to C411, C405 to C412, C407 to C413, C411 to C414, C413 to C415, D403 to D402, D402 to D403, Q403 to Q402, Q402 to Q403, R404 to R401, R408 to R402, R415 to R403, R409 to R404, R416 to R405, R402 to R406, R417 to R407, R410 to R408, R401 to R409, R403 to R410, R418 to R412, R407 to R413, R412 to R414, R413 to R415, R414 to R416, U404 to U401, U401 to U402, U405 to U403, U403 to U404, U402 to U405
Connections:
- net +18V: now also C402.2
- net -18V: now also C405.2, C406.2; no longer C402.2
- net GND: now also C405.1, C406.1
- net Resistor Selector/I_OUT: now also Q402.3 (E), Q404.3 (E)
- net at U403.7: now also C404.1; no longer D402.3 (K)
- net at Q401.3 (E): now also Q403.3 (E), R401.2, R404.2, R408.1
- net at U402.1: now also C403.1; no longer D401.3 (K)
- new net: C403.2, D401.3 (K)
- new net: C404.2, D402.3 (K)
Other:
- moved on the sheet: Q401, Q402, Q403, Q404, R406, R407, R409, R410, R412, U402A

Commit message: hello
Parts:
- Q401, Q404: footprint Package_TO_SOT_THT:TO-220-3_Horizontal_TabDown -> Package_TO_SOT_THT:TO-220-3_Horizontal_TabUp
- Q402: renamed from Q403; footprint Package_TO_SOT_THT:TO-220-3_Horizontal_TabDown -> Package_TO_SOT_THT:TO-220-3_Horizontal_TabUp
- Q403: renamed from Q402; footprint Package_TO_SOT_THT:TO-220-3_Horizontal_TabDown -> Package_TO_SOT_THT:TO-220-3_Horizontal_TabUp
- renumbered C403 to C401, C401 to C402, C405 to C403, C407 to C404, C408 to C405, C412 to C406, C409 to C407, C413 to C408, C404 to C409, C402 to C410, C406 to C411, C410 to C412, C414 to C413, C411 to C414, D403 to D402, D402 to D403, R409 to R401, R406 to R402, R410 to R403, R401 to R404, R413 to R405, R402 to R406, R404 to R407, R411 to R409, R414 to R410, R415 to R411, R416 to R412, R403 to R413, R405 to R414, R407 to R415, R412 to R416, U402 to U401, U405 to U402, U404 to U403, U401 to U404, U403 to U405

Commit message: Krill me
Parts:
- removed C401, C409: 1u, Capacitor_SMD:C_0805_2012Metric, symbol Device:C
Connections:
- net at U405.7: now also D403.3 (K)
- net at U401.1: now also D401.3 (K)
Changed lines of the file:
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@@
 	(wire
 		(pts
-			(xy 215.9 78.74) (xy 228.6 78.74)
+			(xy 215.9 78.74) (xy 236.22 78.74)
 		)
 		(stroke
@@
 	(wire
 		(pts
+			(xy 40.64 73.66) (xy 48.26 73.66)
+		)
+		(stroke
+			(width 0)
+			(type default)
+		)
+	)
+	(wire
+		(pts
 			(xy 92.71 39.37) (xy 92.71 41.91)
 		)
@@
 	)
 	(symbol
-		(lib_id "Device:C")
-		(at 44.45 73.66 90)
-		(mirror x)
-		(unit 1)
-		(exclude_from_sim no)
-		(in_bom yes)
-		(on_board yes)
-		(dnp yes)
-		(property "Reference" "C401"
-			(at 44.45 78.74 90)
-			(effects
-				(font
-					(size 1.27 1.27)
-				)
-			)
-		)
-		(property "Value" "1u"
-			(at 44.45 81.28 90)
-			(effects
-				(font
-					(size 1.27 1.27)
-				)
-			)
-		)
-		(property "Footprint" "Capacitor_SMD:C_0805_2012Metric"
-			(at 48.26 74.6252 0)
-			(effects
-				(font
-					(size 1.27 1.27)
-				)
-				(hide yes)
-			)
-		)
-		(property "Datasheet" "~"
-			(at 44.45 73.66 0)
-			(effects
-				(font
-					(size 1.27 1.27)
-				)
-				(hide yes)
-			)
-		)
-		(property "Description" "Unpolarized capacitor"
-			(at 44.45 73.66 0)
-			(effects
-				(font
-					(size 1.27 1.27)
-				)
-				(hide yes)
-			)
-		)
-		(pin "1"
-		)
-		(pin "2"
-		)
-		(instances
-			(project "Main Board"
-				(path "/20aae4b7-3fb8-4924-82e8-1e7a29a313f8/6b7fef71-3444-4c8f-b2e2-502774ba9b51"
-					(reference "C401")
-					(unit 1)
-				)
-			)
-		)
-	)
-	(symbol
 		(lib_id "More_power:+18V")
 		(at 196.85 137.16 0)
@@
 					(unit 1)
 				)
-			)
-		)
-	)
-	(symbol
-		(lib_id "Device:C")
-		(at 232.41 78.74 90)
-		(mirror x)
-		(unit 1)
-		(exclude_from_sim no)
-		(in_bom yes)
-		(on_board yes)
-		(dnp yes)
-		(property "Reference" "C409"
-			(at 232.41 83.82 90)
-			(effects
-				(font
-					(size 1.27 1.27)
-				)
-			)
-		)
-		(property "Value" "1u"
-			(at 232.41 86.36 90)
-			(effects
-				(font
-					(size 1.27 1.27)
-				)
-			)
-		)
-		(property "Footprint" "Capacitor_SMD:C_0805_2012Metric"
-			(at 236.22 79.7052 0)
-			(effects
-				(font
-					(size 1.27 1.27)
-				)
-				(hide yes)
-			)
-		)
-		(property "Datasheet" "~"
-			(at 232.41 78.74 0)
-			(effects
-				(font
-					(size 1.27 1.27)
-				)
-				(hide yes)
-			)
-		)
-		(property "Description" "Unpolarized capacitor"
-			(at 232.41 78.74 0)
-			(effects
-				(font
-					(size 1.27 1.27)
-				)
-				(hide yes)
-			)
-		)
-		(pin "1"
-		)
-		(pin "2"
-		)
-		(instances
-			(project "Main Board"
-				(path "/20aae4b7-3fb8-4924-82e8-1e7a29a313f8/6b7fef71-3444-4c8f-b2e2-502774ba9b51"
-					(reference "C409")
-					(unit 1)
-				)

Commit message: please be nice
Parts:
- renumbered C402 to C401, C410 to C402, C411 to C404, C404 to C405, C405 to C406, C412 to C408, C414 to C409, C406 to C410, C408 to C411, C413 to C412, C415 to C413, D403 to D402, D402 to D403, Q403 to Q402, Q402 to Q403, R404 to R401, R406 to R402, R413 to R403, R407 to R404, R414 to R405, R402 to R406, R415 to R407, R401 to R409, R403 to R410, R409 to R411, R416 to R412, R405 to R413, R410 to R414, R411 to R415, R412 to R416, U404 to U401, U401 to U402, U405 to U403, U403 to U404, U402 to U405

Commit message: sleepdrunk
Connections:
- net DC_INT_ISO: now also U405.2 (I2); no longer U405.6 (I6)
- net DC_ISO: now also U405.15 (O2); no longer U405.11 (O6)
- net R_SEL_10: now also U405.3 (I3); no longer U405.1 (I1)
- net R_SEL_100: now also U405.4 (I4); no longer U405.2 (I2)
- net R_SEL_100k: now also U405.1 (I1); no longer U405.5 (I5)
- net R_SEL_10k: now also U405.6 (I6); no longer U405.4 (I4)
- net R_SEL_1k: now also U405.5 (I5); no longer U405.3 (I3)
- net SEL_10: now also U405.11 (O6); no longer U405.13 (O4)
- net SEL_100: now also U405.12 (O5); no longer U405.14 (O3)
- net SEL_100k: now also U405.16 (O1); no longer U405.12 (O5)
- net SEL_10k: now also U405.14 (O3); no longer U405.16 (O1)
- net SEL_1k: now also U405.13 (O4); no longer U405.15 (O2)
Changed lines of the file:
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@@
 	)
 	(label "SEL_1k"
-		(at 60.96 162.56 0)
+		(at 60.96 167.64 0)
 		(effects
 			(font
@@
 	)
 	(label "SEL_10"
-		(at 60.96 167.64 0)
+		(at 60.96 172.72 0)
 		(effects
 			(font
@@
 	)
 	(label "SEL_10k"
-		(at 60.96 160.02 0)
+		(at 60.96 165.1 0)
 		(effects
 			(font
@@
 	)
 	(label "SEL_100k"
+		(at 60.96 160.02 0)
+		(effects
+			(font
+				(size 1.27 1.27)
+			)
+			(justify left bottom)
+		)
+	)
+	(label "SEL_100"
 		(at 60.96 170.18 0)
 		(effects
@@
 		)
 	)
-	(label "SEL_100"
-		(at 60.96 165.1 0)
-		(effects
-			(font
-				(size 1.27 1.27)
-			)
-			(justify left bottom)
-		)
-	)
 	(label "DC_ISO"
-		(at 60.96 172.72 0)
+		(at 60.96 162.56 0)
 		(effects
 			(font
@@
 	(hierarchical_label "R_SEL_100k"
 		(shape input)
+		(at 40.64 160.02 180)
+		(effects
+			(font
+				(size 1.27 1.27)
+			)
+			(justify right)
+		)
+	)
+	(hierarchical_label "DC_INT_ISO"
+		(shape input)
+		(at 40.64 162.56 180)
+		(effects
+			(font
+				(size 1.27 1.27)
+			)
+			(justify right)
+		)
+	)
+	(hierarchical_label "R_SEL_1k"
+		(shape input)
 		(at 40.64 170.18 180)
-		(effects
-			(font
-				(size 1.27 1.27)
-			)
-			(justify right)
-		)
-	)
-	(hierarchical_label "DC_INT_ISO"
-		(shape input)
-		(at 40.64 172.72 180)
-		(effects
-			(font
-				(size 1.27 1.27)
-			)
-			(justify right)
-		)
-	)
-	(hierarchical_label "R_SEL_1k"
-		(shape input)
-		(at 40.64 165.1 180)
 		(effects
 			(font
@@
 	(hierarchical_label "R_SEL_10"
 		(shape input)
-		(at 40.64 160.02 180)
+		(at 40.64 165.1 180)
 		(effects
 			(font
@@
 	(hierarchical_label "R_SEL_10k"
 		(shape input)
+		(at 40.64 172.72 180)
+		(effects
+			(font
+				(size 1.27 1.27)
+			)
+			(justify right)
+		)
+	)
+	(hierarchical_label "AC_10k"
+		(shape input)
+		(at 123.19 85.09 180)
+		(effects
+			(font
+				(size 1.27 1.27)
+			)
+			(justify right)
+		)
+	)
+	(hierarchical_label "R_SEL_100"
+		(shape input)
 		(at 40.64 167.64 180)
 		(effects
 			(font
-				(size 1.27 1.27)
-			)
-			(justify right)
-		)
-	)
-	(hierarchical_label "AC_10k"
-		(shape input)
-		(at 123.19 85.09 180)
-		(effects
-			(font
-				(size 1.27 1.27)
-			)
-			(justify right)
-		)
-	)
-	(hierarchical_label "R_SEL_100"
-		(shape input)
-		(at 40.64 162.56 180)
-		(effects
-			(font

Commit message: Final Schematic
Parts:
- removed C406, C410: 100n, Capacitor_SMD:C_0805_2012Metric, symbol Device:C
- renumbered C401 to C22, C403 to C23, C405 to C24, C407 to C25, C411 to C26, C402 to C27, C404 to C28, C408 to C29, C412 to C30, C409 to C31, C413 to C32, D401 to D3, D403 to D4, D402 to D5, JP401 to JP8, K401 to K2, Q401 to Q4, Q403 to Q5, Q402 to Q6, Q404 to Q7, R409 to R30, R406 to R31, R410 to R32, R401 to R33, R413 to R34, R402 to R35, R404 to R36, R408 to R37, R411 to R38, R414 to R39, R415 to R40, R416 to R41, R403 to R42, R405 to R43, R407 to R44, R412 to R45, U401 to U10, U403 to U11, U402 to U7, U405 to U8, U404 to U9
Other:
- title: (none) -> Auto-Balancing Bridge
- moved on the sheet: C22, C23, C24, C25, C26, C29, C30, C31, C32, D3, D4, K2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

Commit message: cryingggggg
Connections:
- net DC_INT_ISO: now also U8.4 (I4); no longer U8.2 (I2)
- net DC_ISO: now also U8.13 (O4); no longer U8.15 (O2)
- net R_SEL_10: now also U8.6 (I6); no longer U8.3 (I3)
- net R_SEL_100: now also U8.5 (I5); no longer U8.4 (I4)
- net R_SEL_100k: now also U8.3 (I3); no longer U8.1 (I1)
- net R_SEL_10k: now also U8.1 (I1); no longer U8.6 (I6)
- net R_SEL_1k: now also U8.2 (I2); no longer U8.5 (I5)
- net SEL_100k: now also U8.14 (O3); no longer U8.16 (O1)
- net SEL_10k: now also U8.16 (O1); no longer U8.14 (O3)
- net SEL_1k: now also U8.15 (O2); no longer U8.13 (O4)
Changed lines of the file:
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@@
 	)
 	(label "SEL_1k"
-		(at 60.96 175.26 0)
+		(at 60.96 170.18 0)
 		(effects
 			(font
@@
 	)
 	(label "SEL_10k"
-		(at 60.96 172.72 0)
+		(at 60.96 167.64 0)
 		(effects
 			(font
@@
 	)
 	(label "SEL_100k"
-		(at 60.96 167.64 0)
+		(at 60.96 172.72 0)
 		(effects
 			(font
@@
 	)
 	(label "DC_ISO"
-		(at 60.96 170.18 0)
+		(at 60.96 175.26 0)
 		(effects
 			(font
@@
 	(hierarchical_label "R_SEL_100k"
 		(shape input)
-		(at 40.64 167.64 180)
+		(at 40.64 172.72 180)
 		(effects
 			(font
@@
 	(hierarchical_label "DC_INT_ISO"
 		(shape input)
+		(at 40.64 175.26 180)
+		(effects
+			(font
+				(size 1.27 1.27)
+			)
+			(justify right)
+		)
+	)
+	(hierarchical_label "R_SEL_1k"
+		(shape input)
 		(at 40.64 170.18 180)
-		(effects
-			(font
-				(size 1.27 1.27)
-			)
-			(justify right)
-		)
-	)
-	(hierarchical_label "R_SEL_1k"
-		(shape input)
-		(at 40.64 177.8 180)
 		(effects
 			(font
@@
 	(hierarchical_label "R_SEL_10"
 		(shape input)
-		(at 40.64 172.72 180)
+		(at 40.64 180.34 180)
 		(effects
 			(font
@@
 	(hierarchical_label "R_SEL_10k"
 		(shape input)
-		(at 40.64 180.34 180)
+		(at 40.64 167.64 180)
 		(effects
 			(font
@@
 	(hierarchical_label "R_SEL_100"
 		(shape input)
-		(at 40.64 175.26 180)
-		(effects
-			(font
+		(at 40.64 177.8 180)
+		(effects
+			(font
