File: PCB/Main Board/Main Board.kicad_pcb (KiCad board)
At the start: 2 copper layers, 152.4 x 134.6 mm, 251 parts, among them J101 Conn_Coaxial, J102 Conn_Coaxial, J103 Conn_Coaxial, J104 Conn_Coaxial, J105 Conn_01x01_Pin, J201 USB_C_Receptacle_USB2.0_16P, J801 Conn_01x03_Pin, J802 Screw_Terminal_01x03, K301 AGQ200A12, K401 AGQ200A12, K501 AGQ200A12, K502 AGQ200A12, K503 AGQ200A12, K504 AGQ200A12, K505 AGQ200A12, Q301 2N4401, Q302 2N4403, Q401 2N4401, Q402 2N4403, Q403 2N4401, Q404 2N4403, SW201 SW_Push, SW202 SW_Push, U201 USBLC6-2SC6, U202 STM32F446RETx, U203 ULN2003, U301 DG201, U302 OPA2197xD, U303 OPA2376xxD, U304 OPA2197xD, U401 OPA2197xD, U402 DG201, U403 OPA2197xD, U404 OPA2197xD, U601 INA828D, U602 DG201, U603 OPA2197xD, U604 DG201, U605 OPA2376xxD, U701 INA828D, U702 DG201, U703 OPA2376xxD, U801 LM317_SOT-223, U802 LM317_SOT-223, U803 LM317_SOT-223, U804 LM337_SOT223, Y201 8MHz

Commit message: checkpoint
Parts:
- removed RN301: 4610X-R2R-103LF, Resistor_THT:R_Array_SIP10
- C501: value 100n -> 16n
- C502: value 100n -> 1.6n
- C503: value 100n -> 160p
- C504, C505: value 100n -> 330p
- C506: value 100n -> 56p
- Q301: value 2N4401 -> TIP41C
- Q302: value 2N4403 -> TIP42C
- Q401, Q403: value 2N4401 -> TIP42C
- Q402, Q404: value 2N4403 -> TIP41C
- moved C408 75.4 mm to (65.5, 59.7)
- moved C803 71.5 mm to (44.0, -28.5)
- moved C804 71.5 mm to (44.0, -23.8)
- moved C801 71.5 mm to (40.6, -28.5)
- moved C802 71.5 mm to (40.6, -23.8)
- moved D801 71.5 mm to (36.1, -31.3)
- moved D802 71.5 mm to (36.1, -21.5)
- moved J801 71.5 mm to (35.1, -28.4)
- moved J802 71.5 mm to (29.3, -29.9)
- moved C409 61.4 mm to (61.5, 67.3)
- moved R401 61.2 mm to (51.2, 65.1)
- moved R404 61.2 mm to (51.2, 61.0)
- moved U401 59.3 mm to (63.5, 63.5)
- moved U402 59.3 mm to (63.5, 50.8)
- moved R411 59.1 mm to (73.7, 62.5)
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Connections:
- D401 pad 1: Net-(Q401-B) -> Net-(Q402-B)
- D403 pad 1: Net-(Q403-B) -> Net-(Q404-B)
- Q301 pad 1: Net-(Q301-E) -> Net-(Q301-B)
- Q301 pad 2: Net-(Q301-B) -> +18V
- Q301 pad 3: +18V -> Net-(Q301-E)
- Q302 pad 1: Net-(Q301-E) -> Net-(D301-A)
- Q302 pad 2: Net-(D301-A) -> -18V
- Q302 pad 3: -18V -> Net-(Q301-E)
- Q401 pad 1: Net-(Q401-E) -> Net-(D401-A)
- Q401 pad 2: Net-(Q401-B) -> -18V
- Q401 pad 3: +18V -> Net-(Q401-E)
- Q402 pad 1: Net-(Q401-E) -> Net-(Q402-B)
- Q402 pad 2: Net-(D401-A) -> +18V
- Q402 pad 3: -18V -> Net-(Q401-E)
- Q403 pad 1: /Auto-Balancing Bridge/OUT+ -> Net-(D403-A)
- Q403 pad 2: Net-(Q403-B) -> -18V
- Q403 pad 3: +18V -> /Auto-Balancing Bridge/OUT+
- Q404 pad 1: /Auto-Balancing Bridge/OUT+ -> Net-(Q404-B)
- Q404 pad 2: Net-(D403-A) -> +18V
- Q404 pad 3: -18V -> /Auto-Balancing Bridge/OUT+
- R402 pad 2: Net-(Q401-B) -> Net-(Q402-B)
- R415 pad 2: Net-(Q403-B) -> Net-(Q404-B)
- U402 pad 14: Net-(R409-Pad2) -> /Auto-Balancing Bridge/OUT+
- U402 pad 15: /Auto-Balancing Bridge/OUT+ -> Net-(R409-Pad2)
Routing:
- net GUARD: track 277.4 -> 339.2 mm
- net Net-(U401B--): track 0.00 -> 51.8 mm
- net Net-(C405-Pad1): track 0.00 -> 43.8 mm
- net Net-(R409-Pad2): track 0.00 -> 30.9 mm
- net Net-(R411-Pad2): track 0.00 -> 30.0 mm
- net Net-(R410-Pad2): track 0.00 -> 22.9 mm
- net /Auto-Balancing Bridge/In: track 80.7 -> 103.2 mm
- net /Auto-Balancing Bridge/OUT+: track 113.8 -> 128.2 mm, vias 0 -> 2
- net Net-(C504-Pad2): track 0.00 -> 10.6 mm
- net +12V: track 65.7 -> 70.2 mm
- net Net-(C505-Pad2): track 7.37 -> 6.07 mm
Other:
- board text removed: "Power Supply"

Commit message: Cryiunbg
Parts:
- added R405: 100m, Resistor_SMD:R_0805_2012Metric, F.Cu at (38.1, 81.3)
- added R406: 100m, Resistor_SMD:R_0805_2012Metric, F.Cu at (38.1, 84.2)
- added R419: 100m, Resistor_SMD:R_0805_2012Metric, F.Cu at (91.4, 97.8)
- added R420: 100m, Resistor_SMD:R_0805_2012Metric, F.Cu at (91.4, 100.7)
- moved JP304 252.0 mm to (217.0, 132.1)
- moved R301 222.0 mm to (212.1, 94.9)
- moved R302 222.0 mm to (212.1, 97.8)
- moved R305 222.0 mm to (212.1, 91.9)
- moved J802 153.4 mm to (170.6, 29.8), turned to 180 degrees
- moved D801 151.9 mm to (172.0, 36.6), turned to -90 degrees
- moved J801 148.5 mm to (169.1, 35.6), turned to -90 degrees
- moved C801 146.2 mm to (169.2, 41.1), turned to 0 degrees
- moved C803 144.9 mm to (169.2, 44.5), turned to 0 degrees
- moved C802 139.8 mm to (164.5, 41.1), turned to 0 degrees
- moved D802 138.9 mm to (162.2, 36.6), turned to 90 degrees
- moved C804 138.5 mm to (164.5, 44.5), turned to 0 degrees
- moved C808 62.0 mm to (152.7, 45.8)
- moved R804 62.0 mm to (144.6, 40.1)
- moved R807 62.0 mm to (132.6, 34.4)
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- renumbered C404 to C402, C402 to C403, C403 to C404, C413 to C411, C411 to C412, C412 to C413, Q402 to Q401, Q401 to Q402, Q404 to Q403, Q403 to Q404, R405 to R407, R406 to R408, R407 to R409, R408 to R410, R409 to R411, R410 to R412, R411 to R413, R412 to R414, R413 to R415, R414 to R416, R415 to R417, R416 to R418
Connections:
- K401 pad 2: GUARD -> unconnected-(K401-Pad2)
- K401 pad 3: Net-(U403A-+) -> unconnected-(K401-Pad3)
- K401 pad 4: /Auto-Balancing Bridge/In -> unconnected-(K401-Pad4)
- K401 pad 5: unconnected-(K401-Pad5) -> /Auto-Balancing Bridge/In
- K401 pad 6: unconnected-(K401-Pad6) -> Net-(U403A-+)
- K401 pad 7: unconnected-(K401-Pad7) -> GUARD
- Q402 pad 3: Net-(Q401-E) -> Net-(Q402-E)
- Q403 pad 3: /Auto-Balancing Bridge/OUT+ -> Net-(Q403-E)
- Q404 pad 3: /Auto-Balancing Bridge/OUT+ -> Net-(Q404-E)
- R404 pad 2: Net-(Q401-E) -> Net-(R404-Pad2)
- R409 pad 2: Net-(Q401-E) -> Net-(R404-Pad2)
- R410 pad 1: Net-(Q401-E) -> Net-(R404-Pad2)
Routing:
- net GUARD: track 339.2 -> 239.9 mm
- net Net-(Q401-E): track 32.2 -> 0.00 mm
- net Net-(R404-Pad2): track 0.00 -> 27.8 mm
- net Net-(U403A-+): track 27.4 -> 0.00 mm
- net /Auto-Balancing Bridge/In: track 103.2 -> 80.1 mm
- net Net-(C505-Pad2): track 6.07 -> 2.05 mm
Other:
- board text added: "Power Supply"

Commit message: eek
Parts:
- moved U203 40.5 mm to (63.5, 38.1)
- moved JP401 18.4 mm to (55.9, 101.6), turned to -90 degrees
- moved R410 10.5 mm to (96.5, 120.0)
- moved R505 6.50 mm to (64.8, 122.9), turned to 0 degrees
- moved C505 3.63 mm to (64.8, 120.9), turned to 0 degrees
Routing:
- net GUARD: track 239.9 -> 428.7 mm
- net /Voltage Amplifier/In+: track 8.31 -> 30.8 mm
- net /Auto-Balancing Bridge/In: track 80.1 -> 100.5 mm
- net Net-(U403A-+): track 0.00 -> 13.6 mm
- net /Voltage Amplifier/In-: track 37.7 -> 50.4 mm
- net Net-(C505-Pad2): track 2.05 -> 9.38 mm
- net /Auto-Balancing Bridge/OUT+: track 128.2 -> 131.8 mm
- net Net-(JP401-A): track 4.00 -> 7.57 mm
- net Net-(R404-Pad2): track 27.8 -> 25.1 mm

Commit message: resistor footprints changed
Parts:
- added R305: 10, Resistor_SMD:R_2512_6332Metric, F.Cu at (234.9, 91.5)
- added R307: 10, Resistor_SMD:R_2512_6332Metric, F.Cu at (234.9, 96.4)
- added R308: 10, Resistor_SMD:R_2512_6332Metric, F.Cu at (234.9, 101.3)
- added R502: 10, Resistor_SMD:R_2512_6332Metric, F.Cu at (224.2, 96.4)
- added R503: 10, Resistor_SMD:R_2512_6332Metric, F.Cu at (224.2, 101.3)
- added R504: 10, Resistor_SMD:R_2512_6332Metric, F.Cu at (224.2, 106.2)
- added RN301: R_Pack08, Package_SO:SOIC-16_3.9x9.9mm_P1.27mm, F.Cu at (243.5, 94.9)
- R304: renamed from R315; footprint Resistor_THT:R_Axial_DIN0516_L15.5mm_D5.0mm_P20.32mm_Horizontal -> Resistor_SMD:R_2512_6332Metric
- R501: footprint Resistor_THT:R_Axial_DIN0516_L15.5mm_D5.0mm_P20.32mm_Horizontal -> Resistor_SMD:R_2512_6332Metric
- moved R501 157.3 mm to (224.2, 91.5), turned to 0 degrees
- moved R304 35.8 mm to (234.9, 106.4), turned to 0 degrees
- renumbered C209 to C201, C204 to C202, C201 to C203, C202 to C204, C203 to C205, C205 to C206, C206 to C207, C207 to C208, C208 to C209, C311 to C301, C312 to C302, C302 to C303, C301 to C304, C313 to C305, C314 to C306, C315 to C307, C303 to C308, C305 to C309, C307 to C310, C309 to C311, C304 to C312, C306 to C313, C308 to C314, C310 to C315, C403 to C402, C410 to C403, C412 to C404, C402 to C405, C404 to C406, C411 to C407, C413 to C408, C405 to C409, C406 to C410, C408 to C411, C414 to C412, C416 to C413, C407 to C414, C409 to C415, C415 to C416, C602 to C601, C614 to C602, C613 to C604, C604 to C605, C605 to C606, C609 to C608, C611 to C609, C615 to C610, C606 to C611, C608 to C612, C610 to C613, C612 to C614, C616 to C615, C601 to C616, C703 to C701, C711 to C702, C704 to C703, C710 to C704, C701 to C706, C706 to C707, C702 to C709, C707 to C710, C709 to C711, C805 to C801, C809 to C802, C806 to C803, C810 to C804, C801 to C805, C803 to C806, C802 to C807, C804 to C808, C807 to C809, C811 to C810, C808 to C811, D403 to D402, D402 to D403, D803 to D801, D801 to D802, D802 to D803, J105 to J101, J101 to J102, J102 to J103, J103 to J104, J104 to J105, J802 to J801, J801 to J802, JP203 to JP202, JP202 to JP203, JP304 to JP301, JP303 to JP302, JP301 to JP303, JP302 to JP304, JP603 to JP601, JP604 to JP602, JP601 to JP603, JP602 to JP604, K505 to K501, K504 to K502, K502 to K504, K501 to K505, Q403 to Q402, Q402 to Q403, R205 to R204, R206 to R205, R207 to R206, R208 to R207, R204 to R208, R307 to R301, R311 to R302, R308 to R303, R309 to R306, R312 to R309, R306 to R310, R310 to R311, R304 to R312, R316 to R313, R303 to R314, R305 to R315, R301 to R316, R313 to R317, R302 to R318, R314 to R319, R404 to R401, R408 to R402, R415 to R403, R409 to R404, R416 to R405, R402 to R406, R417 to R407, R405 to R408, R401 to R409, R419 to R411, R406 to R412, R420 to R413, R411 to R414, R403 to R415, R418 to R416, R407 to R417, R412 to R418, R413 to R419, R414 to R420, R502 to R505, R503 to R506, R504 to R507, R505 to R508, R506 to R509, R609 to R601, R612 to R602, R601 to R603, R610 to R605, R613 to R606, R616 to R607, R617 to R608, R619 to R609, R602 to R610, R620 to R612, R618 to R613, R608 to R616, R603 to R617, R605 to R618, R606 to R619, R607 to R620, R704 to R701, R707 to R702, R701 to R703, R703 to R704, R708 to R706, R709 to R707, R710 to R708, R711 to R709, R702 to R710, R706 to R711, R805 to R801, R801 to R802, R806 to R803, R802 to R804, R807 to R805, R809 to R806, R803 to R807, R804 to R808, R808 to R809, SW202 to SW201, SW201 to SW202, U302 to U301, U301 to U302, U304 to U303, U303 to U304, U403 to U401, U401 to U402, U404 to U403, U402 to U404, U604 to U601, U601 to U602, U605 to U603, U603 to U604, U602 to U605, U702 to U701, U701 to U702
Connections:
- R304 pad 2: Net-(K301-Pad2) -> Net-(R304-Pad2)
- R501 pad 2: Net-(C501-Pad2) -> Net-(R501-Pad2)
Routing:
- net Net-(U303A--): track 0.00 -> 17.9 mm
- net Net-(RN301-R1.2): track 17.9 -> 0.00 mm

Commit message: merge
Parts:
- removed the R305 at (234.9, 91.5)
- removed the R307 at (234.9, 96.4)
- removed the R308 at (234.9, 101.3)
- removed the R503 at (224.2, 101.3)
- removed the R504 at (224.2, 106.2)
- added R316: 10, Resistor_SMD:R_2512_6332Metric, F.Cu at (247.8, 88.1)
- added R318: 10, Resistor_SMD:R_2512_6332Metric, F.Cu at (247.8, 93.0)
- added R319: 10, Resistor_SMD:R_2512_6332Metric, F.Cu at (247.8, 97.9)
- added R508: 10, Resistor_SMD:R_2512_6332Metric, F.Cu at (237.1, 97.9)
- added R509: 10, Resistor_SMD:R_2512_6332Metric, F.Cu at (237.1, 102.9)
- moved R405 65.8 mm to (93.5, 116.8), turned to 180 degrees
- moved R406 59.2 mm to (93.5, 105.2)
- moved R420 57.0 mm to (34.9, 93.2)
- moved R419 55.8 mm to (38.1, 81.3)
- moved Q401 46.2 mm to (100.0, 111.8), turned to -90 degrees
- moved C403 44.6 mm to (93.5, 114.8), turned to 0 degrees
- moved C401 44.0 mm to (93.5, 112.8), turned to 0 degrees
- moved R402 39.0 mm to (93.5, 110.7), turned to 0 degrees
- moved Q403 38.2 mm to (67.7, 78.7), turned to 90 degrees
- moved Q404 38.2 mm to (67.7, 91.4), turned to 90 degrees
- moved R315 35.8 mm to (218.4, 138.2), turned to -90 degrees
- moved Q402 33.2 mm to (100.0, 99.1), turned to -90 degrees
- moved K401 15.3 mm to (82.5, 134.6)
- moved D402 15.2 mm to (73.7, 102.2), turned to 180 degrees
- moved D401 14.4 mm to (93.5, 108.0), turned to 180 degrees
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- renumbered C203 to C201, C204 to C202, C205 to C203, C202 to C204, C206 to C205, C207 to C206, C208 to C207, C209 to C208, C201 to C209, C304 to C301, C303 to C302, C308 to C303, C312 to C304, C309 to C305, C313 to C306, C310 to C307, C314 to C308, C311 to C309, C315 to C310, C301 to C311, C302 to C312, C305 to C313, C306 to C314, C307 to C315, C405 to C402, C402 to C403, C406 to C404, C409 to C405, C410 to C406, C414 to C407, C411 to C408, C415 to C409, C403 to C410, C407 to C411, C404 to C412, C408 to C413, C412 to C414, C416 to C415, C413 to C416, C616 to C601, C601 to C602, C605 to C604, C606 to C605, C611 to C606, C612 to C608, C608 to C609, C613 to C610, C609 to C611, C614 to C612, C604 to C613, C602 to C614, C610 to C615, C615 to C616, C706 to C701, C709 to C702, C701 to C703, C703 to C704, C707 to C706, C710 to C707, C711 to C709, C704 to C710, C702 to C711, C805 to C801, C807 to C802, C806 to C803, C808 to C804, C801 to C805, C803 to C806, C809 to C807, C811 to C808, C802 to C809, C804 to C810, C810 to C811, D403 to D402, D402 to D403, D802 to D801, D803 to D802, D801 to D803, J102 to J101, J103 to J102, J104 to J103, J105 to J104, J101 to J105, J802 to J801, J801 to J802, JP203 to JP202, JP202 to JP203, JP303 to JP301, JP304 to JP302, JP302 to JP303, JP301 to JP304, JP603 to JP601, JP604 to JP602, JP601 to JP603, JP602 to JP604, K505 to K501, K504 to K502, K502 to K504, K501 to K505, Q403 to Q402, Q402 to Q403, R208 to R204, R204 to R205, R205 to R206, R206 to R207, R207 to R208, R316 to R301, R318 to R302, R314 to R303, R312 to R304, R315 to R305, R310 to R306, R301 to R307, R303 to R308, R306 to R309, R311 to R310, R302 to R311, R309 to R312, R317 to R313, R319 to R314, R304 to R315, R313 to R317, R409 to R401, R406 to R402, R415 to R403, R401 to R404, R408 to R405, R412 to R406, R417 to R407, R402 to R408, R404 to R409, R414 to R411, R418 to R412, R419 to R413, R420 to R414, R403 to R415, R405 to R416, R407 to R417, R416 to R418, R411 to R419, R413 to R420, R505 to R503, R506 to R504, R507 to R505, R508 to R506, R509 to R507, R603 to R601, R610 to R602, R617 to R603, R618 to R605, R619 to R606, R620 to R607, R616 to R608, R601 to R609, R605 to R610, R602 to R612, R606 to R613, R607 to R616, R608 to R617, R613 to R618, R609 to R619, R612 to R620, R703 to R701, R710 to R702, R704 to R703, R701 to R704, R711 to R706, R702 to R707, R706 to R708, R707 to R709, R708 to R710, R709 to R711, R802 to R801, R804 to R802, R807 to R803, R808 to R804, R801 to R805, R803 to R806, R805 to R807, R809 to R808, R806 to R809, SW202 to SW201, SW201 to SW202, U302 to U301, U301 to U302, U304 to U303, U303 to U304, U402 to U401, U404 to U402, U401 to U403, U403 to U404, U602 to U601, U605 to U602, U604 to U603, U601 to U604, U603 to U605, U702 to U701, U701 to U702
Connections:
- R502 pad 1: Net-(R501-Pad2) -> /Auto-Balancing Bridge/In
- R502 pad 2: Net-(C501-Pad2) -> Net-(R502-Pad2)
Routing:
- net GUARD: track 428.7 -> 350.0 mm
- net (no net): track 38.1 -> 55.9 mm
- net Net-(U304A--): track 17.9 -> 0.00 mm
- net Net-(D401-A): track 0.00 -> 17.8 mm
- net /Auto-Balancing Bridge/In: track 100.5 -> 88.7 mm
- net /Auto-Balancing Bridge/OUT+: track 131.8 -> 143.0 mm, vias 2 -> 4
- net +18V: track 31.7 -> 42.3 mm
- net -18V: track 31.1 -> 41.7 mm
- net Net-(Q401-B): track 0.00 -> 7.88 mm
- net Net-(Q402-E): track 0.00 -> 6.03 mm
- net Net-(Q401-E): track 0.00 -> 5.61 mm
- net Net-(U403A-+): track 13.6 -> 10.9 mm

Commit message: merge 2.0
Parts:
- removed C402, C403, C411, C412: 100n, Capacitor_SMD:C_0805_2012Metric
- moved C413 51.9 mm to (73.7, 95.8)
- moved R315 43.7 mm to (247.7, 105.7)
- moved R420 42.1 mm to (77.0, 93.7)
- moved R419 36.0 mm to (73.7, 75.7)
- moved C410 11.9 mm to (73.7, 77.7), turned to 180 degrees
- moved C404 4.06 mm to (93.5, 103.1)
- moved R417 2.30 mm to (73.7, 79.8), turned to 180 degrees
- moved R403 2.03 mm to (93.5, 101.1)
Routing:
- net Net-(D401-A): track 17.8 -> 0.00 mm
- net -18V: track 41.7 -> 34.7 mm
- net Net-(Q403-B): track 0.00 -> 1.85 mm

Commit message: co-op test
Parts:
- moved R313 5.08 mm to (183.1, 152.3)
- moved D301 5.08 mm to (177.8, 152.1)
- moved R312 5.08 mm to (172.2, 152.1)
Changed lines of the file:
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@@
 	(footprint "Package_TO_SOT_SMD:SOT-23"
 		(layer "F.Cu")
-		(at 177.8 146.987501 90)
+		(at 177.8 152.067501 90)
 		(descr "SOT, 3 Pin (JEDEC TO-236 Var AB https://www.jedec.org/document_search?search_api_views_fulltext=TO-236), generated with kicad-footprint-generator ipc_gullwing_generator.py")
 		(tags "SOT TO_SOT_SMD")
@@
 	(footprint "Resistor_SMD:R_0805_2012Metric"
 		(layer "F.Cu")
-		(at 183.114668 147.241501 90)
+		(at 183.114668 152.321501 90)
 		(descr "Resistor SMD 0805 (2012 Metric), square (rectangular) end terminal, IPC-7351 nominal, (Body size source: IPC-SM-782 page 72, https://www.pcb-3d.com/wordpress/wp-content/uploads/ipc-sm-782a_amendment_1_and_2.pdf), generated with kicad-footprint-generator")
 		(tags "resistor")
@@
 	(footprint "Resistor_SMD:R_0805_2012Metric"
 		(layer "F.Cu")
-		(at 172.192668 146.987501 -90)
+		(at 172.192668 152.067501 -90)
 		(descr "Resistor SMD 0805 (2012 Metric), square (rectangular) end terminal, IPC-7351 nominal, (Body size source: IPC-SM-782 page 72, https://www.pcb-3d.com/wordpress/wp-content/uploads/ipc-sm-782a_amendment_1_and_2.pdf), generated with kicad-footprint-generator")
 		(tags "resistor")

Commit message: YIPEE
Parts:
- moved R418 10.7 mm to (73.7, 89.4), turned to 0 degrees
- moved R420 9.01 mm to (73.7, 85.3), turned to 180 degrees
- moved C413 8.38 mm to (73.7, 87.4)
- moved R405 2.03 mm to (93.5, 114.8)
Routing:
- net /Auto-Balancing Bridge/OUT+: track 143.0 -> 206.3 mm
- net Net-(D403-A): track 0.00 -> 24.4 mm
- net Net-(D401-A): track 0.00 -> 23.8 mm
- net -18V: track 34.7 -> 48.6 mm
- net +18V: track 42.3 -> 49.2 mm
- net Net-(Q404-E): track 0.00 -> 5.52 mm
- net Net-(Q401-E): track 5.61 -> 6.45 mm
