File: PCB/Main Board/Main Board.kicad_pcb (KiCad board)
At the start: 2 copper layers, 152.4 x 134.6 mm, 261 parts, among them J101 Conn_Coaxial, J102 Conn_Coaxial, J103 Conn_Coaxial, J104 Conn_Coaxial, J105 Conn_01x01_Pin, J201 USB_C_Receptacle_USB2.0_16P, J801 Conn_01x03_Pin, J802 Screw_Terminal_01x03, K301 AGQ200A12, K401 AGQ200A12, K501 AGQ200A12, K502 AGQ200A12, K503 AGQ200A12, K504 AGQ200A12, K505 AGQ200A12, Q301 2N7002, Q302 TIP41C, Q303 TIP42C, Q401 TIP41C, Q402 TIP42C, Q403 TIP41C, Q404 TIP42C, SW201 SW_Push, SW202 SW_Push, U201 USBLC6-2SC6, U202 STM32F446RETx, U301 DG201, U302 OPA2197xD, U303 OPA2376xxD, U304 OPA2197xD, U401 OPA2197xD, U402 ULN2003, U403 DG201, U404 OPA2197xD, U405 OPA2197xD, U601 INA828D, U602 DG201, U603 OPA2197xD, U604 DG201, U605 OPA2376xxD, U701 INA828D, U702 DG201, U703 OPA2376xxD, U801 LM317_SOT-223, U802 LM317_SOT-223, U803 LM317_SOT-223, U804 LM337_SOT223, Y201 8MHz

Commit message: asdfjkhhjk
Parts:
- moved JP604 15.4 mm to (137.7, 95.2)
- moved JP603 5.89 mm to (141.7, 82.5), turned to 180 degrees
Connections:
- U202 pad 59: unconnected-(U202-PB7-Pad59) -> /Current Amplifier/x3
- U202 pad 61: unconnected-(U202-PB8-Pad61) -> /Current Amplifier/x1
- U202 pad 62: unconnected-(U202-PB9-Pad62) -> /Current Amplifier/~{x100}
- U202 pad 8: unconnected-(U202-PC0-Pad8) -> /Current Amplifier//4
Routing:
- net +18V: track 282.0 -> 339.8 mm, vias 14 -> 15
- net -18V: track 278.4 -> 324.9 mm, vias 12 -> 14
- net Net-(U603B--): track 17.2 -> 43.6 mm, vias 0 -> 5
- net unconnected-(U202-PC0-Pad8): track 19.3 -> 0.00 mm
- net /Current Amplifier//4: track 0.00 -> 19.3 mm
- net Net-(C603-Pad1): track 40.5 -> 28.7 mm, vias 2 -> 0
- net Net-(R601-Pad1): track 56.6 -> 67.3 mm, vias 2 -> 5
- net Net-(JP601-A): track 0.00 -> 10.6 mm
- net Net-(JP603-C): track 0.00 -> 5.42 mm
- net Net-(JP604-C): track 0.00 -> 5.42 mm
- net Net-(JP301-C): track 0.00 -> 2.45 mm
- net Net-(C602-Pad1): track 15.6 -> 17.4 mm

Commit message: Krill me
Parts:
- removed C401, C409: 1u, Capacitor_SMD:C_0805_2012Metric
- moved C204 190.6 mm to (207.2, 81.4)
- moved C209 190.6 mm to (207.2, 78.4)
- moved R201 190.6 mm to (202.8, 80.2)
- moved R202 190.6 mm to (202.8, 83.1)
- moved R203 190.6 mm to (202.8, 86.1)
- moved R204 190.6 mm to (213.3, 50.1)
- moved R205 190.6 mm to (202.8, 68.4)
- moved R206 190.6 mm to (202.8, 71.3)
- moved R207 190.6 mm to (202.8, 74.3)
- moved R208 190.6 mm to (202.8, 77.2)
- moved SW201 190.6 mm to (202.5, 59.2)
- moved SW202 190.6 mm to (202.5, 50.6)
- moved C402 51.4 mm to (90.2, 96.8)
- moved C403 48.4 mm to (85.8, 97.8)
- moved C410 43.4 mm to (72.8, 73.4)
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Connections:
- D401 pad 3: Net-(C401-Pad2) -> Net-(D401-K-Pad3)
- D403 pad 3: Net-(C409-Pad2) -> Net-(D403-K-Pad3)
- U401 pad 1: Net-(C401-Pad1) -> Net-(D401-K-Pad3)
- U405 pad 7: Net-(C409-Pad1) -> Net-(D403-K-Pad3)
Routing:
- net Net-(D403-K-Pad3): track 0.00 -> 34.7 mm, vias 0 -> 2
- net (no net): track 34.7 -> 0.00 mm, vias 2 -> 0
- net /Auto-Balancing Bridge/OUT+: track 211.1 -> 238.9 mm
- net /Auto-Balancing Bridge/AC_100: track 79.4 -> 80.4 mm
- net Net-(R411-Pad2): track 30.0 -> 29.0 mm

Commit message: please be nice
Parts:
- removed the C204 at (207.2, 81.4)
- removed the C205 at (165.2, 64.2)
- removed C210: 100n, Capacitor_SMD:C_0805_2012Metric
- removed the R801 at (122.9, 40.7)
- removed the R802 at (87.4, 40.7)
- removed the R803 at (161.1, 40.7)
- removed the R804 at (105.2, 40.7)
- added J202: Conn_01x05_Pin, Connector_PinHeader_2.54mm:PinHeader_1x05_P2.54mm_Vertical, F.Cu at (193.3, 60.2)
- added RV801: 10k, Potentiometer_SMD:Potentiometer_Bourns_3214W_Vertical, F.Cu at (123.2, 40.8)
- added RV802: 10k, Potentiometer_SMD:Potentiometer_Bourns_3214W_Vertical, F.Cu at (87.6, 40.7)
- added RV803: 10k, Potentiometer_SMD:Potentiometer_Bourns_3214W_Vertical, F.Cu at (156.2, 40.8)
- added RV804: 5k, Potentiometer_SMD:Potentiometer_Bourns_3214W_Vertical, F.Cu at (105.4, 40.7)
- J101: renamed from J105; footprint Connector_PinHeader_2.54mm:PinHeader_1x01_P2.54mm_Vertical -> Connector_PinHeader_2.54mm:PinHeader_1x01_P2.54mm_Horizontal
- J802: renamed from J801; footprint Connector_PinHeader_2.00mm:PinHeader_1x03_P2.00mm_Vertical -> Connector_PinHeader_2.54mm:PinHeader_1x03_P2.54mm_Vertical
- JP203: value SolderJumper_2_Bridged -> SolderJumper_2_Open; footprint Jumper:SolderJumper-2_P1.3mm_Bridged_RoundedPad1.0x1.5mm -> Jumper:SolderJumper-2_P1.3mm_Open_RoundedPad1.0x1.5mm
- moved C201 81.6 mm to (127.0, 63.6)
- moved R207 80.5 mm to (123.5, 63.6), turned to 180 degrees
- moved SW201 79.7 mm to (123.1, 56.6)
- moved R204 50.2 mm to (152.9, 73.8), turned to 180 degrees
- moved R206 50.1 mm to (152.9, 69.7), turned to 180 degrees
- moved R205 49.9 mm to (152.9, 71.8), turned to 180 degrees
- moved R201 44.8 mm to (175.5, 44.7), turned to -90 degrees
- moved JP203 44.3 mm to (191.4, 38.0)
- moved R202 40.3 mm to (191.2, 44.5)
- moved R203 40.3 mm to (191.2, 47.4)
- moved C203 39.9 mm to (126.9, 71.1), turned to 90 degrees
- moved C202 39.8 mm to (126.9, 67.6), turned to -90 degrees
- moved C208 39.7 mm to (130.5, 63.6), turned to 180 degrees
- moved RN301 39.5 mm to (165.5, 58.7)
- moved R208 35.6 mm to (178.2, 56.2), turned to -90 degrees
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- renumbered C209 to C201, C201 to C202, C202 to C203, C203 to C204, C206 to C205, C207 to C206, C208 to C207, C211 to C208, C312 to C301, C311 to C303, C301 to C304, C313 to C305, C314 to C306, C303 to C307, C305 to C308, C307 to C309, C309 to C310, C304 to C311, C306 to C312, C308 to C313, C310 to C314, C402 to C401, C410 to C402, C411 to C404, C404 to C405, C405 to C406, C412 to C408, C414 to C409, C406 to C410, C408 to C411, C413 to C412, C415 to C413, C602 to C601, C614 to C602, C613 to C604, C604 to C605, C605 to C606, C609 to C608, C611 to C609, C615 to C610, C606 to C611, C608 to C612, C610 to C613, C612 to C614, C616 to C615, C601 to C616, C703 to C701, C711 to C702, C704 to C703, C710 to C704, C701 to C706, C706 to C707, C702 to C709, C707 to C710, C709 to C711, C805 to C801, C809 to C802, C806 to C803, C810 to C804, C801 to C805, C803 to C806, C802 to C807, C804 to C808, C807 to C809, C811 to C810, C808 to C811, D403 to D402, D402 to D403, D803 to D801, D801 to D802, D802 to D803, J101 to J102, J102 to J103, J103 to J104, J104 to J105, J802 to J801, JP304 to JP301, JP303 to JP302, JP301 to JP303, JP302 to JP304, JP603 to JP601, JP604 to JP602, JP601 to JP603, JP602 to JP604, K505 to K501, K504 to K502, K502 to K504, K501 to K505, Q302 to Q301, Q303 to Q302, Q301 to Q303, Q403 to Q402, Q402 to Q403, R205 to R204, R206 to R205, R207 to R206, R208 to R207, R204 to R208, R307 to R301, R313 to R302, R308 to R303, R315 to R304, R319 to R305, R309 to R306, R316 to R307, R320 to R308, R311 to R309, R306 to R310, R310 to R311, R304 to R312, R317 to R313, R321 to R314, R318 to R315, R322 to R316, R303 to R317, R305 to R318, R301 to R319, R312 to R320, R302 to R321, R314 to R322, R404 to R401, R406 to R402, R413 to R403, R407 to R404, R414 to R405, R402 to R406, R415 to R407, R401 to R409, R403 to R410, R409 to R411, R416 to R412, R405 to R413, R410 to R414, R411 to R415, R412 to R416, R503 to R501, R509 to R502, R504 to R503, R510 to R504, R501 to R505, R511 to R506, R502 to R507, R512 to R508, R505 to R509, R506 to R510, R507 to R511, R508 to R512, R609 to R601, R612 to R602, R601 to R603, R610 to R605, R613 to R606, R616 to R607, R617 to R608, R619 to R609, R602 to R610, R620 to R612, R618 to R613, R608 to R616, R603 to R617, R605 to R618, R606 to R619, R607 to R620, R704 to R701, R707 to R702, R701 to R703, R703 to R704, R708 to R706, R709 to R707, R710 to R708, R711 to R709, R702 to R710, R706 to R711, R805 to R801, R806 to R802, R807 to R803, R809 to R804, R808 to R805, SW202 to SW201, SW201 to SW202, U302 to U301, U301 to U302, U304 to U303, U303 to U304, U404 to U401, U401 to U402, U405 to U403, U403 to U404, U402 to U405, U604 to U601, U601 to U602, U605 to U603, U603 to U604, U602 to U605, U702 to U701, U701 to U702
Connections:
- C202 pad 1: /Processor/XTAL2 -> /Processor/XTAL1
- C203 pad 1: /Processor/XTAL1 -> /Processor/XTAL2
- J201 pad A4: VBUS -> unconnected-(J201-VBUS-PadA4)
- J201 pad A9: VBUS -> unconnected-(J201-VBUS-PadA4)_3
- J201 pad B4: VBUS -> unconnected-(J201-VBUS-PadA4)_1
- J201 pad B9: VBUS -> unconnected-(J201-VBUS-PadA4)_2
- J201 pad S1: GND -> Net-(J201-SHIELD)
- JP203 pad 1: /Processor/BOOT0 -> Net-(J201-SHIELD)
- JP203 pad 2: Net-(JP203-B) -> GND
- U201 pad 5: VBUS -> unconnected-(U201-VBUS-Pad5)
- U202 pad 16: unconnected-(U202-PA2-Pad16) -> /Processor/SW1
- U202 pad 22: /Processor/DAC_0 -> unconnected-(U202-PA6-Pad22)
- U202 pad 23: /Processor/DAC_1 -> unconnected-(U202-PA7-Pad23)
- U202 pad 37: unconnected-(U202-PC6-Pad37) -> /Auto-Balancing Bridge/DC_INT_ISO
- U202 pad 38: unconnected-(U202-PC7-Pad38) -> /Processor/DAC_0
- U202 pad 39: unconnected-(U202-PC8-Pad39) -> /Processor/DAC_7
- U202 pad 40: unconnected-(U202-PC9-Pad40) -> /Processor/DAC_6
- U202 pad 41: /Processor/DAC_2 -> /Processor/DAC_5
- U202 pad 42: /Processor/DAC_3 -> /Processor/DAC_4
- U202 pad 43: /Processor/DAC_4 -> /Processor/DAC_3
- U202 pad 44: /Processor/DAC_5 -> /Processor/DAC_2
- U202 pad 45: /Processor/DAC_6 -> /Processor/DAC_1
- U202 pad 46: /Processor/DAC_7 -> /Processor/SWDIO
- U202 pad 49: /Auto-Balancing Bridge/DC_INT_ISO -> /Processor/SWCLK
- U202 pad 60: Net-(JP203-B) -> /Processor/BOOT0
- Y201 pad 1: /Processor/XTAL2 -> /Processor/XTAL1
- Y201 pad 2: /Processor/XTAL1 -> /Processor/XTAL2
Routing:
- net VIN+: track 0.00 -> 94.7 mm
- net +3.3V: track 0.00 -> 62.1 mm
- net VIN-: track 0.00 -> 46.0 mm, vias 0 -> 10
- net +18V: track 339.8 -> 378.7 mm
- net Net-(J201-SHIELD): track 0.00 -> 36.1 mm
- net -18V: track 324.9 -> 360.5 mm
- net /Processor/BOOT0: track 0.00 -> 23.6 mm
- net GND: track 1.46 -> 24.4 mm
- net +12V: track 239.1 -> 255.0 mm
- net /Processor/XTAL2: track 0.00 -> 13.8 mm
- net /Processor/XTAL1: track 0.00 -> 12.6 mm
- net Net-(U801-ADJ): track 0.00 -> 12.4 mm
- net Net-(U802-ADJ): track 0.00 -> 12.3 mm
- net Net-(U803-ADJ): track 0.00 -> 12.3 mm
- net Net-(U804-ADJ): track 0.00 -> 12.2 mm
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Other:
- board text added: "USB"
- board text added: "pretty please can you move me (DAC_0) to the top of this bus when you rearrange the pins thankkyou"

Commit message: sufferage
Parts:
- moved R204 37.8 mm to (188.9, 62.3), turned to 0 degrees
- moved R205 36.7 mm to (188.9, 64.4), turned to 0 degrees
- moved R206 36.1 mm to (188.9, 66.5), turned to 0 degrees
- moved SW202 27.5 mm to (154.3, 69.0), turned to 0 degrees
- moved R208 20.9 mm to (159.9, 66.3), turned to 180 degrees
- moved R203 17.8 mm to (176.5, 37.5), turned to 180 degrees
- moved RN301 13.2 mm to (177.5, 64.1)
- moved R202 9.88 mm to (184.3, 37.5)
- moved C308 8.38 mm to (179.3, 89.1), turned to 180 degrees
- moved U302 8.15 mm to (177.5, 95.4)
- moved C312 7.99 mm to (175.7, 89.1), turned to 180 degrees
- moved Q301 5.74 mm to (180.9, 134.2)
- moved Q302 2.67 mm to (168.7, 134.2)
- moved C302 2.54 mm to (169.8, 113.6)
- moved R303 2.41 mm to (187.3, 107.8)
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Routing:
- net +3.3V: track 62.1 -> 165.6 mm
- net Net-(RN301-R1.2): track 0.00 -> 39.1 mm, vias 0 -> 2
- net Net-(D301-A): track 54.3 -> 15.3 mm, vias 2 -> 0
- net +3.3VA: track 11.7 -> 43.0 mm, vias 0 -> 8
- net /Processor/~{RST}: track 0.00 -> 30.3 mm, vias 0 -> 2
- net /Processor/SWCLK: track 0.00 -> 29.3 mm, vias 0 -> 2
- net Net-(Q301-E): track 0.00 -> 27.7 mm
- net /Processor/SWDIO: track 6.78 -> 29.3 mm, vias 0 -> 2
- net -18V: track 360.5 -> 347.4 mm
- net /Processor/VAmp.Out: track 25.6 -> 35.0 mm
- net +1.65VA: track 65.7 -> 59.3 mm
- net +18V: track 378.7 -> 372.7 mm
- net Net-(U304B-+): track 6.53 -> 11.1 mm
- net Net-(U303B--): track 38.3 -> 41.4 mm
- net Net-(R321-Pad2): track 25.1 -> 22.0 mm
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
Commit message: sufferage 2
Parts:
- removed C303: 1u, Capacitor_SMD:C_0805_2012Metric
- moved C608 12.9 mm to (133.8, 95.3)
- moved C613 3.20 mm to (130.2, 95.3)
- moved R410 1.91 mm to (91.3, 103.0)
- moved JP602 0.25 mm to (137.9, 95.2)
Connections:
- D301 pad 3: Net-(C303-Pad2) -> Net-(D301-K-Pad3)
- U202 pad 10: unconnected-(U202-PC2-Pad10) -> /Processor/VAmp.AC_EN
- U202 pad 11: unconnected-(U202-PC3-Pad11) -> /Processor/VAmp.AC_100
- U202 pad 14: unconnected-(U202-PA0-Pad14) -> /Processor/VAmp.~{x100}
- U202 pad 15: unconnected-(U202-PA1-Pad15) -> /Processor/SIG_SOURCE
- U202 pad 2: unconnected-(U202-PC13-Pad2) -> /Processor/VAmp./4
- U202 pad 24: unconnected-(U202-PC4-Pad24) -> /Processor/VAmp.AC_1k
- U202 pad 25: unconnected-(U202-PC5-Pad25) -> /Processor/VAmp.AC_10k
- U202 pad 3: unconnected-(U202-PC14-Pad3) -> /Processor/VAmp.x1
- U202 pad 38: /Processor/DAC_0 -> /Processor/DAC_7
- U202 pad 39: /Processor/DAC_7 -> /Processor/DAC_6
- U202 pad 4: unconnected-(U202-PC15-Pad4) -> /Processor/VAmp.x3
- U202 pad 40: /Processor/DAC_6 -> /Processor/DAC_5
- U202 pad 41: /Processor/DAC_5 -> /Processor/DAC_4
- U202 pad 42: /Processor/DAC_4 -> /Processor/DAC_3
- U202 pad 43: /Processor/DAC_3 -> /Processor/DAC_2
- U202 pad 44: /Processor/DAC_2 -> /Processor/DAC_1
- U202 pad 45: /Processor/DAC_1 -> /Processor/DAC_0
- U303 pad 7: Net-(C303-Pad1) -> Net-(D301-K-Pad3)
Routing:
- net +18V: track 372.7 -> 473.6 mm, vias 15 -> 20
- net -18V: track 347.4 -> 447.3 mm, vias 14 -> 22
- net +3.3VA: track 43.0 -> 121.1 mm, vias 8 -> 14
- net /Processor/SIG_SOURCE: track 81.0 -> 149.8 mm, vias 0 -> 2
- net +1.65VA: track 59.3 -> 122.5 mm, vias 4 -> 10
- net /Processor/Source.Bias: track 0.00 -> 57.3 mm, vias 0 -> 2
- net /Processor/Source.Signal: track 0.00 -> 53.7 mm, vias 0 -> 2
- net /Processor/SWCLK: track 29.3 -> 67.3 mm, vias 2 -> 4
- net /Processor/SWDIO: track 29.3 -> 65.9 mm, vias 2 -> 4
- net /Processor/~{RST}: track 30.3 -> 65.5 mm, vias 2 -> 4
- net /Processor/DAC_0: track 0.00 -> 34.5 mm
- net /Processor/DAC_7: track 3.26 -> 34.7 mm
- net /Processor/DAC_6: track 3.73 -> 34.7 mm
- net /Processor/DAC_5: track 4.24 -> 34.6 mm
- net /Processor/DAC_4: track 4.75 -> 34.6 mm
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Other:
- board text removed: "pretty please can you move me (DAC_0) to the top of this bus when you rearrange the pins thankkyou"

Commit message: sleepdrunk
Parts:
- removed C608, C609, C613, C614, C708, C711: 100n, Capacitor_SMD:C_0805_2012Metric
- removed R208: 10k, Resistor_SMD:R_0805_2012Metric
- removed SW202: SW_Push, Button_Switch_THT:SW_PUSH_6mm
- moved JP302 21.2 mm to (166.4, 85.6), turned to -90 degrees
- moved JP303 19.4 mm to (185.4, 87.9), turned to -90 degrees
- moved R204 6.24 mm to (189.0, 68.6)
- moved C404 5.86 mm to (73.4, 85.9), turned to 180 degrees
- moved JP304 4.66 mm to (170.2, 87.9), turned to 90 degrees
- moved C402 3.10 mm to (73.4, 76.5)
- moved C205 1.74 mm to (141.5, 54.7), turned to 180 degrees
- moved R412 1.55 mm to (73.4, 87.9), turned to 180 degrees
- moved C202 0.38 mm to (126.9, 68.0)
- moved C203 0.38 mm to (126.9, 71.5)
- moved Y201 0.38 mm to (123.7, 69.6)
- moved R322 0.35 mm to (170.2, 81.8)
- moved R205 0.13 mm to (189.0, 64.5)
- moved R206 0.11 mm to (189.0, 66.5)
Connections:
- J202 pad 1: GND -> +3.3V
- J202 pad 2: /Processor/~{RST} -> /Processor/SWCLK
- J202 pad 3: /Processor/SWCLK -> GND
- J202 pad 5: +3.3V -> /Processor/~{RST}
- U202 pad 10: /Processor/VAmp.AC_EN -> /Processor/VAmp.AC_1k
- U202 pad 14: /Processor/VAmp.~{x100} -> /Processor/VAmp.AC_10k
- U202 pad 15: /Processor/SIG_SOURCE -> /Processor/VAmp.AC_EN
- U202 pad 16: /Processor/SW1 -> unconnected-(U202-PA2-Pad16)
- U202 pad 2: /Processor/VAmp./4 -> /Current Amplifier/x1
- U202 pad 22: unconnected-(U202-PA6-Pad22) -> /Processor/VAmp.x1
- U202 pad 23: unconnected-(U202-PA7-Pad23) -> /Processor/VAmp./4
- U202 pad 24: /Processor/VAmp.AC_1k -> /Processor/VAmp.x3
- U202 pad 25: /Processor/VAmp.AC_10k -> /Processor/VAmp.~{x100}
- U202 pad 26: unconnected-(U202-PB0-Pad26) -> /Processor/Source./10
- U202 pad 27: unconnected-(U202-PB1-Pad27) -> /Processor/Source.~{x4}
- U202 pad 28: unconnected-(U202-PB2-Pad28) -> /Processor/SIG_SOURCE
- U202 pad 3: /Processor/VAmp.x1 -> /Current Amplifier/x3
- U202 pad 37: /Auto-Balancing Bridge/DC_INT_ISO -> unconnected-(U202-PC6-Pad37)
- U202 pad 4: /Processor/VAmp.x3 -> /Current Amplifier//4
- U202 pad 50: /Auto-Balancing Bridge/R_SEL_100k -> /Auto-Balancing Bridge/R_SEL_10k
- U202 pad 51: /Auto-Balancing Bridge/R_SEL_10k -> /Auto-Balancing Bridge/R_SEL_1k
- U202 pad 52: /Auto-Balancing Bridge/R_SEL_1k -> /Auto-Balancing Bridge/R_SEL_100
- U202 pad 53: /Auto-Balancing Bridge/R_SEL_100 -> /Auto-Balancing Bridge/R_SEL_10
- U202 pad 54: /Auto-Balancing Bridge/R_SEL_10 -> /Auto-Balancing Bridge/DC_INT_ISO
- U202 pad 55: /Auto-Balancing Bridge/AC_EN -> /Auto-Balancing Bridge/R_SEL_100k
- U202 pad 56: /Auto-Balancing Bridge/AC_10k -> /Auto-Balancing Bridge/AC_EN
- U202 pad 57: /Auto-Balancing Bridge/AC_100 -> /Auto-Balancing Bridge/AC_10k
- U202 pad 58: /Auto-Balancing Bridge/AC_1k -> /Auto-Balancing Bridge/AC_100
- U202 pad 59: /Current Amplifier/x3 -> /Auto-Balancing Bridge/AC_1k
- U202 pad 61: /Current Amplifier/x1 -> unconnected-(U202-PB8-Pad61)
- U202 pad 62: /Current Amplifier/~{x100} -> unconnected-(U202-PB9-Pad62)
- U202 pad 8: /Current Amplifier//4 -> /Current Amplifier/~{x100}
- U302 pad 2: Net-(R321-Pad2) -> +1.65VA
- U302 pad 3: +1.65VA -> Net-(R321-Pad2)
- U405 pad 1: /Auto-Balancing Bridge/R_SEL_10 -> /Auto-Balancing Bridge/R_SEL_100k
- U405 pad 11: /Auto-Balancing Bridge/DC_ISO -> /Auto-Balancing Bridge/SEL_10
- U405 pad 12: /Auto-Balancing Bridge/SEL_100k -> /Auto-Balancing Bridge/SEL_100
- U405 pad 13: /Auto-Balancing Bridge/SEL_10 -> /Auto-Balancing Bridge/SEL_1k
- U405 pad 14: /Auto-Balancing Bridge/SEL_100 -> /Auto-Balancing Bridge/SEL_10k
- U405 pad 15: /Auto-Balancing Bridge/SEL_1k -> /Auto-Balancing Bridge/DC_ISO
- U405 pad 16: /Auto-Balancing Bridge/SEL_10k -> /Auto-Balancing Bridge/SEL_100k
- U405 pad 2: /Auto-Balancing Bridge/R_SEL_100 -> /Auto-Balancing Bridge/DC_INT_ISO
- U405 pad 3: /Auto-Balancing Bridge/R_SEL_1k -> /Auto-Balancing Bridge/R_SEL_10
- U405 pad 4: /Auto-Balancing Bridge/R_SEL_10k -> /Auto-Balancing Bridge/R_SEL_100
- U405 pad 5: /Auto-Balancing Bridge/R_SEL_100k -> /Auto-Balancing Bridge/R_SEL_1k
- U405 pad 6: /Auto-Balancing Bridge/DC_INT_ISO -> /Auto-Balancing Bridge/R_SEL_10k
Routing:
- net +1.65VA: track 122.5 -> 245.2 mm, vias 10 -> 17
- net +3.3VA: track 121.1 -> 182.1 mm, vias 14 -> 12
- net /Processor/Source./10: track 0.00 -> 56.6 mm, vias 0 -> 2
- net +18V: track 473.6 -> 528.6 mm
- net /Processor/Source.~{x4}: track 0.00 -> 50.7 mm
- net /Processor/VAmp.AC_100: track 6.74 -> 55.2 mm, vias 2 -> 6
- net -18V: track 447.3 -> 494.3 mm
- net /Processor/VAmp.AC_EN: track 0.00 -> 45.1 mm, vias 0 -> 6
- net /Processor/VAmp.AC_1k: track 12.3 -> 51.7 mm, vias 2 -> 4
- net /Processor/VAmp.x1: track 12.8 -> 51.5 mm, vias 2 -> 4
- net /Processor/VAmp./4: track 14.6 -> 48.5 mm, vias 2 -> 4
- net /Processor/VAmp.x3: track 11.3 -> 44.5 mm, vias 2 -> 4
- net /Processor/VAmp.~{x100}: track 8.34 -> 41.3 mm, vias 2 -> 4
- net /Processor/SW1: track 28.7 -> 0.00 mm, vias 2 -> 0
- net /Processor/VAmp.AC_10k: track 13.7 -> 41.2 mm, vias 2 -> 4
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
Commit message: Final Schematic
Parts:
- removed C406, C410: 100n, Capacitor_SMD:C_0805_2012Metric
- added D1: BAV99, Package_TO_SOT_SMD:SOT-23, F.Cu at (181.4, 163.6)
- moved C22 16.1 mm to (91.4, 112.8)
- moved C23 9.29 mm to (91.4, 105.2)
- moved C27 1.30 mm to (73.7, 77.7), turned to 180 degrees
- moved C28 0.57 mm to (73.7, 85.3)
- moved R45 0.36 mm to (73.7, 87.6), turned to 0 degrees
- moved R32 0.18 mm to (91.4, 103.1)
- renumbered C202 to C1, C302 to C10, C308 to C11, C312 to C12, C309 to C13, C313 to C14, C310 to C15, C314 to C16, C307 to C17, C311 to C18, C301 to C19, C203 to C2, C305 to C20, C306 to C21, C401 to C22, C403 to C23, C405 to C24, C407 to C25, C411 to C26, C402 to C27, C404 to C28, C408 to C29, C204 to C3, C412 to C30, C409 to C31, C413 to C32, C501 to C33, C502 to C34, C503 to C35, C504 to C36, C505 to C37, C506 to C38, C616 to C39, C205 to C4, C601 to C40, C603 to C41, C605 to C42, C606 to C43, C611 to C44, C607 to C45, C612 to C46, C604 to C47, C602 to C48, C610 to C49, C206 to C5, C615 to C50, C706 to C51, C709 to C52, C701 to C53, C703 to C54, C705 to C55, C707 to C56, C710 to C57, C704 to C58, C702 to C59, C207 to C6, C805 to C60, C807 to C61, C806 to C62, C808 to C63, C801 to C64, C803 to C65, C809 to C66, C811 to C67, C802 to C68, C804 to C69, C201 to C7, C810 to C70, C812 to C71, C208 to C8, C304 to C9, D301 to D2, D401 to D3, D403 to D4, D402 to D5, D802 to D6, D803 to D7, D801 to D8, D804 to D9, FB801 to FB1, FL201 to FL1, H101 to H1, H102 to H2, H103 to H3, H104 to H4, J102 to J1, J103 to J2, J104 to J3, J105 to J4, J101 to J5, J201 to J6, J202 to J7, J802 to J8, J801 to J9, JP203 to JP1, JP604 to JP10, JP601 to JP11, JP602 to JP12, JP701 to JP13, JP702 to JP14, JP201 to JP2, JP202 to JP3, JP303 to JP4, JP304 to JP5, JP302 to JP6, JP301 to JP7, JP401 to JP8, JP603 to JP9, K301 to K1, K401 to K2, K505 to K3, K504 to K4, K503 to K5, K502 to K6, K501 to K7, Q303 to Q1, Q301 to Q2, Q302 to Q3, Q401 to Q4, Q403 to Q5, Q402 to Q6, Q404 to Q7, R201 to R1, R317 to R10, R312 to R11, R318 to R12, R310 to R13, R301 to R14, R303 to R15, R306 to R16, R311 to R17, R309 to R18, R320 to R19, R202 to R2, R302 to R20, R322 to R21, R304 to R22, R307 to R23, R313 to R24, R315 to R25, R305 to R26, R308 to R27, R314 to R28, R316 to R29, R203 to R3, R409 to R30, R406 to R31, R410 to R32, R401 to R33, R413 to R34, R402 to R35, R404 to R36, R408 to R37, R411 to R38, R414 to R39, R204 to R4, R415 to R40, R416 to R41, R403 to R42, R405 to R43, R407 to R44, R412 to R45, R505 to R46, R507 to R47, R501 to R48, R503 to R49, R205 to R5, R509 to R50, R510 to R51, R511 to R52, R512 to R53, R502 to R54, R504 to R55, R506 to R56, R508 to R57, R603 to R58, R610 to R59, R206 to R6, R617 to R60, R604 to R61, R618 to R62, R619 to R63, R620 to R64, R616 to R65, R601 to R66, R605 to R67, R611 to R68, R602 to R69, R207 to R7, R606 to R70, R614 to R71, R615 to R72, R607 to R73, R608 to R74, R613 to R75, R609 to R76, R612 to R77, R703 to R78, R710 to R79, R319 to R8, R704 to R80, R701 to R81, R705 to R82, R711 to R83, R702 to R84, R706 to R85, R707 to R86, R708 to R87, R709 to R88, R712 to R89, R321 to R9, R801 to R90, R802 to R91, R803 to R92, R805 to R93, R804 to R94, RN301 to RN1, RV801 to RV1, RV802 to RV2, RV803 to RV3, RV804 to RV4, SW201 to SW1, U201 to U1, U401 to U10, U403 to U11, U602 to U12, U605 to U13, U604 to U14, U601 to U15, U603 to U16, U702 to U17, U701 to U18, U703 to U19, U202 to U2, U801 to U20, U802 to U21, U803 to U22, U804 to U23, U302 to U3, U301 to U4, U303 to U5, U304 to U6, U402 to U7, U405 to U8, U404 to U9, Y201 to Y1
Routing:
- net /Auto-Balancing Bridge/DC_ISO: track 205.6 -> 36.4 mm
- net /Auto-Balancing Bridge/SEL_100k: track 189.4 -> 23.0 mm
- net /Auto-Balancing Bridge/SEL_1k: track 104.5 -> 237.5 mm
- net /Auto-Balancing Bridge/SEL_10k: track 90.2 -> 212.2 mm
- net Net-(Q4-E): track 30.7 -> 145.6 mm, vias 0 -> 4
- net Net-(D3-K-Pad3): track 0.00 -> 97.2 mm, vias 0 -> 4
- net +3.3VA: track 182.1 -> 213.5 mm, vias 12 -> 14
- net /Auto-Balancing Bridge/OUT+: track 230.5 -> 252.4 mm, vias 5 -> 8
- net -18V: track 494.3 -> 516.1 mm
- net Net-(D3-A): track 0.36 -> 19.3 mm
- net Net-(D5-A): track 0.00 -> 18.7 mm
- net /Auto-Balancing Bridge/SEL_100: track 146.3 -> 137.4 mm
- net +18V: track 528.6 -> 535.4 mm
- net Net-(U6B-+): track 5.95 -> 12.7 mm, vias 0 -> 2
- net Net-(Q6-B): track 0.04 -> 6.44 mm
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
Commit message: cryingggggg
Parts:
- JP11, JP12: footprint Jumper:SolderJumper-3_P1.3mm_Bridged123_RoundedPad1.0x1.5mm -> Jumper:SolderJumper-3_P1.3mm_Bridged12_RoundedPad1.0x1.5mm_NumberLabels
- moved D1 12.4 mm to (183.9, 151.4), turned to 180 degrees
- turned C6 to 180 degrees
Connections:
- U2 pad 50: /Auto-Balancing Bridge/R_SEL_10k -> /Auto-Balancing Bridge/R_SEL_10
- U2 pad 51: /Auto-Balancing Bridge/R_SEL_1k -> /Auto-Balancing Bridge/R_SEL_100
- U2 pad 52: /Auto-Balancing Bridge/R_SEL_100 -> /Auto-Balancing Bridge/DC_INT_ISO
- U2 pad 53: /Auto-Balancing Bridge/R_SEL_10 -> /Auto-Balancing Bridge/R_SEL_100k
- U2 pad 54: /Auto-Balancing Bridge/DC_INT_ISO -> /Auto-Balancing Bridge/R_SEL_1k
- U2 pad 55: /Auto-Balancing Bridge/R_SEL_100k -> /Auto-Balancing Bridge/R_SEL_10k
- U8 pad 1: /Auto-Balancing Bridge/R_SEL_100k -> /Auto-Balancing Bridge/R_SEL_10k
- U8 pad 13: /Auto-Balancing Bridge/SEL_1k -> /Auto-Balancing Bridge/DC_ISO
- U8 pad 14: /Auto-Balancing Bridge/SEL_10k -> /Auto-Balancing Bridge/SEL_100k
- U8 pad 15: /Auto-Balancing Bridge/DC_ISO -> /Auto-Balancing Bridge/SEL_1k
- U8 pad 16: /Auto-Balancing Bridge/SEL_100k -> /Auto-Balancing Bridge/SEL_10k
- U8 pad 2: /Auto-Balancing Bridge/DC_INT_ISO -> /Auto-Balancing Bridge/R_SEL_1k
- U8 pad 3: /Auto-Balancing Bridge/R_SEL_10 -> /Auto-Balancing Bridge/R_SEL_100k
- U8 pad 4: /Auto-Balancing Bridge/R_SEL_100 -> /Auto-Balancing Bridge/DC_INT_ISO
- U8 pad 5: /Auto-Balancing Bridge/R_SEL_1k -> /Auto-Balancing Bridge/R_SEL_100
- U8 pad 6: /Auto-Balancing Bridge/R_SEL_10k -> /Auto-Balancing Bridge/R_SEL_10
Routing:
- net /Auto-Balancing Bridge/DC_ISO: track 36.4 -> 194.6 mm
- net /Auto-Balancing Bridge/SEL_100k: track 23.0 -> 178.2 mm
- net +12V: track 255.0 -> 395.6 mm, vias 10 -> 11
- net /Auto-Balancing Bridge/SEL_1k: track 237.5 -> 104.5 mm
- net /Auto-Balancing Bridge/SEL_10k: track 212.2 -> 90.2 mm
- net GND: track 25.6 -> 71.9 mm, vias 2 -> 113
- net /Auto-Balancing Bridge/SEL_100: track 137.4 -> 149.8 mm
- net Net-(JP2-A): track 2.02 -> 10.1 mm
- net VIN-: track 46.0 -> 53.8 mm, vias 10 -> 12
- net +18V: track 535.4 -> 541.7 mm
- net /Signal Source/RELAY_DRIVE: track 4.16 -> 8.55 mm, vias 0 -> 2
- net /Auto-Balancing Bridge/R_SEL_10k: track 85.3 -> 81.3 mm
- net VIN+: track 94.7 -> 97.3 mm
- net /Auto-Balancing Bridge/R_SEL_10: track 83.1 -> 85.3 mm
- net /Auto-Balancing Bridge/R_SEL_1k: track 84.5 -> 82.3 mm
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- added copper zone on F.Cu, net GND
