File: PCB/Main Board/Source.kicad_sch (KiCad schematic)
At the start: 47 parts, among them K301 AGQ200A12, Q301 TIP41C, Q302 TIP42C, U301 DG201, U302 OPA2197xD, U303 OPA2376xxD, U304 OPA2197xD

Commit message: merge 2.0
Parts:
- gave numbers to parts that had none: 4
- renumbered R316 to R317
Changed lines of the file:
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@@
 		(on_board yes)
 		(dnp no)
-		(property "Reference" "R?"
+		(property "Reference" "R319"
 			(at 240.03 57.15 90)
 			(effects
@@
 			(project "Main Board"
 				(path "/20aae4b7-3fb8-4924-82e8-1e7a29a313f8/018dbbaa-4414-4e5b-943a-751bd604c3b0"
-					(reference "R?")
+					(reference "R319")
 					(unit 1)
 				)
@@
 		(on_board yes)
 		(dnp no)
-		(property "Reference" "R316"
+		(property "Reference" "R317"
 			(at 237.49 80.01 90)
 			(effects
@@
 			(project "Main Board"
 				(path "/20aae4b7-3fb8-4924-82e8-1e7a29a313f8/018dbbaa-4414-4e5b-943a-751bd604c3b0"
-					(reference "R316")
+					(reference "R317")
 					(unit 1)
 				)
@@
 		(on_board yes)
 		(dnp no)
-		(property "Reference" "R?"
+		(property "Reference" "R316"
 			(at 232.41 57.15 90)
 			(effects
@@
 			(project "Main Board"
 				(path "/20aae4b7-3fb8-4924-82e8-1e7a29a313f8/018dbbaa-4414-4e5b-943a-751bd604c3b0"
-					(reference "R?")
+					(reference "R316")
 					(unit 1)
 				)
@@
 		(dnp no)
 		(fields_autoplaced yes)
-		(property "Reference" "RN?"
+		(property "Reference" "RN301"
 			(at 198.12 121.92 90)
 			(effects
@@
 			(project ""
 				(path "/20aae4b7-3fb8-4924-82e8-1e7a29a313f8/018dbbaa-4414-4e5b-943a-751bd604c3b0"
-					(reference "RN?")
+					(reference "RN301")
 					(unit 1)
 				)
@@
 		(dnp no)
 		(fields_autoplaced yes)
-		(property "Reference" "R?"
+		(property "Reference" "R318"
 			(at 240.03 39.37 90)
 			(effects
@@
 			(project "Main Board"
 				(path "/20aae4b7-3fb8-4924-82e8-1e7a29a313f8/018dbbaa-4414-4e5b-943a-751bd604c3b0"
-					(reference "R?")
+					(reference "R318")
 					(unit 1)
 				)

Commit message: sig source finished
Parts:
- removed C311, C313: 10µ, Capacitor_SMD:C_0805_2012Metric, symbol Device:C
- removed C312, C314: 100n, Capacitor_SMD:C_0805_2012Metric, symbol Device:C
- removed R312: 2k, Resistor_SMD:R_0805_2012Metric, symbol Device:R
- removed R317: 100, Resistor_SMD:R_0805_2012Metric, symbol Device:R
- added C301, C305: 10µ, Capacitor_SMD:C_0805_2012Metric, symbol Device:C
- added C303: 1u, Capacitor_SMD:C_0805_2012Metric, symbol Device:C
- added Q303: 2N7002, Package_TO_SOT_SMD:SOT-23, symbol Transistor_FET:2N7002
- added R309, R320: 2k, Resistor_SMD:R_0805_2012Metric, symbol Device:R
- added R314, R315, R316: 100, Resistor_SMD:R_0805_2012Metric, symbol Device:R
- R313: value 2k -> 100
- renumbered C301 to C304, C315 to C306, C303 to C307, C305 to C308, C307 to C309, C309 to C310, C304 to C311, C306 to C312, C308 to C313, C310 to C314, JP304 to JP301, JP303 to JP302, JP301 to JP303, JP302 to JP304, R307 to R301, R311 to R302, R308 to R303, R315 to R304, R318 to R305, R309 to R306, R316 to R307, R319 to R308, R306 to R310, R310 to R311, R304 to R312, R303 to R317, R305 to R318, R301 to R319, R302 to R321, R314 to R322, U302 to U301, U301 to U302, U304 to U303, U303 to U304
Connections:
- net +18V: now also C301.2, R309.1
- net -18V: now also C305.2, R320.2; no longer R313.2
- net GND: now also C301.1, C305.1, Q303.2 (S)
- net SIG_SOURCE: now also Q303.1 (G); no longer K301.8
- net at D301.2 (A), Q302.1 (B): now also R320.1; no longer R313.1
- net at Q301.3 (E), Q302.3 (E), R302.2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: now also R313.1, R315.1
- net at JP301.2 (B), K301.4: now also R314.2, R316.2
- net at D301.1 (K), Q301.1 (B): now also R309.2
- net at U303.7: now also C303.1; no longer D301.3 (K)
- new net: R315.2, R316.1
- new net: R313.2, R314.1
- new net: C303.2, D301.3 (K)
- new net RELAY_DRIVE: K301.8, Q303.3 (D)
Other:
- moved on the sheet: R310, R311, U302B, U302C, U302D, U303B

Commit message: hello
Parts:
- Q302: renamed from Q301; footprint Package_TO_SOT_THT:TO-220-3_Horizontal_TabDown -> Package_TO_SOT_THT:TO-220-3_Horizontal_TabUp
- Q303: renamed from Q302; footprint Package_TO_SOT_THT:TO-220-3_Horizontal_TabDown -> Package_TO_SOT_THT:TO-220-3_Horizontal_TabUp
- renumbered C304 to C301, C307 to C303, C311 to C304, C308 to C305, C312 to C306, C309 to C307, C313 to C308, C310 to C309, C314 to C310, C303 to C311, C301 to C312, C305 to C313, C306 to C314, JP303 to JP301, JP304 to JP302, JP302 to JP303, JP301 to JP304, Q303 to Q301, R319 to R301, R321 to R302, R317 to R303, R312 to R304, R318 to R305, R310 to R306, R301 to R307, R303 to R308, R306 to R309, R311 to R310, R309 to R311, R320 to R312, R302 to R313, R322 to R314, R304 to R315, R307 to R316, R313 to R317, R315 to R318, R305 to R319, R308 to R320, R314 to R321, R316 to R322, U302 to U301, U301 to U302, U304 to U303, U303 to U304

Commit message: please be nice
Parts:
- renumbered C312 to C301, C311 to C303, C301 to C304, C313 to C305, C314 to C306, C303 to C307, C305 to C308, C307 to C309, C309 to C310, C304 to C311, C306 to C312, C308 to C313, C310 to C314, JP304 to JP301, JP303 to JP302, JP301 to JP303, JP302 to JP304, Q302 to Q301, Q303 to Q302, Q301 to Q303, R307 to R301, R313 to R302, R308 to R303, R315 to R304, R319 to R305, R309 to R306, R316 to R307, R320 to R308, R311 to R309, R306 to R310, R310 to R311, R304 to R312, R317 to R313, R321 to R314, R318 to R315, R322 to R316, R303 to R317, R305 to R318, R301 to R319, R312 to R320, R302 to R321, R314 to R322, U302 to U301, U301 to U302, U304 to U303, U303 to U304

Commit message: sufferage 2
Parts:
- removed C303: 1u, Capacitor_SMD:C_0805_2012Metric, symbol Device:C
Connections:
- net at U303.7: now also D301.3 (K)
Changed lines of the file:
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@@
 	(wire
 		(pts
+			(xy 180.34 73.66) (xy 187.96 73.66)
+		)
+		(stroke
+			(width 0)
+			(type default)
+		)
+	)
+	(wire
+		(pts
 			(xy 227.33 45.72) (xy 227.33 48.26)
 		)
@@
 					(unit 1)
 				)
-			)
-		)
-	)
-	(symbol
-		(lib_id "Device:C")
-		(at 184.15 73.66 90)
-		(mirror x)
-		(unit 1)
-		(exclude_from_sim no)
-		(in_bom yes)
-		(on_board yes)
-		(dnp yes)
-		(property "Reference" "C303"
-			(at 184.15 78.74 90)
-			(effects
-				(font
-					(size 1.27 1.27)
-				)
-			)
-		)
-		(property "Value" "1u"
-			(at 184.15 81.28 90)
-			(effects
-				(font
-					(size 1.27 1.27)
-				)
-			)
-		)
-		(property "Footprint" "Capacitor_SMD:C_0805_2012Metric"
-			(at 187.96 74.6252 0)
-			(effects
-				(font
-					(size 1.27 1.27)
-				)
-				(hide yes)
-			)
-		)
-		(property "Datasheet" "~"
-			(at 184.15 73.66 0)
-			(effects
-				(font
-					(size 1.27 1.27)
-				)
-				(hide yes)
-			)
-		)
-		(property "Description" "Unpolarized capacitor"
-			(at 184.15 73.66 0)
-			(effects
-				(font
-					(size 1.27 1.27)
-				)
-				(hide yes)
-			)
-		)
-		(pin "1"
-		)
-		(pin "2"
-		)
-		(instances
-			(project "Main Board"
-				(path "/20aae4b7-3fb8-4924-82e8-1e7a29a313f8/018dbbaa-4414-4e5b-943a-751bd604c3b0"
-					(reference "C303")
-					(unit 1)
-				)

Commit message: sleepdrunk
Connections:
- net +1.65VA: now also U302.2; no longer U302.3
- net at R321.2: now also U302.3; no longer U302.2
Changed lines of the file:
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@@
 		(lib_id "More_symbols:DG201")
 		(at 46.99 113.03 90)
-		(mirror x)
 		(unit 1)
 		(exclude_from_sim no)
@@
 		(dnp no)
 		(property "Reference" "U302"
-			(at 43.18 111.7601 90)
+			(at 43.18 111.7599 90)
 			(effects
 				(font
@@
 		)
 		(property "Value" "DG201"
-			(at 43.18 114.3001 90)
+			(at 43.18 114.2999 90)
 			(effects
 				(font

Commit message: Final Schematic
Parts:
- added D1: BAV99, Package_TO_SOT_SMD:SOT-23, symbol Diode:BAV99
- renumbered C302 to C10, C308 to C11, C312 to C12, C309 to C13, C313 to C14, C310 to C15, C314 to C16, C307 to C17, C311 to C18, C301 to C19, C305 to C20, C306 to C21, C304 to C9, D301 to D2, JP303 to JP4, JP304 to JP5, JP302 to JP6, JP301 to JP7, K301 to K1, Q303 to Q1, Q301 to Q2, Q302 to Q3, R317 to R10, R312 to R11, R318 to R12, R310 to R13, R301 to R14, R303 to R15, R306 to R16, R311 to R17, R309 to R18, R320 to R19, R302 to R20, R322 to R21, R304 to R22, R307 to R23, R313 to R24, R315 to R25, R305 to R26, R308 to R27, R314 to R28, R316 to R29, R319 to R8, R321 to R9, RN301 to RN1, U302 to U3, U301 to U4, U303 to U5, U304 to U6
Connections:
- net +12V: now also D1.2 (A)
- net RELAY_DRIVE: now also D1.3 (K)
- no-connect marks 13 -> 14
Other:
- note added: "Additional DAC Optional"
- note added: "Bias range: ±4V RMS ±5.7V Pk Gain: ~3.7"
- note removed: "AC signal x1 /10"
- note removed: "Bias range: ±4V RMS ±5.7V Pk Gain: ~3.7 2nd order chebyshev"
- title: (none) -> Signal Source
- moved on the sheet: C11, C12, C13, C14, C15, C16, C17, C18, C21, JP4, JP5, JP6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

Commit message: minor cleanup from the party
Parts:
- renumbered C19 to C301, C10 to C302, C9 to C303, C20 to C304, C17 to C305, C18 to C306, C21 to C307, C11 to C308, C13 to C309, C15 to C310, C12 to C311, C14 to C312, C16 to C313, D2 to D301, D1 to D302, JP7 to JP301, JP4 to JP302, JP6 to JP303, JP5 to JP304, K1 to K301, Q2 to Q301, Q3 to Q302, Q1 to Q303, R14 to R301, R20 to R302, R15 to R303, R22 to R304, R26 to R305, R16 to R306, R23 to R307, R27 to R308, R18 to R309, R13 to R310, R17 to R311, R11 to R312, R24 to R313, R28 to R314, R25 to R315, R29 to R316, R10 to R317, R12 to R318, R8 to R319, R19 to R320, R9 to R321, R21 to R322, RN1 to RN301, U4 to U301, U3 to U302, U5 to U303, U6 to U304
