File: PCB/Main Board/Source.kicad_sch (KiCad schematic)
At the start: 50 parts, among them K301 AGQ200A12, Q301 TIP41C, Q302 TIP42C, Q303 2N7002, U301 OPA2197xD, U302 DG201, U303 OPA2197xD, U304 OPA2376xxD

Commit message: footprints and tps
Parts:
- added TP?: TEST_SIGNAL, TestPoint:TestPoint_Pad_2.0x2.0mm, symbol Connector:TestPoint
- added TP?: TEST_SIGNAL_DC, TestPoint:TestPoint_Pad_2.0x2.0mm, symbol Connector:TestPoint
- added TP?: AUX_DAC_OUT, TestPoint:TestPoint_Pad_2.0x2.0mm, symbol Connector:TestPoint
- added TP?: TEST_SIGNAL_AC, TestPoint:TestPoint_Pad_2.0x2.0mm, symbol Connector:TestPoint
Connections:
- net AUX_DAC_OUT: now also TP?.1
- net at R303.1, U301.6 (-), U301.7: now also TP?.1
- net at C302.2, R306.1, R310.1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: now also TP?.1
- net at Q301.3 (E), Q302.3 (E), R302.2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: now also TP?.1

Commit message: :(
Parts:
- gave numbers to parts that had none: 4
- renumbered C302 to C10, C308 to C11, C311 to C12, C309 to C13, C312 to C14, C310 to C15, C313 to C16, C305 to C17, C306 to C18, C301 to C19, C304 to C20, C307 to C21, C303 to C9, D302 to D1, D301 to D2, JP302 to JP4, JP304 to JP5, JP303 to JP6, JP301 to JP7, K301 to K1, Q303 to Q1, Q301 to Q2, Q302 to Q3, R317 to R10, R312 to R11, R318 to R12, R310 to R13, R301 to R14, R303 to R15, R306 to R16, R311 to R17, R309 to R18, R320 to R19, R302 to R20, R322 to R21, R304 to R22, R307 to R23, R313 to R24, R315 to R25, R305 to R26, R308 to R27, R314 to R28, R316 to R29, R319 to R8, R321 to R9, RN301 to RN1, U302 to U3, U301 to U4, U303 to U5, U304 to U6

Commit message: bleh
Connections:
- net +1.65VA: now also U3.6; no longer U3.2
- net GND: now also U3.1; no longer U3.8
- net ~{x4}: now also U3.8; no longer U3.1
- net at R9.2: now also U3.7; no longer U3.3
Other:
- moved on the sheet: U3A, U3B
Changed lines of the file:
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@@
 	(symbol
 		(lib_id "More_symbols:DG201")
-		(at 50.8 177.8 0)
+		(at 46.99 113.03 90)
 		(unit 2)
 		(exclude_from_sim no)
@@
 		(on_board yes)
 		(dnp no)
-		(fields_autoplaced yes)
 		(property "Reference" "U3"
-			(at 50.8 170.18 0)
+			(at 43.18 111.76 90)
 			(effects
 				(font
 					(size 1.27 1.27)
 				)
+				(justify left)
 			)
 		)
 		(property "Value" "DG201"
-			(at 50.8 172.72 0)
+			(at 43.18 114.3 90)
 			(effects
 				(font
 					(size 1.27 1.27)
 				)
+				(justify left)
 			)
 		)
 		(property "Footprint" "Package_SO:SOIC-16_3.9x9.9mm_P1.27mm"
-			(at 50.8 180.34 0)
+			(at 49.53 113.03 0)
 			(effects
 				(font
@@
 		)
 		(property "Datasheet" "https://www.vishay.com/docs/70037/dg201b.pdf"
-			(at 50.8 177.8 0)
+			(at 46.99 113.03 0)
 			(effects
 				(font
@@
 		)
 		(property "Description" "Improved Quad CMOS Analog Switches, normally ON, 45Ohm Ron, SOIC-16"
-			(at 50.8 177.8 0)
+			(at 46.99 113.03 0)
 			(effects
 				(font
@@
 	(symbol
 		(lib_id "More_symbols:DG201")
-		(at 46.99 113.03 90)
+		(at 50.8 177.8 0)
 		(unit 1)
 		(exclude_from_sim no)
@@
 		(dnp no)
 		(property "Reference" "U3"
-			(at 43.18 111.7599 90)
+			(at 50.8 170.18 0)
 			(effects
 				(font
 					(size 1.27 1.27)
 				)
-				(justify left)
 			)
 		)
 		(property "Value" "DG201"
-			(at 43.18 114.2999 90)
+			(at 50.8 172.72 0)
 			(effects
 				(font
 					(size 1.27 1.27)
 				)
-				(justify left)
 			)
 		)
 		(property "Footprint" "Package_SO:SOIC-16_3.9x9.9mm_P1.27mm"
-			(at 49.53 113.03 0)
+			(at 50.8 180.34 0)
 			(effects
 				(font
@@
 		)
 		(property "Datasheet" "https://www.vishay.com/docs/70037/dg201b.pdf"
-			(at 46.99 113.03 0)
+			(at 50.8 177.8 0)
 			(effects
 				(font
@@
 		)
 		(property "Description" "Improved Quad CMOS Analog Switches, normally ON, 45Ohm Ron, SOIC-16"
-			(at 46.99 113.03 0)
+			(at 50.8 177.8 0)
 			(effects
 				(font

Commit message: dsfsdff
Parts:
- Q2, Q3: footprint Package_TO_SOT_THT:TO-220-3_Horizontal_TabUp -> Package_TO_SOT_THT:TO-220-3_Vertical
Changed lines of the file:
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@@
 			)
 		)
-		(property "Footprint" "Package_TO_SOT_THT:TO-220-3_Horizontal_TabUp"
+		(property "Footprint" "Package_TO_SOT_THT:TO-220-3_Vertical"
 			(at 214.63 66.675 0)
 			(effects
@@
 			)
 		)
-		(property "Footprint" "Package_TO_SOT_THT:TO-220-3_Horizontal_TabUp"
+		(property "Footprint" "Package_TO_SOT_THT:TO-220-3_Vertical"
 			(at 214.63 80.645 0)
 			(effects

Commit message: :(
Parts:
- removed TP8: AUX_DAC_OUT, TestPoint:TestPoint_Pad_2.0x2.0mm, symbol Connector:TestPoint
Connections:
- net GND: now also U3.16; no longer U3.9
- net /10: now also U3.9; no longer U3.16
- net at U3.14: no longer R17.2
- net at R14.2, R15.2, R16.2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: now also U3.11; no longer U3.15
- net at U3.10: now also R17.2
Other:
- moved on the sheet: U3C, U3D
Changed lines of the file:
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@@
 	(wire
 		(pts
-			(xy 264.16 135.89) (xy 264.16 138.43)
-		)
-		(stroke
-			(width 0)
-			(type default)
-		)
-	)
-	(wire
-		(pts
 			(xy 78.74 35.56) (xy 83.82 35.56)
 		)
@@
 	(symbol
 		(lib_id "More_symbols:DG201")
-		(at 151.13 63.5 0)
-		(mirror y)
+		(at 25.4 177.8 0)
 		(unit 4)
 		(exclude_from_sim no)
@@
 		(dnp no)
 		(property "Reference" "U3"
-			(at 151.13 55.88 0)
+			(at 25.4 170.18 0)
 			(effects
 				(font
@@
 		)
 		(property "Value" "DG201"
-			(at 151.13 58.42 0)
+			(at 25.4 172.72 0)
 			(effects
 				(font
@@
 		)
 		(property "Footprint" "Package_SO:SOIC-16_3.9x9.9mm_P1.27mm"
-			(at 151.13 66.04 0)
+			(at 25.4 180.34 0)
 			(effects
 				(font
@@
 		)
 		(property "Datasheet" "https://www.vishay.com/docs/70037/dg201b.pdf"
-			(at 151.13 63.5 0)
+			(at 25.4 177.8 0)
 			(effects
 				(font
@@
 		)
 		(property "Description" "Improved Quad CMOS Analog Switches, normally ON, 45Ohm Ron, SOIC-16"
-			(at 151.13 63.5 0)
+			(at 25.4 177.8 0)
 			(effects
 				(font
@@
 	)
 	(symbol
-		(lib_id "Connector:TestPoint")
-		(at 264.16 135.89 0)
-		(unit 1)
-		(exclude_from_sim no)
-		(in_bom yes)
-		(on_board yes)
-		(dnp no)
-		(fields_autoplaced yes)
-		(property "Reference" "TP8"
-			(at 266.7 131.3179 0)
-			(effects
-				(font
-					(size 1.27 1.27)
-				)
-				(justify left)
-			)
-		)
-		(property "Value" "AUX_DAC_OUT"
-			(at 266.7 133.8579 0)
-			(effects
-				(font
-					(size 1.27 1.27)
-				)
-				(justify left)
-			)
-		)
-		(property "Footprint" "TestPoint:TestPoint_Pad_2.0x2.0mm"
-			(at 269.24 135.89 0)
-			(effects
-				(font
-					(size 1.27 1.27)
-				)
-				(hide yes)
-			)
-		)
-		(property "Datasheet" "~"
-			(at 269.24 135.89 0)
-			(effects
-				(font
-					(size 1.27 1.27)
-				)
-				(hide yes)
-			)
-		)
-		(property "Description" "test point"
-			(at 264.16 135.89 0)
-			(effects
-				(font
-					(size 1.27 1.27)
-				)
-				(hide yes)
-			)
-		)
-		(pin "1"
-		)
-		(instances
-			(project "Main Board"
-				(path "/20aae4b7-3fb8-4924-82e8-1e7a29a313f8/018dbbaa-4414-4e5b-943a-751bd604c3b0"
-					(reference "TP8")
-					(unit 1)
-				)
-			)
-		)
-	)
-	(symbol
 		(lib_id "Device:C")
 		(at 186.69 54.61 90)
@@
 	(symbol
 		(lib_id "More_symbols:DG201")
-		(at 25.4 177.8 0)
+		(at 151.13 63.5 0)
 		(unit 3)
 		(exclude_from_sim no)
@@
 		(on_board yes)
 		(dnp no)
-		(fields_autoplaced yes)
 		(property "Reference" "U3"
-			(at 25.4 170.18 0)
+			(at 151.13 55.88 0)
 			(effects
 				(font
@@
 		)
 		(property "Value" "DG201"
-			(at 25.4 172.72 0)
+			(at 151.13 58.42 0)
 			(effects
 				(font
@@
 		)
 		(property "Footprint" "Package_SO:SOIC-16_3.9x9.9mm_P1.27mm"
-			(at 25.4 180.34 0)
+			(at 151.13 66.04 0)
 			(effects
 				(font
@@
 		)
 		(property "Datasheet" "https://www.vishay.com/docs/70037/dg201b.pdf"
-			(at 25.4 177.8 0)
+			(at 151.13 63.5 0)
 			(effects
 				(font
@@
 		)
 		(property "Description" "Improved Quad CMOS Analog Switches, normally ON, 45Ohm Ron, SOIC-16"
-			(at 25.4 177.8 0)
+			(at 151.13 63.5 0)
 			(effects
 				(font

Commit message: edits
Parts:
- removed C10: 47p, Capacitor_SMD:C_0805_2012Metric, symbol Device:C
- removed R11: 2.4k, Resistor_SMD:R_0805_2012Metric, symbol Device:R
- removed R12: 1.3k, Resistor_SMD:R_0805_2012Metric, symbol Device:R
Connections:
- net at U5.2 (-): now also C9.1, R10.2

Commit message: BLEH
Parts:
- renumbered C11 to C10, C12 to C11, C13 to C12, C14 to C13, C15 to C14, C16 to C15, C17 to C16, C18 to C17, C19 to C18, C20 to C19, C21 to C20, JP4 to JP1, JP5 to JP2, JP6 to JP3, JP7 to JP4, R13 to R11, R14 to R12, R15 to R13, R16 to R14, R17 to R15, R18 to R16, R19 to R17, R20 to R18, R21 to R19, R22 to R20, R23 to R21, R24 to R22, R25 to R23, R26 to R24, R27 to R25, R28 to R26, R29 to R27, U3 to U2, U4 to U3, U5 to U4, U6 to U5

Commit message: minor
Parts:
- removed unit 1 of U4
- added U?: OPA2197xD, Package_SO:SOIC-8_3.9x4.9mm_P1.27mm, symbol Amplifier_Operational:OPA2197xD
Connections:
- net at R11.1, R14.1, TP6.1: now also U?.1, U?.2 (-)
- net at C9.1, R10.2: now also U?.3 (+)
Other:
- note removed: "Sim"
- moved on the sheet: C10, C11, C12, C13, C14, C15, C16, C17, C18, C19, C20, C9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
