File: PCB/Main Board/Main Board.kicad_sch (KiCad schematic)
At the start: 9 parts, among them J101 Conn_01x01_Pin, J102 Conn_Coaxial, J103 Conn_Coaxial, J104 Conn_Coaxial, J105 Conn_Coaxial

Commit message: Final Schematic
Parts:
- renumbered H101 to H1, H102 to H2, H103 to H3, H104 to H4, J102 to J1, J103 to J2, J104 to J3, J105 to J4, J101 to J5
Other:
- title: (none) -> Interconnect
- moved on the sheet: J1, J2, J3, J4, J5

Commit message: change footprints
Parts:
- J1, J2, J3, J4: footprint Connector_Coaxial:BNC_TEConnectivity_1478035_Horizontal -> Connector_Coaxial:BNC_Amphenol_B6252HB-NPP3G-50_Horizontal
Other:
- note added: "https://www.aliexpress.com/item/1005005482292733.html"
Changed lines of the file:
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@@
+		)
+	)
+	(text "https://www.aliexpress.com/item/1005005482292733.html"
+		(exclude_from_sim no)
+		(at 195.58 66.04 0)
+		(effects
+			(font
+				(size 1.27 1.27)
+			)
 		)
 	)
@@
 			)
 		)
-		(property "Footprint" "Connector_Coaxial:BNC_TEConnectivity_1478035_Horizontal"
+		(property "Footprint" "Connector_Coaxial:BNC_Amphenol_B6252HB-NPP3G-50_Horizontal"
 			(at 165.1 114.3 0)
 			(effects
@@
 			)
 		)
-		(property "Footprint" "Connector_Coaxial:BNC_TEConnectivity_1478035_Horizontal"
+		(property "Footprint" "Connector_Coaxial:BNC_Amphenol_B6252HB-NPP3G-50_Horizontal"
 			(at 165.1 72.39 0)
 			(effects
@@
 			)
 		)
-		(property "Footprint" "Connector_Coaxial:BNC_TEConnectivity_1478035_Horizontal"
+		(property "Footprint" "Connector_Coaxial:BNC_Amphenol_B6252HB-NPP3G-50_Horizontal"
 			(at 165.1 92.71 0)
 			(effects
@@
 			)
 		)
-		(property "Footprint" "Connector_Coaxial:BNC_TEConnectivity_1478035_Horizontal"
+		(property "Footprint" "Connector_Coaxial:BNC_Amphenol_B6252HB-NPP3G-50_Horizontal"
 			(at 165.1 50.8 0)
 			(effects

Commit message: minor cleanup from the party
Parts:
- removed J5: Conn_01x01_Pin, Connector_PinHeader_2.54mm:PinHeader_1x01_P2.54mm_Horizontal, symbol Connector:Conn_01x01_Pin
- added J101: Conn_01x02_Pin, Connector_PinHeader_2.54mm:PinHeader_1x02_P2.54mm_Horizontal, symbol Connector:Conn_01x02_Pin
- renumbered H1 to H101, H2 to H102, H3 to H103, H4 to H104, J1 to J102, J2 to J103, J3 to J104, J4 to J105
Connections:
- net GND: now also J101.1 (Pin_1)
- net Signal Source/AUX_DAC_OUT: now also J101.2 (Pin_2)
Changed lines of the file:
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@@
+	(wire
+		(pts
+			(xy 158.75 40.64) (xy 161.29 40.64)
+		)
+		(stroke
+			(width 0)
+			(type default)
+		)
+	)
 	(wire
 		(pts
@@
 		(pts
 			(xy 50.8 92.71) (xy 68.58 92.71)
+		)
+		(stroke
+			(width 0)
+			(type default)
+		)
+	)
+	(wire
+		(pts
+			(xy 158.75 41.91) (xy 158.75 40.64)
 		)
 		(stroke
@@
 		(dnp no)
 		(fields_autoplaced yes)
-		(property "Reference" "H4"
+		(property "Reference" "H104"
 			(at 234.95 152.3999 0)
 			(effects
@@
 			(project "Main Board"
 				(path "/20aae4b7-3fb8-4924-82e8-1e7a29a313f8"
-					(reference "H4")
+					(reference "H104")
 					(unit 1)
 				)
@@
 		(dnp no)
 		(fields_autoplaced yes)
-		(property "Reference" "H3"
+		(property "Reference" "H103"
 			(at 234.95 147.3199 0)
 			(effects
@@
 			(project "Main Board"
 				(path "/20aae4b7-3fb8-4924-82e8-1e7a29a313f8"
-					(reference "H3")
+					(reference "H103")
 					(unit 1)
 				)
@@
 		(dnp no)
 		(fields_autoplaced yes)
-		(property "Reference" "#PWR01"
+		(property "Reference" "#PWR0102"
 			(at 165.1 62.23 0)
 			(effects
@@
 			(project ""
 				(path "/20aae4b7-3fb8-4924-82e8-1e7a29a313f8"
-					(reference "#PWR01")
+					(reference "#PWR0102")
+					(unit 1)
+				)
+			)
+		)
+	)
+	(symbol
+		(lib_id "power:GND")
+		(at 158.75 41.91 0)
+		(unit 1)
+		(exclude_from_sim no)
+		(in_bom yes)
+		(on_board yes)
+		(dnp no)
+		(fields_autoplaced yes)
+		(property "Reference" "#PWR0101"
+			(at 158.75 48.26 0)
+			(effects
+				(font
+					(size 1.27 1.27)
+				)
+				(hide yes)
+			)
+		)
+		(property "Value" "GND"
+			(at 158.75 46.99 0)
+			(effects
+				(font
+					(size 1.27 1.27)
+				)
+			)
+		)
+		(property "Footprint" ""
+			(at 158.75 41.91 0)
+			(effects
+				(font
+					(size 1.27 1.27)
+				)
+				(hide yes)
+			)
+		)
+		(property "Datasheet" ""
+			(at 158.75 41.91 0)
+			(effects
+				(font
+					(size 1.27 1.27)
+				)
+				(hide yes)
+			)
+		)
+		(property "Description" "Power symbol creates a global label with name \"GND\" , ground"
+			(at 158.75 41.91 0)
+			(effects
+				(font
+					(size 1.27 1.27)
+				)
+				(hide yes)
+			)
+		)
+		(pin "1"
+		)
+		(instances
+			(project "Main Board"
+				(path "/20aae4b7-3fb8-4924-82e8-1e7a29a313f8"
+					(reference "#PWR0101")
 					(unit 1)
 				)
@@
 		(dnp no)
 		(fields_autoplaced yes)
-		(property "Reference" "J4"
+		(property "Reference" "J105"
 			(at 168.91 113.3231 0)
 			(effects
@@
 			(project "Main Board"
 				(path "/20aae4b7-3fb8-4924-82e8-1e7a29a313f8"
-					(reference "J4")
-					(unit 1)
-				)
-			)
-		)
-	)
-	(symbol
-		(lib_id "Connector:Conn_01x01_Pin")
-		(at 166.37 38.1 180)
-		(unit 1)
-		(exclude_from_sim no)
-		(in_bom yes)
-		(on_board yes)
-		(dnp no)
-		(property "Reference" "J5"
-			(at 171.4256 38.1 0)
-			(effects
-				(font
-					(size 1.27 1.27)
-				)
-			)
-		)
-		(property "Value" "Conn_01x01_Pin"
-			(at 165.735 35.56 0)
-			(effects
-				(font
-					(size 1.27 1.27)
-				)
-				(hide yes)
-			)
-		)
-		(property "Footprint" "Connector_PinHeader_2.54mm:PinHeader_1x01_P2.54mm_Horizontal"
-			(at 166.37 38.1 0)
-			(effects
-				(font
-					(size 1.27 1.27)
-				)
-				(hide yes)
-			)
-		)
-		(property "Datasheet" "~"
-			(at 166.37 38.1 0)
-			(effects
-				(font
-					(size 1.27 1.27)
-				)
-				(hide yes)
-			)
-		)
-		(property "Description" "Generic connector, single row, 01x01, script generated"
-			(at 166.37 38.1 0)
-			(effects
-				(font
-					(size 1.27 1.27)
-				)
-				(hide yes)
-			)
-		)
-		(pin "1"
-		)
-		(instances
-			(project "Main Board"
-				(path "/20aae4b7-3fb8-4924-82e8-1e7a29a313f8"
-					(reference "J5")
+					(reference "J105")
 					(unit 1)
 				)
@@
 		(dnp no)
 		(fields_autoplaced yes)
-		(property "Reference" "J2"
+		(property "Reference" "J103"
 			(at 168.91 71.4131 0)
 			(effects
@@
 			(project "Main Board"
 				(path "/20aae4b7-3fb8-4924-82e8-1e7a29a313f8"
-					(reference "J2")
+					(reference "J103")
 					(unit 1)
 				)
@@
 		(dnp no)
 		(fields_autoplaced yes)
-		(property "Reference" "#PWR02"
+		(property "Reference" "#PWR0103"
 			(at 165.1 83.82 0)
 			(effects
@@
 			(project "Main Board"
 				(path "/20aae4b7-3fb8-4924-82e8-1e7a29a313f8"
-					(reference "#PWR02")
+					(reference "#PWR0103")
 					(unit 1)
 				)
@@
 		(dnp no)
 		(fields_autoplaced yes)
-		(property "Reference" "H2"
+		(property "Reference" "H102"
 			(at 234.95 142.2399 0)
 			(effects
@@
 			(project "Main Board"
 				(path "/20aae4b7-3fb8-4924-82e8-1e7a29a313f8"
-					(reference "H2")
+					(reference "H102")
+					(unit 1)
+				)
+			)
+		)
+	)
+	(symbol
+		(lib_id "Connector:Conn_01x02_Pin")
+		(at 166.37 40.64 180)
+		(unit 1)
+		(exclude_from_sim no)
+		(in_bom yes)
+		(on_board yes)
+		(dnp no)
+		(property "Reference" "J101"
+			(at 167.64 39.3699 0)
+			(effects
+				(font
+					(size 1.27 1.27)
+				)
+				(justify right)
+			)
+		)
+		(property "Value" "Conn_01x02_Pin"
+			(at 167.64 40.6399 0)
+			(effects
+				(font
+					(size 1.27 1.27)
+				)
+				(justify right)
+				(hide yes)
+			)
+		)
+		(property "Footprint" "Connector_PinHeader_2.54mm:PinHeader_1x02_P2.54mm_Horizontal"
+			(at 166.37 40.64 0)
+			(effects
+				(font
+					(size 1.27 1.27)
+				)
+				(hide yes)
+			)
+		)
+		(property "Datasheet" "~"
+			(at 166.37 40.64 0)
+			(effects
+				(font
+					(size 1.27 1.27)
+				)
+				(hide yes)
+			)
+		)
+		(property "Description" "Generic connector, single row, 01x02, script generated"
+			(at 166.37 40.64 0)
+			(effects
+				(font
+					(size 1.27 1.27)
+				)
+				(hide yes)
+			)
+		)
+		(pin "2"
+		)
+		(pin "1"
+		)
+		(instances
+			(project ""
+				(path "/20aae4b7-3fb8-4924-82e8-1e7a29a313f8"
+					(reference "J101")
 					(unit 1)
 				)
@@
 		(dnp no)
 		(fields_autoplaced yes)
-		(property "Reference" "J3"
+		(property "Reference" "J104"
 			(at 168.91 91.7331 0)
 			(effects
@@
 			(project "Main Board"
 				(path "/20aae4b7-3fb8-4924-82e8-1e7a29a313f8"
-					(reference "J3")
+					(reference "J104")
 					(unit 1)
 				)
@@
 		(dnp no)
 		(fields_autoplaced yes)
-		(property "Reference" "H1"
+		(property "Reference" "H101"
 			(at 234.95 137.1599 0)
 			(effects
@@
 			(project ""
 				(path "/20aae4b7-3fb8-4924-82e8-1e7a29a313f8"
-					(reference "H1")
+					(reference "H101")
 					(unit 1)
 				)
@@
 		(dnp no)
 		(fields_autoplaced yes)
-		(property "Reference" "J1"
+		(property "Reference" "J102"
 			(at 168.91 49.8231 0)
 			(effects
@@
 			(project ""
 				(path "/20aae4b7-3fb8-4924-82e8-1e7a29a313f8"
-					(reference "J1")
-					(unit 1)
-				)
+					(reference "J102")
+					(unit 1)
+				)

Commit message: footprints and tps
Parts:
- added TP?: ADC_2, TestPoint:TestPoint_Pad_2.0x2.0mm, symbol Connector:TestPoint
- added TP?: ADC_1, TestPoint:TestPoint_Pad_2.0x2.0mm, symbol Connector:TestPoint
- added TP?: DAC_1, TestPoint:TestPoint_Pad_2.0x2.0mm, symbol Connector:TestPoint
- added TP?: DAC_2, TestPoint:TestPoint_Pad_2.0x2.0mm, symbol Connector:TestPoint
Connections:
- net Current Amplifier/Out: now also TP?.1
- net Processor/Source.Bias: now also TP?.1
- net Processor/Source.Signal: now also TP?.1
- net Processor/VAmp.Out: now also TP?.1

Commit message: :(
Parts:
- gave numbers to parts that had none: 4
- renumbered H101 to H1, H102 to H2, H103 to H3, H104 to H4, J102 to J1, J103 to J2, J104 to J3, J105 to J4, J101 to J5
Changed lines of the file:
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@@
 		(dnp no)
 		(fields_autoplaced yes)
-		(property "Reference" "H104"
+		(property "Reference" "H4"
 			(at 234.95 152.3999 0)
 			(effects
@@
 			(project "Main Board"
 				(path "/20aae4b7-3fb8-4924-82e8-1e7a29a313f8"
-					(reference "H104")
+					(reference "H4")
 					(unit 1)
 				)
@@
 		(on_board yes)
 		(dnp no)
-		(property "Reference" "TP?"
+		(property "Reference" "TP2"
 			(at 55.88 96.0119 0)
 			(effects
@@
 			(project "Main Board"
 				(path "/20aae4b7-3fb8-4924-82e8-1e7a29a313f8"
-					(reference "TP?")
+					(reference "TP2")
 					(unit 1)
 				)
@@
 		(on_board yes)
 		(dnp no)
-		(property "Reference" "TP?"
+		(property "Reference" "TP3"
 			(at 55.88 118.8719 0)
 			(effects
@@
 			(project "Main Board"
 				(path "/20aae4b7-3fb8-4924-82e8-1e7a29a313f8"
-					(reference "TP?")
+					(reference "TP3")
 					(unit 1)
 				)
@@
 		(on_board yes)
 		(dnp no)
-		(property "Reference" "TP?"
+		(property "Reference" "TP4"
 			(at 57.15 18.2881 0)
 			(effects
@@
 			(project "Main Board"
 				(path "/20aae4b7-3fb8-4924-82e8-1e7a29a313f8"
-					(reference "TP?")
+					(reference "TP4")
 					(unit 1)
 				)
@@
 		(dnp no)
 		(fields_autoplaced yes)
-		(property "Reference" "H103"
+		(property "Reference" "H3"
 			(at 234.95 147.3199 0)
 			(effects
@@
 			(project "Main Board"
 				(path "/20aae4b7-3fb8-4924-82e8-1e7a29a313f8"
-					(reference "H103")
+					(reference "H3")
 					(unit 1)
 				)
@@
 		(dnp no)
 		(fields_autoplaced yes)
-		(property "Reference" "#PWR0102"
+		(property "Reference" "#PWR02"
 			(at 165.1 62.23 0)
 			(effects
@@
 			(project ""
 				(path "/20aae4b7-3fb8-4924-82e8-1e7a29a313f8"
-					(reference "#PWR0102")
+					(reference "#PWR02")
 					(unit 1)
 				)
@@
 		(dnp no)
 		(fields_autoplaced yes)
-		(property "Reference" "#PWR0101"
+		(property "Reference" "#PWR01"
 			(at 158.75 48.26 0)
 			(effects
@@
 			(project "Main Board"
 				(path "/20aae4b7-3fb8-4924-82e8-1e7a29a313f8"
-					(reference "#PWR0101")
+					(reference "#PWR01")
 					(unit 1)
 				)
@@
 		(dnp no)
 		(fields_autoplaced yes)
-		(property "Reference" "J105"
+		(property "Reference" "J4"
 			(at 168.91 113.3231 0)
 			(effects
@@
 			(project "Main Board"
 				(path "/20aae4b7-3fb8-4924-82e8-1e7a29a313f8"
-					(reference "J105")
+					(reference "J4")
 					(unit 1)
 				)
@@
 		(dnp no)
 		(fields_autoplaced yes)
-		(property "Reference" "J103"
+		(property "Reference" "J2"
 			(at 168.91 71.4131 0)
 			(effects
@@
 			(project "Main Board"
 				(path "/20aae4b7-3fb8-4924-82e8-1e7a29a313f8"
-					(reference "J103")
+					(reference "J2")
 					(unit 1)
 				)
@@
 		(dnp no)
 		(fields_autoplaced yes)
-		(property "Reference" "#PWR0103"
+		(property "Reference" "#PWR03"
 			(at 165.1 83.82 0)
 			(effects
@@
 			(project "Main Board"
 				(path "/20aae4b7-3fb8-4924-82e8-1e7a29a313f8"
-					(reference "#PWR0103")
+					(reference "#PWR03")
 					(unit 1)
 				)
@@
 		(on_board yes)
 		(dnp no)
-		(property "Reference" "TP?"
+		(property "Reference" "TP1"
 			(at 50.8 23.3681 0)
 			(effects
@@
 			(project "Main Board"
 				(path "/20aae4b7-3fb8-4924-82e8-1e7a29a313f8"
-					(reference "TP?")
+					(reference "TP1")
 					(unit 1)
 				)
@@
 		(dnp no)
 		(fields_autoplaced yes)
-		(property "Reference" "H102"
+		(property "Reference" "H2"
 			(at 234.95 142.2399 0)
 			(effects
@@
 			(project "Main Board"
 				(path "/20aae4b7-3fb8-4924-82e8-1e7a29a313f8"
-					(reference "H102")
+					(reference "H2")
 					(unit 1)
 				)
@@
 		(on_board yes)
 		(dnp no)
-		(property "Reference" "J101"
+		(property "Reference" "J5"
 			(at 167.64 39.3699 0)
 			(effects
@@
 			(project ""
 				(path "/20aae4b7-3fb8-4924-82e8-1e7a29a313f8"
-					(reference "J101")
+					(reference "J5")
 					(unit 1)
 				)
@@
 		(dnp no)
 		(fields_autoplaced yes)
-		(property "Reference" "J104"
+		(property "Reference" "J3"
 			(at 168.91 91.7331 0)
 			(effects
@@
 			(project "Main Board"
 				(path "/20aae4b7-3fb8-4924-82e8-1e7a29a313f8"
-					(reference "J104")
+					(reference "J3")
 					(unit 1)
 				)
@@
 		(dnp no)
 		(fields_autoplaced yes)
-		(property "Reference" "H101"
+		(property "Reference" "H1"
 			(at 234.95 137.1599 0)
 			(effects
@@
 			(project ""
 				(path "/20aae4b7-3fb8-4924-82e8-1e7a29a313f8"
-					(reference "H101")
+					(reference "H1")
 					(unit 1)
 				)
@@
 		(dnp no)
 		(fields_autoplaced yes)
-		(property "Reference" "J102"
+		(property "Reference" "J1"
 			(at 168.91 49.8231 0)
 			(effects
@@
 			(project ""
 				(path "/20aae4b7-3fb8-4924-82e8-1e7a29a313f8"
-					(reference "J102")
-					(unit 1)
-				)
+					(reference "J1")
+					(unit 1)
+				)

Commit message: :(
Parts:
- J5: footprint Connector_PinHeader_2.54mm:PinHeader_1x02_P2.54mm_Horizontal -> Connector_PinHeader_2.54mm:PinHeader_1x02_P2.54mm_Vertical
Changed lines of the file:
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@@
 			)
 		)
-		(property "Footprint" "Connector_PinHeader_2.54mm:PinHeader_1x02_P2.54mm_Horizontal"
+		(property "Footprint" "Connector_PinHeader_2.54mm:PinHeader_1x02_P2.54mm_Vertical"
 			(at 166.37 40.64 0)
 			(effects

Commit message: tired
Other:
- sheet Processor ports: added I_B_MON; removed none
Changed lines of the file:
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@@
+			)
+		)
+		(pin "I_B_MON" input
+			(at 50.8 130.81 0)
+			(effects
+				(font
+					(size 1.27 1.27)
+				)
+				(justify right)
 			)
 		)

Commit message: xcfdfxgfdfgdsf
Other:
- note removed: "https://www.aliexpress.com/item/1005005482292733.html"
Changed lines of the file:
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@@
-		)
-	)
-	(text "https://www.aliexpress.com/item/1005005482292733.html"
-		(exclude_from_sim no)
-		(at 195.58 66.04 0)
-		(effects
-			(font
-				(size 1.27 1.27)
-			)
 		)
 	)
